Commit message: add ccs configuration

File: rokae_ar5_description/xacro/arm_srs.xacro (robot description, xacro)
@@ -13,11 +13,11 @@
 			<visual>
 				<geometry>
-					<mesh filename="file://$(find rokae_ar5_description)/meshes/base.obj" scale="1 ${direction} 1"/>
-				</geometry>
-			</visual>
-			<xacro:if value="${collider == 'convex'}">
-				<collision>
-					<geometry>
-						<mesh filename="file://$(find rokae_ar5_description)/meshes/base.obj" scale="1 ${direction} 1"/>
+					<mesh filename="file://$(find rokae_ar5_description)/meshes/srs/base.obj" scale="1 ${direction} 1"/>
+				</geometry>
+			</visual>
+			<xacro:if value="${collider == 'convex'}">
+				<collision>
+					<geometry>
+						<mesh filename="file://$(find rokae_ar5_description)/meshes/srs/base.obj" scale="1 ${direction} 1"/>
 					</geometry>
 				</collision>
@@ -49,11 +49,11 @@
 			<visual>
 				<geometry>
-					<mesh filename="file://$(find rokae_ar5_description)/meshes/link1.obj" scale="1 ${direction} 1"/>
-				</geometry>
-			</visual>
-			<xacro:if value="${collider == 'convex'}">
-				<collision>
-					<geometry>
-						<mesh filename="file://$(find rokae_ar5_description)/meshes/link1.obj" scale="1 ${direction} 1"/>
+					<mesh filename="file://$(find rokae_ar5_description)/meshes/srs/link1.obj" scale="1 ${direction} 1"/>
+				</geometry>
+			</visual>
+			<xacro:if value="${collider == 'convex'}">
+				<collision>
+					<geometry>
+						<mesh filename="file://$(find rokae_ar5_description)/meshes/srs/link1.obj" scale="1 ${direction} 1"/>
 					</geometry>
 				</collision>
@@ -85,11 +85,11 @@
 			<visual>
 				<geometry>
-					<mesh filename="file://$(find rokae_ar5_description)/meshes/link2.obj" scale="1 ${direction} 1"/>
-				</geometry>
-			</visual>
-			<xacro:if value="${collider == 'convex'}">
-				<collision>
-					<geometry>
-						<mesh filename="file://$(find rokae_ar5_description)/meshes/link2.obj" scale="1 ${direction} 1"/>
+					<mesh filename="file://$(find rokae_ar5_description)/meshes/srs/link2.obj" scale="1 ${direction} 1"/>
+				</geometry>
+			</visual>
+			<xacro:if value="${collider == 'convex'}">
+				<collision>
+					<geometry>
+						<mesh filename="file://$(find rokae_ar5_description)/meshes/srs/link2.obj" scale="1 ${direction} 1"/>
 					</geometry>
 				</collision>
@@ -119,13 +119,15 @@
 				<origin xyz="${direction*-0.007574792} 0.001848523 -0.017501298"/>
 			</inertial>
-			<visual>
-				<geometry>
-					<mesh filename="file://$(find rokae_ar5_description)/meshes/link3.obj" scale="1 ${direction} 1"/>
-				</geometry>
-			</visual>
-			<xacro:if value="${collider == 'convex'}">
-				<collision>
-					<geometry>
-						<mesh filename="file://$(find rokae_ar5_description)/meshes/link3.obj" scale="1 ${direction} 1"/>
+			<xacro:if value="${collider == 'convex'}">
+				<visual>
+					<geometry>
+						<mesh filename="file://$(find rokae_ar5_description)/meshes/srs/link3.obj" scale="1 ${direction} 1"/>
+					</geometry>
+				</visual>
+			</xacro:if>
+			<xacro:if value="${collider == 'convex'}">
+				<collision>
+					<geometry>
+						<mesh filename="file://$(find rokae_ar5_description)/meshes/srs/link3.obj" scale="1 ${direction} 1"/>
 					</geometry>
 				</collision>
@@ -164,17 +166,17 @@
 			<visual>
 				<geometry>
-					<mesh filename="file://$(find rokae_ar5_description)/meshes/link4.obj" scale="1 ${direction} 1"/>
-				</geometry>
-			</visual>
-			<xacro:if value="${collider == 'convex'}">
-				<collision>
-					<geometry>
-						<mesh filename="file://$(find rokae_ar5_description)/meshes/link4.obj" scale="1 ${direction} 1"/>
-					</geometry>
-				</collision>
-			</xacro:if>
-			<xacro:if value="${collider == 'simple'}">
-				<collision>
-					<origin xyz="-0.01 0 0.10085"/>
+					<mesh filename="file://$(find rokae_ar5_description)/meshes/srs/link4.obj" scale="1 ${direction} 1"/>
+				</geometry>
+			</visual>
+			<xacro:if value="${collider == 'convex'}">
+				<collision>
+					<geometry>
+						<mesh filename="file://$(find rokae_ar5_description)/meshes/srs/link4.obj" scale="1 ${direction} 1"/>
+					</geometry>
+				</collision>
+			</xacro:if>
+			<xacro:if value="${collider == 'simple'}">
+				<collision>
+					<origin xyz="-0.01 0 0.08085"/>
 					<geometry>
 						<cylinder length="0.10" radius="0.03789"/>
@@ -200,11 +202,11 @@
 			<visual>
 				<geometry>
-					<mesh filename="file://$(find rokae_ar5_description)/meshes/link5.obj" scale="1 ${direction} 1"/>
-				</geometry>
-			</visual>
-			<xacro:if value="${collider == 'convex'}">
-				<collision>
-					<geometry>
-						<mesh filename="file://$(find rokae_ar5_description)/meshes/link5.obj" scale="1 ${direction} 1"/>
+					<mesh filename="file://$(find rokae_ar5_description)/meshes/srs/link5.obj" scale="1 ${direction} 1"/>
+				</geometry>
+			</visual>
+			<xacro:if value="${collider == 'convex'}">
+				<collision>
+					<geometry>
+						<mesh filename="file://$(find rokae_ar5_description)/meshes/srs/link5.obj" scale="1 ${direction} 1"/>
 					</geometry>
 				</collision>
@@ -236,11 +238,11 @@
 			<visual>
 				<geometry>
-					<mesh filename="file://$(find rokae_ar5_description)/meshes/link6.obj" scale="1 ${direction} 1"/>
-				</geometry>
-			</visual>
-			<xacro:if value="${collider == 'convex'}">
-				<collision>
-					<geometry>
-						<mesh filename="file://$(find rokae_ar5_description)/meshes/link6.obj" scale="1 ${direction} 1"/>
+					<mesh filename="file://$(find rokae_ar5_description)/meshes/srs/link6.obj" scale="1 ${direction} 1"/>
+				</geometry>
+			</visual>
+			<xacro:if value="${collider == 'convex'}">
+				<collision>
+					<geometry>
+						<mesh filename="file://$(find rokae_ar5_description)/meshes/srs/link6.obj" scale="1 ${direction} 1"/>
 					</geometry>
 				</collision>
@@ -272,5 +274,5 @@
 			<visual>
 				<geometry>
-					<mesh filename="file://$(find rokae_ar5_description)/meshes/link7.obj" scale="1 ${direction} 1"/>
+					<mesh filename="file://$(find rokae_ar5_description)/meshes/srs/link7.obj" scale="1 ${direction} 1"/>
 				</geometry>
 			</visual>

File: rokae_ar5_description/xacro/robot.xacro (robot description, xacro)
@@ -3,9 +3,11 @@
   <xacro:arg name="collider" default="convex"/>
   <xacro:arg name="type" default="left"/>
-  <xacro:include filename="$(find rokae_ar5_description)/xacro/arm.xacro"/>
+  <!-- SRS ARM Configurations -->
   <xacro:if value="${'$(arg type)' == 'left'}">
+    <xacro:include filename="$(find rokae_ar5_description)/xacro/arm_srs.xacro"/>
     <xacro:Arm name="" collider="$(arg collider)"/>
   </xacro:if>
   <xacro:if value="${'$(arg type)' == 'left_rg75'}">
+    <xacro:include filename="$(find rokae_ar5_description)/xacro/arm_srs.xacro"/>
     <xacro:Arm name="" collider="$(arg collider)"/>
     <xacro:include filename="$(find jodell_description)/xacro/RG75-300.xacro"/>
@@ -18,7 +20,9 @@
   </xacro:if>
   <xacro:if value="${'$(arg type)' == 'right'}">
+    <xacro:include filename="$(find rokae_ar5_description)/xacro/arm_srs.xacro"/>
     <xacro:Arm name="" collider="$(arg collider)" direction="-1"/>
   </xacro:if>
   <xacro:if value="${'$(arg type)' == 'right_rg75'}">
+    <xacro:include filename="$(find rokae_ar5_description)/xacro/arm_srs.xacro"/>
     <xacro:Arm name="" collider="$(arg collider)" direction="-1"/>
     <xacro:include filename="$(find jodell_description)/xacro/RG75-300.xacro"/>
@@ -31,4 +35,5 @@
   </xacro:if>
   <xacro:if value="${'$(arg type)' == 'dual' or '$(arg type)' == 'dual_rg75'}">
+    <xacro:include filename="$(find rokae_ar5_description)/xacro/arm_srs.xacro"/>
     <link name="base_link"/>
     <link name="arm_base">
@@ -72,3 +77,77 @@
     </xacro:if>
   </xacro:if>
+  <!-- CCS ARM Configurations -->
+  <xacro:if value="${'$(arg type)' == 'ccs_left'}">
+    <xacro:include filename="$(find rokae_ar5_description)/xacro/arm_ccs.xacro"/>
+    <xacro:Arm name="" collider="$(arg collider)" direction="1"/>
+  </xacro:if>
+  <xacro:if value="${'$(arg type)' == 'ccs_left_rg75'}">
+    <xacro:include filename="$(find rokae_ar5_description)/xacro/arm_ccs.xacro"/>
+    <xacro:Arm name="" collider="$(arg collider)"/>
+    <xacro:include filename="$(find jodell_description)/xacro/RG75-300.xacro"/>
+    <xacro:RG75-300 name="" use_flange="true"/>
+    <joint name="gripper_base_joint" type="fixed">
+      <origin xyz="0 0 -0.0045" rpy="0 0 -1.5708"/>
+      <parent link="tcp"/>
+      <child link="flange"/>
+    </joint>
+  </xacro:if>
+  <xacro:if value="${'$(arg type)' == 'ccs_right'}">
+    <xacro:include filename="$(find rokae_ar5_description)/xacro/arm_ccs.xacro"/>
+    <xacro:Arm name="" collider="$(arg collider)" direction="-1"/>
+  </xacro:if>
+  <xacro:if value="${'$(arg type)' == 'ccs_right_rg75'}">
+    <xacro:include filename="$(find rokae_ar5_description)/xacro/arm_ccs.xacro"/>
+    <xacro:Arm name="" collider="$(arg collider)" direction="-1"/>
+    <xacro:include filename="$(find jodell_description)/xacro/RG75-300.xacro"/>
+    <xacro:RG75-300 name="" use_flange="true"/>
+    <joint name="gripper_base_joint" type="fixed">
+      <origin xyz="0 0 -0.0045" rpy="0 0 1.5708"/>
+      <parent link="tcp"/>
+      <child link="flange"/>
+    </joint>
+  </xacro:if>
+  <xacro:if value="${'$(arg type)' == 'ccs_dual' or '$(arg type)' == 'ccs_dual_rg75'}">
+    <xacro:include filename="$(find rokae_ar5_description)/xacro/arm_ccs.xacro"/>
+    <link name="base_link"/>
+    <link name="arm_base">
+      <collision>
+        <origin xyz="0.0091 0 -0.086"/>
+        <geometry>
+          <box size="0.2509 0.35 0.5029"/>
+        </geometry>
+      </collision>
+    </link>
+    <joint name="arm_base_joint" type="fixed">
+      <parent link="base_link"/>
+      <child link="arm_base"/>
+    </joint>
+    <joint name="left_arm_mount" type="fixed">
+      <parent link="arm_base"/>
+      <child link="left_base_link"/>
+      <origin xyz="0.0 0.12 0" rpy="-1.57 1.57 0"/>
+    </joint>
+    <joint name="right_arm_mount" type="fixed">
+      <parent link="arm_base"/>
+      <child link="right_base_link"/>
+      <origin xyz="0.0 -0.12 0" rpy="1.57 1.57 0"/>
+    </joint>
+    <xacro:Arm name="left" collider="$(arg collider)" direction="1"/>
+    <xacro:Arm name="right" collider="$(arg collider)" direction="-1"/>
+    <xacro:if value="${'$(arg type)' == 'ccs_dual_rg75'}">
+      <xacro:include filename="$(find jodell_description)/xacro/RG75-300.xacro"/>
+      <xacro:RG75-300 name="left" use_flange="true"/>
+      <xacro:RG75-300 name="right" use_flange="true"/>
+      <joint name="left_gripper_base_joint" type="fixed">
+        <origin xyz="0 0 -0.0045"/>
+        <parent link="left_tcp"/>
+        <child link="left_flange"/>
+      </joint>
+      <joint name="right_gripper_base_joint" type="fixed">
+        <origin xyz="0 0 -0.0045"/>
+        <parent link="right_tcp"/>
+        <child link="right_flange"/>
+      </joint>
+    </xacro:if>
+  </xacro:if>
 </robot>

Commit message: fix srs mesh problem

File: rokae_ar5_description/xacro/arm_srs.xacro (robot description, xacro)
@@ -119,11 +119,9 @@
 				<origin xyz="${direction*-0.007574792} 0.001848523 -0.017501298"/>
 			</inertial>
-			<xacro:if value="${collider == 'convex'}">
-				<visual>
-					<geometry>
-						<mesh filename="file://$(find rokae_ar5_description)/meshes/srs/link3.obj" scale="1 ${direction} 1"/>
-					</geometry>
-				</visual>
-			</xacro:if>
+			<visual>
+				<geometry>
+					<mesh filename="file://$(find rokae_ar5_description)/meshes/srs/link3.obj" scale="1 ${direction} 1"/>
+				</geometry>
+			</visual>
 			<xacro:if value="${collider == 'convex'}">
 				<collision>
