Commit message: add arm base frame

File: rokae_ar5_description/urdf/rokae_ar5_dual.urdf (robot description, URDF)
Before this commit: robot RokaeAR5Dual, 17 links, 16 joints
Links:
- added link arm_base
Joints:
- added joint arm_base_joint: type fixed, parent base_link, child arm_base
- joint left_arm_mount: parent base_link -> arm_base
- joint right_arm_mount: parent base_link -> arm_base

File: rokae_ar5_description/xacro/robot.xacro (robot description, xacro)
@@ -12,11 +12,16 @@
   <xacro:if value="${'$(arg type)' == 'dual'}">
     <link name="base_link"/>
+    <link name="arm_base"/>
+    <joint name="arm_base_joint" type="fixed">
+      <parent link="base_link"/>
+      <child link="arm_base"/>
+    </joint>
     <joint name="left_arm_mount" type="fixed">
-      <parent link="base_link"/>
+      <parent link="arm_base"/>
       <child link="left_base_link"/>
       <origin xyz="0.0 0.12 0" rpy="-1.57 1.57 0"/>
     </joint>
     <joint name="right_arm_mount" type="fixed">
-      <parent link="base_link"/>
+      <parent link="arm_base"/>
       <child link="right_base_link"/>
       <origin xyz="0.0 -0.12 0" rpy="1.57 1.57 0"/>

Commit message: ADD self collision config for rokae ar5 dual

File: rokae_ar5_description/urdf/rokae_ar5_dual.urdf (robot description, URDF)
Before this commit: robot RokaeAR5, 18 links, 17 joints
Links:
- link arm_base: geometry collision box size=0.2509 0.35 0.5029
- link left_base_link: geometry collision cylinder length=0.105 radius=0.045; visual mesh filename=package://rokae_ar5_description/meshes/base.obj scale=1 1 1
- link left_link1: geometry collision cylinder length=0.1354 radius=0.0560; visual mesh filename=package://rokae_ar5_description/meshes/link1.obj scale=1 1 1
- link left_link2: geometry collision cylinder length=0.11413 radius=0.053; visual mesh filename=package://rokae_ar5_description/meshes/link2.obj scale=1 1 1
- link left_link3: geometry collision cylinder length=0.096 radius=0.053; collision cylinder length=0.1284 radius=0.0484
- link left_link4: geometry collision cylinder length=0.10 radius=0.03789; visual mesh filename=package://rokae_ar5_description/meshes/link4.obj scale=1 1 1
- link left_link5: geometry collision cylinder length=0.107 radius=0.0383; visual mesh filename=package://rokae_ar5_description/meshes/link5.obj scale=1 1 1
- link left_link6: geometry collision cylinder length=0.1238 radius=0.04; visual mesh filename=package://rokae_ar5_description/meshes/link6.obj scale=1 1 1
- link right_base_link: geometry collision cylinder length=0.105 radius=0.045; visual mesh filename=package://rokae_ar5_description/meshes/base.obj scale=1 -1 1
- link right_link1: geometry collision cylinder length=0.1354 radius=0.0560; visual mesh filename=package://rokae_ar5_description/meshes/link1.obj scale=1 -1 1
- link right_link2: geometry collision cylinder length=0.11413 radius=0.053; visual mesh filename=package://rokae_ar5_description/meshes/link2.obj scale=1 -1 1
- link right_link3: geometry collision cylinder length=0.096 radius=0.053; collision cylinder length=0.1284 radius=0.0484
- link right_link4: geometry collision cylinder length=0.10 radius=0.03789; visual mesh filename=package://rokae_ar5_description/meshes/link4.obj scale=1 -1 1
- link right_link5: geometry collision cylinder length=0.107 radius=0.0383; visual mesh filename=package://rokae_ar5_description/meshes/link5.obj scale=1 -1 1
- link right_link6: geometry collision cylinder length=0.1238 radius=0.04; visual mesh filename=package://rokae_ar5_description/meshes/link6.obj scale=1 -1 1

File: rokae_ar5_description/xacro/arm.xacro (robot description, xacro)
@@ -16,9 +16,19 @@
 				</geometry>
 			</visual>
-			<collision>
-				<geometry>
-					<mesh filename="file://$(find rokae_ar5_description)/meshes/base.obj" scale="1 ${direction} 1"/>
-				</geometry>
-			</collision>
+			<xacro:if value="${collider == 'convex'}">
+				<collision>
+					<geometry>
+						<mesh filename="file://$(find rokae_ar5_description)/meshes/base.obj" scale="1 ${direction} 1"/>
+					</geometry>
+				</collision>
+			</xacro:if>
+			<xacro:if value="${collider == 'simple'}">
+				<collision>
+					<origin xyz="0 0 0.05025"/>
+					<geometry>
+						<cylinder length="0.105" radius="0.045"/>
+					</geometry>
+				</collision>
+			</xacro:if>
 		</link>
 		<!-- Joint 1 -->
@@ -42,9 +52,19 @@
 				</geometry>
 			</visual>
-			<collision>
-				<geometry>
-					<mesh filename="file://$(find rokae_ar5_description)/meshes/link1.obj" scale="1 ${direction} 1"/>
-				</geometry>
-			</collision>
+			<xacro:if value="${collider == 'convex'}">
+				<collision>
+					<geometry>
+						<mesh filename="file://$(find rokae_ar5_description)/meshes/link1.obj" scale="1 ${direction} 1"/>
+					</geometry>
+				</collision>
+			</xacro:if>
+			<xacro:if value="${collider == 'simple'}">
+				<collision>
+					<origin rpy="1.5708 0 0"/>
+					<geometry>
+						<cylinder length="0.1354" radius="0.0560"/>
+					</geometry>
+				</collision>
+			</xacro:if>
 		</link>
 		<!-- Joint 2 -->
@@ -68,9 +88,19 @@
 				</geometry>
 			</visual>
-			<collision>
-				<geometry>
-					<mesh filename="file://$(find rokae_ar5_description)/meshes/link2.obj" scale="1 ${direction} 1"/>
-				</geometry>
-			</collision>
+			<xacro:if value="${collider == 'convex'}">
+				<collision>
+					<geometry>
+						<mesh filename="file://$(find rokae_ar5_description)/meshes/link2.obj" scale="1 ${direction} 1"/>
+					</geometry>
+				</collision>
+			</xacro:if>
+			<xacro:if value="${collider == 'simple'}">
+				<collision>
+					<origin xyz="0 0 0.10600"/>
+					<geometry>
+						<cylinder length="0.11413" radius="0.053"/>
+					</geometry>
+				</collision>
+			</xacro:if>
 		</link>
 		<!-- Joint 3 -->
@@ -94,9 +124,25 @@
 				</geometry>
 			</visual>
-			<collision>
-				<geometry>
-					<mesh filename="file://$(find rokae_ar5_description)/meshes/link3.obj" scale="1 ${direction} 1"/>
-				</geometry>
-			</collision>
+			<xacro:if value="${collider == 'convex'}">
+				<collision>
+					<geometry>
+						<mesh filename="file://$(find rokae_ar5_description)/meshes/link3.obj" scale="1 ${direction} 1"/>
+					</geometry>
+				</collision>
+			</xacro:if>
+			<xacro:if value="${collider == 'simple'}">
+				<collision>
+					<origin xyz="0 0 -0.0863"/>
+					<geometry>
+						<cylinder length="0.096" radius="0.053"/>
+					</geometry>
+				</collision>
+				<collision>
+					<origin xyz="0.00946 0 0" rpy="1.5708 0 0"/>
+					<geometry>
+						<cylinder length="0.1284" radius="0.0484"/>
+					</geometry>
+				</collision>
+			</xacro:if>
 		</link>
 		<!-- Joint 4 -->
@@ -121,9 +167,19 @@
 				</geometry>
 			</visual>
-			<collision>
-				<geometry>
-					<mesh filename="file://$(find rokae_ar5_description)/meshes/link4.obj" scale="1 ${direction} 1"/>
-				</geometry>
-			</collision>
+			<xacro:if value="${collider == 'convex'}">
+				<collision>
+					<geometry>
+						<mesh filename="file://$(find rokae_ar5_description)/meshes/link4.obj" scale="1 ${direction} 1"/>
+					</geometry>
+				</collision>
+			</xacro:if>
+			<xacro:if value="${collider == 'simple'}">
+				<collision>
+					<origin xyz="-0.01 0 0.10085"/>
+					<geometry>
+						<cylinder length="0.10" radius="0.03789"/>
+					</geometry>
+				</collision>
+			</xacro:if>
 		</link>
 		<!-- Joint 5 -->
@@ -147,9 +203,19 @@
 				</geometry>
 			</visual>
-			<collision>
-				<geometry>
-					<mesh filename="file://$(find rokae_ar5_description)/meshes/link5.obj" scale="1 ${direction} 1"/>
-				</geometry>
-			</collision>
+			<xacro:if value="${collider == 'convex'}">
+				<collision>
+					<geometry>
+						<mesh filename="file://$(find rokae_ar5_description)/meshes/link5.obj" scale="1 ${direction} 1"/>
+					</geometry>
+				</collision>
+			</xacro:if>
+			<xacro:if value="${collider == 'simple'}">
+				<collision>
+					<origin rpy="1.5708 0 0"/>
+					<geometry>
+						<cylinder length="0.107" radius="0.0383"/>
+					</geometry>
+				</collision>
+			</xacro:if>
 		</link>
 		<!-- Joint 6 -->
@@ -173,9 +239,19 @@
 				</geometry>
 			</visual>
-			<collision>
-				<geometry>
-					<mesh filename="file://$(find rokae_ar5_description)/meshes/link6.obj" scale="1 ${direction} 1"/>
-				</geometry>
-			</collision>
+			<xacro:if value="${collider == 'convex'}">
+				<collision>
+					<geometry>
+						<mesh filename="file://$(find rokae_ar5_description)/meshes/link6.obj" scale="1 ${direction} 1"/>
+					</geometry>
+				</collision>
+			</xacro:if>
+			<xacro:if value="${collider == 'simple'}">
+				<collision>
+					<origin xyz="0 0 0.10401"/>
+					<geometry>
+						<cylinder length="0.1238" radius="0.04"/>
+					</geometry>
+				</collision>
+			</xacro:if>
 		</link>
 		<!-- Joint 7 -->

File: rokae_ar5_description/xacro/robot.xacro (robot description, xacro)
@@ -12,5 +12,12 @@
   <xacro:if value="${'$(arg type)' == 'dual'}">
     <link name="base_link"/>
-    <link name="arm_base"/>
+    <link name="arm_base">
+      <collision>
+        <origin xyz="0.0091 0 -0.086"/>
+        <geometry>
+          <box size="0.2509 0.35 0.5029"/>
+        </geometry>
+      </collision>
+    </link>
     <joint name="arm_base_joint" type="fixed">
       <parent link="base_link"/>
@@ -27,6 +34,6 @@
       <origin xyz="0.0 -0.12 0" rpy="1.57 1.57 0"/>
     </joint>
-    <xacro:Arm name="left" direction="1"/>
-    <xacro:Arm name="right" direction="-1"/>
+    <xacro:Arm name="left" collider="$(arg collider)" direction="1"/>
+    <xacro:Arm name="right" collider="$(arg collider)" direction="-1"/>
   </xacro:if>
 </robot>
