Commit message: ocs2 arm controller config for dual ccs

File: rokae_ar5_description/xacro/ros2_control/robot.xacro (robot description, xacro)
@@ -1,120 +1,139 @@
 <?xml version="1.0"?>
 <robot xmlns:xacro="http://www.ros.org/wiki/xacro" name="AR5">
-    <xacro:arg name="ros2_control_hardware_type" default="mock_components"/>
-    <link name="world"/>
-    <joint name="world_fixed" type="fixed">
-        <parent link="world"/>
-        <child link="base_link"/>
-        <origin/>
-    </joint>
-    <xacro:include filename="$(find rokae_ar5_description)/xacro/robot.xacro"/>
-    <xacro:include filename="$(find rokae_ar5_description)/xacro/ros2_control/interfaces.xacro"/>
-    <xacro:if value="${'$(arg ros2_control_hardware_type)' == 'real'}">
-        <xacro:if value="${'$(arg type)' == 'dual' or '$(arg type)' == 'dual_rg75' }">
-            <ros2_control name="ar5_left_system" type="system">
-                <hardware>
-                    <plugin>rokae_ros2_control/RokaeHardware</plugin>
-                    <param name="arm_ip">192.168.2.160</param>
-                    <param name="joint_impedance">500,500,500,500,50,50,50</param>
-                </hardware>
-                <xacro:ar5_interfaces name="left"/>
-                <xacro:if value="${'$(arg type)' != 'dual'}">
-                    <joint name="left_gripper_joint">
-                        <command_interface name="position"/>
-                        <state_interface name="position">
-                            <param name="initial_value">0</param>
-                        </state_interface>
-                    </joint>
-                </xacro:if>
-            </ros2_control>
-            <ros2_control name="ar5_right_system" type="system">
-                <hardware>
-                    <plugin>rokae_ros2_control/RokaeHardware</plugin>
-                    <param name="arm_ip">192.168.2.161</param>
-                    <param name="joint_impedance">500,500,500,500,50,50,50</param>
-                </hardware>
-                <xacro:ar5_interfaces name="right"/>
-                <xacro:if value="${'$(arg type)' != 'dual'}">
-                    <joint name="right_gripper_joint">
-                        <command_interface name="position"/>
-                        <state_interface name="position">
-                            <param name="initial_value">0</param>
-                        </state_interface>
-                    </joint>
-                </xacro:if>
-            </ros2_control>
-        </xacro:if>
-        <xacro:unless value="${'$(arg type)' == 'dual' or '$(arg type)' == 'dual_rg75'}">
-            <ros2_control name="ar5System" type="system">
-                <hardware>
-                    <plugin>rokae_ros2_control/RokaeHardware</plugin>
-                    <xacro:if value="${'$(arg type)' == 'left'}">
-                        <param name="arm_ip">192.168.2.160</param>
-                    </xacro:if>
-                    <xacro:if value="${'$(arg type)' == 'left_rg75'}">
-                        <param name="arm_ip">192.168.2.160</param>
-                    </xacro:if>
-                    <xacro:if value="${'$(arg type)' == 'right'}">
-                        <param name="arm_ip">192.168.2.161</param>
-                    </xacro:if>
-                    <xacro:if value="${'$(arg type)' == 'right_rg75'}">
-                        <param name="arm_ip">192.168.2.161</param>
-                    </xacro:if>
-                    <!--					<param name="joint_impedance">200,200,200,200,100,100,100</param>-->
-                    <param name="local_ip">192.168.2.233</param>
-                </hardware>
-                <xacro:ar5_interfaces name=""/>
-                <xacro:if value="${'$(arg type)' != 'left' and '$(arg type)' != 'right'}">
-                    <joint name="gripper_joint">
-                        <command_interface name="position"/>
-                        <state_interface name="position">
-                            <param name="initial_value">0</param>
-                        </state_interface>
-                    </joint>
-                </xacro:if>
-            </ros2_control>
-        </xacro:unless>
-    </xacro:if>
-    <xacro:unless value="${'$(arg ros2_control_hardware_type)' == 'real'}">
-        <ros2_control name="ar5System" type="system">
-            <hardware>
-                <xacro:if value="${'$(arg ros2_control_hardware_type)' == 'gz'}">
-                    <plugin>gz_ros2_control/GazeboSimSystem</plugin>
-                </xacro:if>
-                <xacro:if value="${'$(arg ros2_control_hardware_type)' == 'mock_components'}">
-                    <plugin>mock_components/GenericSystem</plugin>
-                </xacro:if>
-                <xacro:if value="${'$(arg ros2_control_hardware_type)' == 'isaac'}">
-                    <plugin>topic_based_ros2_control/TopicBasedSystem</plugin>
-                    <param name="joint_commands_topic">/isaac/joint_command</param>
-                    <param name="joint_states_topic">/isaac/joint_states</param>
-                    <param name="sum_wrapped_joint_states">false</param>
-                    <param name="initialize_commands_from_state">true</param>
-                </xacro:if>
-            </hardware>
-            <xacro:if value="${'$(arg type)' == 'dual'}">
-                <xacro:ar5_interfaces name="left"/>
-                <xacro:ar5_interfaces name="right"/>
-            </xacro:if>
-            <xacro:unless value="${'$(arg type)' == 'dual'}">
-                <xacro:ar5_interfaces name=""/>
-            </xacro:unless>
-        </ros2_control>
-    </xacro:unless>
-    <xacro:arg name="gazebo" default="false"/>
-    <xacro:if value="$(arg gazebo)">
-        <gazebo>
-            <plugin filename="gz_ros2_control-system" name="gz_ros2_control::GazeboSimROS2ControlPlugin">
-                <xacro:if value="${'$(arg type)' == 'left'}">
-                    <parameters>$(find rokae_ar5_description)/config/ros2_control/ros2_controllers.yaml</parameters>
-                </xacro:if>
-                <xacro:if value="${'$(arg type)' == 'right'}">
-                    <parameters>$(find rokae_ar5_description)/config/ros2_control/right.yaml</parameters>
-                </xacro:if>
-                <xacro:if value="${'$(arg type)' == 'dual'}">
-                    <parameters>$(find rokae_ar5_description)/config/ros2_control/dual.yaml</parameters>
-                </xacro:if>
-            </plugin>
-        </gazebo>
-    </xacro:if>
+	<xacro:arg name="ros2_control_hardware_type" default="mock_components"/>
+	<link name="world"/>
+	<joint name="world_fixed" type="fixed">
+		<parent link="world"/>
+		<child link="base_link"/>
+		<origin/>
+	</joint>
+	<xacro:include filename="$(find rokae_ar5_description)/xacro/robot.xacro"/>
+	<xacro:include filename="$(find rokae_ar5_description)/xacro/ros2_control/interfaces.xacro"/>
+	<!-- 使用 robot.xacro 中已定义的 property 来判断 -->
+	<!-- selected_arm_config: left, right, dual -->
+	<!-- selected_gripper_type: '' 或 rg75 -->
+	<xacro:if value="${'$(arg ros2_control_hardware_type)' == 'real'}">
+		<xacro:if value="${selected_arm_config == 'dual'}">
+			<ros2_control name="ar5_left_system" type="system">
+				<hardware>
+					<plugin>rokae_ros2_control/RokaeHardware</plugin>
+					<param name="arm_ip">192.168.2.160</param>
+					<param name="joint_impedance">500,500,500,500,50,50,50</param>
+				</hardware>
+				<xacro:ar5_interfaces name="left"/>
+				<xacro:if value="${selected_gripper_type != ''}">
+					<joint name="left_gripper_joint">
+						<command_interface name="position"/>
+						<state_interface name="position">
+							<param name="initial_value">0</param>
+						</state_interface>
+					</joint>
+				</xacro:if>
+			</ros2_control>
+			<ros2_control name="ar5_right_system" type="system">
+				<hardware>
+					<plugin>rokae_ros2_control/RokaeHardware</plugin>
+					<param name="arm_ip">192.168.2.161</param>
+					<param name="joint_impedance">500,500,500,500,50,50,50</param>
+				</hardware>
+				<xacro:ar5_interfaces name="right"/>
+				<xacro:if value="${selected_gripper_type != ''}">
+					<joint name="right_gripper_joint">
+						<command_interface name="position"/>
+						<state_interface name="position">
+							<param name="initial_value">0</param>
+						</state_interface>
+					</joint>
+				</xacro:if>
+			</ros2_control>
+		</xacro:if>
+		<xacro:unless value="${selected_arm_config == 'dual'}">
+			<ros2_control name="ar5System" type="system">
+				<hardware>
+					<plugin>rokae_ros2_control/RokaeHardware</plugin>
+					<!-- 根据 arm_config 设置 arm_ip -->
+					<xacro:if value="${selected_arm_config == 'left'}">
+						<param name="arm_ip">192.168.2.160</param>
+					</xacro:if>
+					<xacro:if value="${selected_arm_config == 'right'}">
+						<param name="arm_ip">192.168.2.161</param>
+					</xacro:if>
+					<param name="local_ip">192.168.2.233</param>
+				</hardware>
+				<xacro:ar5_interfaces name=""/>
+				<xacro:if value="${selected_gripper_type != ''}">
+					<joint name="gripper_joint">
+						<command_interface name="position"/>
+						<state_interface name="position">
+							<param name="initial_value">0</param>
+						</state_interface>
+					</joint>
+				</xacro:if>
+			</ros2_control>
+		</xacro:unless>
+	</xacro:if>
+	<xacro:unless value="${'$(arg ros2_control_hardware_type)' == 'real'}">
+		<ros2_control name="ar5System" type="system">
+			<hardware>
+				<xacro:if value="${'$(arg ros2_control_hardware_type)' == 'gz'}">
+					<plugin>gz_ros2_control/GazeboSimSystem</plugin>
+				</xacro:if>
+				<xacro:if value="${'$(arg ros2_control_hardware_type)' == 'mock_components'}">
+					<plugin>mock_components/GenericSystem</plugin>
+				</xacro:if>
+				<xacro:if value="${'$(arg ros2_control_hardware_type)' == 'isaac'}">
+					<plugin>topic_based_ros2_control/TopicBasedSystem</plugin>
+					<param name="joint_commands_topic">/isaac/joint_command</param>
+					<param name="joint_states_topic">/isaac/joint_states</param>
+					<param name="sum_wrapped_joint_states">false</param>
+					<param name="initialize_commands_from_state">true</param>
+				</xacro:if>
+			</hardware>
+			<xacro:if value="${selected_arm_config == 'dual'}">
+				<xacro:ar5_interfaces name="left"/>
+				<xacro:ar5_interfaces name="right"/>
+				<xacro:if value="${selected_gripper_type != ''}">
+					<joint name="left_gripper_joint">
+						<command_interface name="position"/>
+						<state_interface name="position">
+							<param name="initial_value">0</param>
+						</state_interface>
+					</joint>
+					<joint name="right_gripper_joint">
+						<command_interface name="position"/>
+						<state_interface name="position">
+							<param name="initial_value">0</param>
+						</state_interface>
+					</joint>
+				</xacro:if>
+			</xacro:if>
+			<xacro:unless value="${selected_arm_config == 'dual'}">
+				<xacro:ar5_interfaces name=""/>
+				<xacro:if value="${selected_gripper_type != ''}">
+					<joint name="gripper_joint">
+						<command_interface name="position"/>
+						<state_interface name="position">
+							<param name="initial_value">0</param>
+						</state_interface>
+					</joint>
+				</xacro:if>
+			</xacro:unless>
+		</ros2_control>
+	</xacro:unless>
+	<xacro:arg name="gazebo" default="false"/>
+	<xacro:if value="$(arg gazebo)">
+		<gazebo>
+			<plugin filename="gz_ros2_control-system" name="gz_ros2_control::GazeboSimROS2ControlPlugin">
+				<xacro:if value="${selected_arm_config == 'left'}">
+					<parameters>$(find rokae_ar5_description)/config/ros2_control/ros2_controllers.yaml</parameters>
+				</xacro:if>
+				<xacro:if value="${selected_arm_config == 'right'}">
+					<parameters>$(find rokae_ar5_description)/config/ros2_control/right.yaml</parameters>
+				</xacro:if>
+				<xacro:if value="${selected_arm_config == 'dual'}">
+					<parameters>$(find rokae_ar5_description)/config/ros2_control/dual.yaml</parameters>
+				</xacro:if>
+			</plugin>
+		</gazebo>
+	</xacro:if>
 </robot>
