Commit message: fix rokae urdf

File: rokae_ar5_description/urdf/rokae_ar5.urdf (robot description, URDF)
Before this commit: robot DobotCR5, 8 links, 7 joints
Joints:
- joint joint1: origin xyz=0.0 0.0 0.1745 rpy=0 0 1.5708 -> xyz=0.0 0.0 0.1745 rpy=0 0 -3.14159

File: rokae_ar5_description/urdf/rokae_ar5_right.urdf (robot description, URDF)
Before this commit: robot DobotCR5, 8 links, 7 joints
Joints:
- joint joint1: origin xyz=0.0 0.0 0.1745 rpy=0 0 -1.5708 -> xyz=0.0 0.0 0.1745 rpy=0 0 -3.14159

File: rokae_ar5_description/xacro/arm.xacro (robot description, xacro)
@@ -28,5 +28,5 @@
 			<limit effort="108" lower="-3.1414" upper="3.1414" velocity="3.9269908169872414"/>
 			<axis xyz="0 0 1"/>
-			<origin xyz="0.0 0.0 0.1745" rpy="0 0 ${direction*1.5708}"/>
+			<origin xyz="0.0 0.0 0.1745" rpy="0 0 -3.14159"/>
 		</joint>
 		<!-- Arm Link 1 -->

File: rokae_ar5_description/xacro/ros2_control/robot.xacro (robot description, xacro)
@@ -27,5 +27,10 @@
       <xacro:if value="${'$(arg ros2_control_hardware_type)' == 'real'}">
         <plugin>rokae_ros2_control/RokaeHardware</plugin>
-        <param name="arm_ip">192.168.2.160</param>
+        <xacro:if value="${'$(arg type)' == 'left'}">
+          <param name="arm_ip">192.168.2.160</param>
+        </xacro:if>
+        <xacro:if value="${'$(arg type)' == 'right'}">
+          <param name="arm_ip">192.168.2.161</param>
+        </xacro:if>
       </xacro:if>
     </hardware>

Commit message: config for impedence control

File: rokae_ar5_description/urdf/rokae_ar5.urdf (robot description, URDF)
Before this commit: robot DobotCR5, 8 links, 7 joints
Joints:
- joint joint1: limit lower=-3.1414 upper=3.1414 effort=108 velocity=3.9269908169872414 -> lower=-3.14 upper=3.14 effort=108 velocity=3.9269908169872414
- joint joint2: limit lower=-2.1293 upper=2.1293 effort=108 velocity=3.9269908169872414 -> lower=-2.12 upper=2.12 effort=108 velocity=3.9269908169872414
- joint joint3: limit lower=-3.1416 upper=3.1416 effort=66 velocity=5.235987755982989 -> lower=-3.14 upper=3.14 effort=66 velocity=5.235987755982989
- joint joint4: limit lower=-1.3963 upper=2.5307 effort=66 velocity=5.235987755982989 -> lower=-1.39 upper=2.50 effort=66 velocity=5.235987755982989
- joint joint5: limit lower=-3.1416 upper=3.1416 effort=19 velocity=4.1887902047863905 -> lower=-3.14 upper=3.14 effort=19 velocity=4.1887902047863905
- joint joint6: limit lower=-1.9722 upper=1.9722 effort=19 velocity=4.1887902047863905 -> lower=-1.96 upper=1.96 effort=19 velocity=4.1887902047863905
- joint joint7: limit lower=-3.1416 upper=3.1416 effort=19 velocity=4.1887902047863905 -> lower=-3.14 upper=3.14 effort=19 velocity=4.1887902047863905

File: rokae_ar5_description/xacro/arm.xacro (robot description, xacro)
@@ -26,5 +26,5 @@
 			<parent link="${prefix}base_link"/>
 			<child link="${prefix}link1"/>
-			<limit effort="108" lower="-3.1414" upper="3.1414" velocity="3.9269908169872414"/>
+			<limit effort="108" lower="-3.14" upper="3.14" velocity="3.9269908169872414"/>
 			<axis xyz="0 0 1"/>
 			<origin xyz="0.0 0.0 0.1745" rpy="0 0 -3.14159"/>
@@ -52,5 +52,5 @@
 			<parent link="${prefix}link1"/>
 			<child link="${prefix}link2"/>
-			<limit effort="108" lower="-2.1293" upper="2.1293" velocity="3.9269908169872414"/>
+			<limit effort="108" lower="-2.12" upper="2.12" velocity="3.9269908169872414"/>
 			<axis xyz="0 -1 0"/>
 		</joint>
@@ -78,5 +78,5 @@
 			<parent link="${prefix}link2"/>
 			<child link="${prefix}link3"/>
-			<limit effort="66" lower="-3.1416" upper="3.1416" velocity="5.235987755982989"/>
+			<limit effort="66" lower="-3.14" upper="3.14" velocity="5.235987755982989"/>
 			<axis xyz="0 0 1"/>
 			<origin xyz="0.0 0.0 0.305" rpy="0 0 3.1415926535"/>
@@ -104,5 +104,5 @@
 			<parent link="${prefix}link3"/>
 			<child link="${prefix}link4"/>
-			<limit effort="66" lower="-1.3963" upper="2.5307" velocity="5.235987755982989"/>
+			<limit effort="66" lower="-1.39" upper="2.50" velocity="5.235987755982989"/>
 			<axis xyz="0 1 0"/>
 			<origin xyz="0.01 0.0 0.0"/>
@@ -131,5 +131,5 @@
 			<parent link="${prefix}link4"/>
 			<child link="${prefix}link5"/>
-			<limit effort="19" lower="-3.1416" upper="3.1416" velocity="4.1887902047863905"/>
+			<limit effort="19" lower="-3.14" upper="3.14" velocity="4.1887902047863905"/>
 			<axis xyz="0 0 1"/>
 			<origin xyz="-0.01 0.0 0.179"/>
@@ -157,5 +157,5 @@
 			<parent link="${prefix}link5"/>
 			<child link="${prefix}link6"/>
-			<limit effort="19" lower="-1.9722" upper="1.9722" velocity="4.1887902047863905"/>
+			<limit effort="19" lower="-1.96" upper="1.96" velocity="4.1887902047863905"/>
 			<axis xyz="0 1 0"/>
 		</joint>
@@ -183,5 +183,5 @@
 			<parent link="${prefix}link6"/>
 			<child link="${prefix}link7"/>
-			<limit effort="19" lower="-3.1416" upper="3.1416" velocity="4.1887902047863905"/>
+			<limit effort="19" lower="-3.14" upper="3.14" velocity="4.1887902047863905"/>
 			<axis xyz="0 0 1"/>
 			<origin xyz="0.0 0.0 0.166"/>

File: rokae_ar5_description/xacro/ros2_control/robot.xacro (robot description, xacro)
@@ -33,4 +33,6 @@
           <param name="arm_ip">192.168.2.161</param>
         </xacro:if>
+        <param name="joint_impedance">200,200,200,200,100,100,100</param>
+        <param name="rt_network_tolerance">20</param>
       </xacro:if>
     </hardware>

Commit message: dual config with rg 75

File: rokae_ar5_description/urdf/rokae_ar5.urdf (robot description, URDF)
Before this commit: robot DobotCR5, 8 links, 7 joints
Links:
- link base_link: geometry collision cylinder length=0.105 radius=0.045; visual mesh filename=package://rokae_ar5_description/meshes/base.obj scale=1 1 1
- link link1: geometry collision cylinder length=0.1354 radius=0.0560; visual mesh filename=package://rokae_ar5_description/meshes/link1.obj scale=1 1 1
- link link2: geometry collision cylinder length=0.11413 radius=0.053; visual mesh filename=package://rokae_ar5_description/meshes/link2.obj scale=1 1 1
- link link3: geometry collision cylinder length=0.096 radius=0.053; collision cylinder length=0.1284 radius=0.0484
- link link4: geometry collision cylinder length=0.10 radius=0.03789; visual mesh filename=package://rokae_ar5_description/meshes/link4.obj scale=1 1 1
- link link5: geometry collision cylinder length=0.107 radius=0.0383; visual mesh filename=package://rokae_ar5_description/meshes/link5.obj scale=1 1 1
- link link6: geometry collision cylinder length=0.1238 radius=0.04; visual mesh filename=package://rokae_ar5_description/meshes/link6.obj scale=1 1 1
- link link7: geometry visual mesh filename=package://rokae_ar5_description/meshes/link7.obj scale=1 1 1

File: rokae_ar5_description/urdf/rokae_ar5_dual.urdf (robot description, URDF)
Before this commit: robot RokaeAR5, 18 links, 17 joints
Links:
- added link left_eef
- added link right_eef
- link right_link7: geometry visual mesh filename=package://rokae_ar5_description/meshes/link7.obj scale=1 -1 1
Joints:
- added joint left_eef_joint: type fixed, parent left_link7, child left_eef
- added joint right_eef_joint: type fixed, parent right_link7, child right_eef

File: rokae_ar5_description/xacro/arm.xacro (robot description, xacro)
@@ -275,9 +275,4 @@
 				</geometry>
 			</visual>
-			<collision>
-				<geometry>
-					<mesh filename="file://$(find rokae_ar5_description)/meshes/link7.obj" scale="1 ${direction} 1"/>
-				</geometry>
-			</collision>
 		</link>
 	</xacro:macro>

File: rokae_ar5_description/xacro/robot.xacro (robot description, xacro)
@@ -30,5 +30,5 @@
     </joint>
   </xacro:if>
-  <xacro:if value="${'$(arg type)' == 'dual'}">
+  <xacro:if value="${'$(arg type)' == 'dual' or '$(arg type)' == 'dual_rg75'}">
     <link name="base_link"/>
     <link name="arm_base">
@@ -56,4 +56,19 @@
     <xacro:Arm name="left" collider="$(arg collider)" direction="1"/>
     <xacro:Arm name="right" collider="$(arg collider)" direction="-1"/>
+    <xacro:if value="${'$(arg type)' == 'dual_rg75'}">
+      <xacro:include filename="$(find jodell_description)/xacro/RG75-300.xacro"/>
+      <xacro:RG75-300 name="left" use_flange="true"/>
+      <xacro:RG75-300 name="right" use_flange="true"/>
+      <joint name="left_gripper_base_joint" type="fixed">
+        <origin xyz="0 0 -0.0045"/>
+        <parent link="left_link7"/>
+        <child link="left_flange"/>
+      </joint>
+      <joint name="right_gripper_base_joint" type="fixed">
+        <origin xyz="0 0 -0.0045"/>
+        <parent link="right_link7"/>
+        <child link="right_flange"/>
+      </joint>
+    </xacro:if>
   </xacro:if>
 </robot>

File: rokae_ar5_description/xacro/ros2_control/robot.xacro (robot description, xacro)
@@ -1,104 +1,120 @@
 <?xml version="1.0"?>
 <robot xmlns:xacro="http://www.ros.org/wiki/xacro" name="AR5">
-	<xacro:arg name="ros2_control_hardware_type" default="mock_components"/>
-	<link name="world"/>
-	<joint name="world_fixed" type="fixed">
-		<parent link="world"/>
-		<child link="base_link"/>
-		<origin/>
-	</joint>
-	<xacro:include filename="$(find rokae_ar5_description)/xacro/robot.xacro"/>
-	<xacro:include filename="$(find rokae_ar5_description)/xacro/ros2_control/interfaces.xacro"/>
-	<xacro:if value="${'$(arg ros2_control_hardware_type)' == 'real'}">
-		<xacro:if value="${'$(arg type)' == 'dual'}">
-			<ros2_control name="ar5_left_system" type="system">
-				<hardware>
-					<plugin>rokae_ros2_control/RokaeHardware</plugin>
-					<param name="arm_ip">192.168.2.160</param>
-					<param name="joint_impedance">500,500,500,500,50,50,50</param>
-				</hardware>
-				<xacro:ar5_interfaces name="left"/>
-			</ros2_control>
-			<ros2_control name="ar5_right_system" type="system">
-				<hardware>
-					<plugin>rokae_ros2_control/RokaeHardware</plugin>
-					<param name="arm_ip">192.168.2.161</param>
-					<param name="joint_impedance">500,500,500,500,50,50,50</param>
-				</hardware>
-				<xacro:ar5_interfaces name="right"/>
-			</ros2_control>
-		</xacro:if>
-		<xacro:unless value="${'$(arg type)' == 'dual'}">
-			<ros2_control name="ar5System" type="system">
-				<hardware>
-					<plugin>rokae_ros2_control/RokaeHardware</plugin>
-					<xacro:if value="${'$(arg type)' == 'left'}">
-						<param name="arm_ip">192.168.2.160</param>
-					</xacro:if>
-					<xacro:if value="${'$(arg type)' == 'left_rg75'}">
-						<param name="arm_ip">192.168.2.160</param>
-					</xacro:if>
-					<xacro:if value="${'$(arg type)' == 'right'}">
-						<param name="arm_ip">192.168.2.161</param>
-					</xacro:if>
-					<xacro:if value="${'$(arg type)' == 'right_rg75'}">
-						<param name="arm_ip">192.168.2.161</param>
-					</xacro:if>
-<!--					<param name="joint_impedance">200,200,200,200,100,100,100</param>-->
-					<param name="local_ip">192.168.2.233</param>
-				</hardware>
-				<xacro:ar5_interfaces name=""/>
-				<xacro:if value="${'$(arg type)' != 'left' and '$(arg type)' != 'right'}">
-					<joint name="gripper_joint">
-						<command_interface name="position"/>
-						<state_interface name="position">
-							<param name="initial_value">0</param>
-						</state_interface>
-					</joint>
-				</xacro:if>
-			</ros2_control>
-		</xacro:unless>
-	</xacro:if>
-	<xacro:unless value="${'$(arg ros2_control_hardware_type)' == 'real'}">
-		<ros2_control name="ar5System" type="system">
-			<hardware>
-				<xacro:if value="${'$(arg ros2_control_hardware_type)' == 'gz'}">
-					<plugin>gz_ros2_control/GazeboSimSystem</plugin>
-				</xacro:if>
-				<xacro:if value="${'$(arg ros2_control_hardware_type)' == 'mock_components'}">
-					<plugin>mock_components/GenericSystem</plugin>
-				</xacro:if>
-				<xacro:if value="${'$(arg ros2_control_hardware_type)' == 'isaac'}">
-					<plugin>topic_based_ros2_control/TopicBasedSystem</plugin>
-					<param name="joint_commands_topic">/isaac/joint_command</param>
-					<param name="joint_states_topic">/isaac/joint_states</param>
-					<param name="sum_wrapped_joint_states">false</param>
-					<param name="initialize_commands_from_state">true</param>
-				</xacro:if>
-			</hardware>
-			<xacro:if value="${'$(arg type)' == 'dual'}">
-				<xacro:ar5_interfaces name="left"/>
-				<xacro:ar5_interfaces name="right"/>
-			</xacro:if>
-			<xacro:unless value="${'$(arg type)' == 'dual'}">
-				<xacro:ar5_interfaces name=""/>
-			</xacro:unless>
-		</ros2_control>
-	</xacro:unless>
-	<xacro:arg name="gazebo" default="false"/>
-	<xacro:if value="$(arg gazebo)">
-		<gazebo>
-			<plugin filename="gz_ros2_control-system" name="gz_ros2_control::GazeboSimROS2ControlPlugin">
-				<xacro:if value="${'$(arg type)' == 'left'}">
-					<parameters>$(find rokae_ar5_description)/config/ros2_control/ros2_controllers.yaml</parameters>
-				</xacro:if>
-				<xacro:if value="${'$(arg type)' == 'right'}">
-					<parameters>$(find rokae_ar5_description)/config/ros2_control/right.yaml</parameters>
-				</xacro:if>
-				<xacro:if value="${'$(arg type)' == 'dual'}">
-					<parameters>$(find rokae_ar5_description)/config/ros2_control/dual.yaml</parameters>
-				</xacro:if>
-			</plugin>
-		</gazebo>
-	</xacro:if>
+    <xacro:arg name="ros2_control_hardware_type" default="mock_components"/>
+    <link name="world"/>
+    <joint name="world_fixed" type="fixed">
+        <parent link="world"/>
+        <child link="base_link"/>
+        <origin/>
+    </joint>
+    <xacro:include filename="$(find rokae_ar5_description)/xacro/robot.xacro"/>
+    <xacro:include filename="$(find rokae_ar5_description)/xacro/ros2_control/interfaces.xacro"/>
+    <xacro:if value="${'$(arg ros2_control_hardware_type)' == 'real'}">
+        <xacro:if value="${'$(arg type)' == 'dual' or '$(arg type)' == 'dual_rg75' }">
+            <ros2_control name="ar5_left_system" type="system">
+                <hardware>
+                    <plugin>rokae_ros2_control/RokaeHardware</plugin>
+                    <param name="arm_ip">192.168.2.160</param>
+                    <param name="joint_impedance">500,500,500,500,50,50,50</param>
+                </hardware>
+                <xacro:ar5_interfaces name="left"/>
+                <xacro:if value="${'$(arg type)' != 'dual'}">
+                    <joint name="left_gripper_joint">
+                        <command_interface name="position"/>
+                        <state_interface name="position">
+                            <param name="initial_value">0</param>
+                        </state_interface>
+                    </joint>
+                </xacro:if>
+            </ros2_control>
+            <ros2_control name="ar5_right_system" type="system">
+                <hardware>
+                    <plugin>rokae_ros2_control/RokaeHardware</plugin>
+                    <param name="arm_ip">192.168.2.161</param>
+                    <param name="joint_impedance">500,500,500,500,50,50,50</param>
+                </hardware>
+                <xacro:ar5_interfaces name="right"/>
+                <xacro:if value="${'$(arg type)' != 'dual'}">
+                    <joint name="right_gripper_joint">
+                        <command_interface name="position"/>
+                        <state_interface name="position">
+                            <param name="initial_value">0</param>
+                        </state_interface>
+                    </joint>
+                </xacro:if>
+            </ros2_control>
+        </xacro:if>
+        <xacro:unless value="${'$(arg type)' == 'dual' or '$(arg type)' == 'dual_rg75'}">
+            <ros2_control name="ar5System" type="system">
+                <hardware>
+                    <plugin>rokae_ros2_control/RokaeHardware</plugin>
+                    <xacro:if value="${'$(arg type)' == 'left'}">
+                        <param name="arm_ip">192.168.2.160</param>
+                    </xacro:if>
+                    <xacro:if value="${'$(arg type)' == 'left_rg75'}">
+                        <param name="arm_ip">192.168.2.160</param>
+                    </xacro:if>
+                    <xacro:if value="${'$(arg type)' == 'right'}">
+                        <param name="arm_ip">192.168.2.161</param>
+                    </xacro:if>
+                    <xacro:if value="${'$(arg type)' == 'right_rg75'}">
+                        <param name="arm_ip">192.168.2.161</param>
+                    </xacro:if>
+                    <!--					<param name="joint_impedance">200,200,200,200,100,100,100</param>-->
+                    <param name="local_ip">192.168.2.233</param>
+                </hardware>
+                <xacro:ar5_interfaces name=""/>
+                <xacro:if value="${'$(arg type)' != 'left' and '$(arg type)' != 'right'}">
+                    <joint name="gripper_joint">
+                        <command_interface name="position"/>
+                        <state_interface name="position">
+                            <param name="initial_value">0</param>
+                        </state_interface>
+                    </joint>
+                </xacro:if>
+            </ros2_control>
+        </xacro:unless>
+    </xacro:if>
+    <xacro:unless value="${'$(arg ros2_control_hardware_type)' == 'real'}">
+        <ros2_control name="ar5System" type="system">
+            <hardware>
+                <xacro:if value="${'$(arg ros2_control_hardware_type)' == 'gz'}">
+                    <plugin>gz_ros2_control/GazeboSimSystem</plugin>
+                </xacro:if>
+                <xacro:if value="${'$(arg ros2_control_hardware_type)' == 'mock_components'}">
+                    <plugin>mock_components/GenericSystem</plugin>
+                </xacro:if>
+                <xacro:if value="${'$(arg ros2_control_hardware_type)' == 'isaac'}">
+                    <plugin>topic_based_ros2_control/TopicBasedSystem</plugin>
+                    <param name="joint_commands_topic">/isaac/joint_command</param>
+                    <param name="joint_states_topic">/isaac/joint_states</param>
+                    <param name="sum_wrapped_joint_states">false</param>
+                    <param name="initialize_commands_from_state">true</param>
+                </xacro:if>
+            </hardware>
+            <xacro:if value="${'$(arg type)' == 'dual'}">
+                <xacro:ar5_interfaces name="left"/>
+                <xacro:ar5_interfaces name="right"/>
+            </xacro:if>
+            <xacro:unless value="${'$(arg type)' == 'dual'}">
+                <xacro:ar5_interfaces name=""/>
+            </xacro:unless>
+        </ros2_control>
+    </xacro:unless>
+    <xacro:arg name="gazebo" default="false"/>
+    <xacro:if value="$(arg gazebo)">
+        <gazebo>
+            <plugin filename="gz_ros2_control-system" name="gz_ros2_control::GazeboSimROS2ControlPlugin">
+                <xacro:if value="${'$(arg type)' == 'left'}">
+                    <parameters>$(find rokae_ar5_description)/config/ros2_control/ros2_controllers.yaml</parameters>
+                </xacro:if>
+                <xacro:if value="${'$(arg type)' == 'right'}">
+                    <parameters>$(find rokae_ar5_description)/config/ros2_control/right.yaml</parameters>
+                </xacro:if>
+                <xacro:if value="${'$(arg type)' == 'dual'}">
+                    <parameters>$(find rokae_ar5_description)/config/ros2_control/dual.yaml</parameters>
+                </xacro:if>
+            </plugin>
+        </gazebo>
+    </xacro:if>
 </robot>
