Commit message: ccs left ocs2 arm controller config

File: rokae_ar5_description/urdf/rokae_ar5.urdf (robot description, URDF)
Before this commit: robot RokaeAR5, 8 links, 7 joints
Links:
- link base_link: geometry collision cylinder length=0.105 radius=0.045; visual mesh filename=package://rokae_ar5_description/meshes/srs/base.obj scale=1 1 1
- link link1: geometry collision cylinder length=0.1354 radius=0.0560; visual mesh filename=package://rokae_ar5_description/meshes/srs/link1.obj scale=1 1 1
- link link2: geometry collision cylinder length=0.11413 radius=0.053; visual mesh filename=package://rokae_ar5_description/meshes/srs/link2.obj scale=1 1 1
- link link3: geometry collision cylinder length=0.096 radius=0.053; collision cylinder length=0.1284 radius=0.0484
- link link4: geometry collision cylinder length=0.10 radius=0.03789; visual mesh filename=package://rokae_ar5_description/meshes/srs/link4.obj scale=1 1 1
- link link5: geometry collision cylinder length=0.107 radius=0.0383; visual mesh filename=package://rokae_ar5_description/meshes/srs/link5.obj scale=1 1 1
- link link6: geometry collision cylinder length=0.1238 radius=0.04; visual mesh filename=package://rokae_ar5_description/meshes/srs/link6.obj scale=1 1 1
- link link7: geometry visual mesh filename=package://rokae_ar5_description/meshes/srs/link7.obj scale=1 1 1

File: rokae_ar5_description/urdf/rokae_ar5_dual.urdf (robot description, URDF)
Before this commit: robot RokaeAR5, 20 links, 19 joints
Links:
- link left_base_link: geometry collision cylinder length=0.105 radius=0.045; visual mesh filename=package://rokae_ar5_description/meshes/srs/base.obj scale=1 1 1
- link left_link1: geometry collision cylinder length=0.1354 radius=0.0560; visual mesh filename=package://rokae_ar5_description/meshes/srs/link1.obj scale=1 1 1
- link left_link2: geometry collision cylinder length=0.11413 radius=0.053; visual mesh filename=package://rokae_ar5_description/meshes/srs/link2.obj scale=1 1 1
- link left_link3: geometry collision cylinder length=0.096 radius=0.053; collision cylinder length=0.1284 radius=0.0484
- link left_link4: geometry collision cylinder length=0.10 radius=0.03789; visual mesh filename=package://rokae_ar5_description/meshes/srs/link4.obj scale=1 1 1
- link left_link5: geometry collision cylinder length=0.107 radius=0.0383; visual mesh filename=package://rokae_ar5_description/meshes/srs/link5.obj scale=1 1 1
- link left_link6: geometry collision cylinder length=0.1238 radius=0.04; visual mesh filename=package://rokae_ar5_description/meshes/srs/link6.obj scale=1 1 1
- link left_link7: geometry collision mesh filename=package://rokae_ar5_description/meshes/srs/link7.obj scale=1 1 1; visual mesh filename=package://rokae_ar5_description/meshes/srs/link7.obj scale=1 1 1
- link right_base_link: geometry collision cylinder length=0.105 radius=0.045; visual mesh filename=package://rokae_ar5_description/meshes/srs/base.obj scale=1 -1 1
- link right_link1: geometry collision cylinder length=0.1354 radius=0.0560; visual mesh filename=package://rokae_ar5_description/meshes/srs/link1.obj scale=1 -1 1
- link right_link2: geometry collision cylinder length=0.11413 radius=0.053; visual mesh filename=package://rokae_ar5_description/meshes/srs/link2.obj scale=1 -1 1
- link right_link3: geometry collision cylinder length=0.096 radius=0.053; collision cylinder length=0.1284 radius=0.0484
- link right_link4: geometry collision cylinder length=0.10 radius=0.03789; visual mesh filename=package://rokae_ar5_description/meshes/srs/link4.obj scale=1 -1 1
- link right_link5: geometry collision cylinder length=0.107 radius=0.0383; visual mesh filename=package://rokae_ar5_description/meshes/srs/link5.obj scale=1 -1 1
- link right_link6: geometry collision cylinder length=0.1238 radius=0.04; visual mesh filename=package://rokae_ar5_description/meshes/srs/link6.obj scale=1 -1 1
- link right_link7: geometry visual mesh filename=package://rokae_ar5_description/meshes/srs/link7.obj scale=1 -1 1

File: rokae_ar5_description/urdf/rokae_ar5_dual_rg75.urdf (robot description, URDF)
Before this commit: robot RokaeAR5, 32 links, 31 joints
Links:
- link left_base_link: geometry collision cylinder length=0.105 radius=0.045; visual mesh filename=package://rokae_ar5_description/meshes/srs/base.obj scale=1 1 1
- link left_flange: geometry collision mesh filename=package://jodell_description/meshes/srs/RG75/flange.obj; visual mesh filename=package://jodell_description/meshes/srs/RG75/flange.obj
- link left_gripper_base: geometry collision mesh filename=package://jodell_description/meshes/srs/RG75/base.obj; visual mesh filename=package://jodell_description/meshes/srs/RG75/base.obj
- link left_left_finger: geometry collision mesh filename=package://jodell_description/meshes/srs/RG75/finger.obj; visual mesh filename=package://jodell_description/meshes/srs/RG75/finger.obj
- link left_left_finger_pad: geometry collision mesh filename=package://jodell_description/meshes/srs/RG75/pad_fiveages.o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; visual mesh filename=package://jodell_description/meshes/srs/RG75/pad_fiveages.o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
- link left_link1: geometry collision cylinder length=0.1354 radius=0.0560; visual mesh filename=package://rokae_ar5_description/meshes/srs/link1.obj scale=1 1 1
- link left_link2: geometry collision cylinder length=0.11413 radius=0.053; visual mesh filename=package://rokae_ar5_description/meshes/srs/link2.obj scale=1 1 1
- link left_link3: geometry collision cylinder length=0.096 radius=0.053; collision cylinder length=0.1284 radius=0.0484
- link left_link4: geometry collision cylinder length=0.10 radius=0.03789; visual mesh filename=package://rokae_ar5_description/meshes/srs/link4.obj scale=1 1 1
- link left_link5: geometry collision cylinder length=0.107 radius=0.0383; visual mesh filename=package://rokae_ar5_description/meshes/srs/link5.obj scale=1 1 1
- link left_link6: geometry collision cylinder length=0.1238 radius=0.04; visual mesh filename=package://rokae_ar5_description/meshes/srs/link6.obj scale=1 1 1
- link left_link7: geometry visual mesh filename=package://rokae_ar5_description/meshes/srs/link7.obj scale=1 1 1
- link left_right_finger: geometry collision mesh filename=package://jodell_description/meshes/srs/RG75/finger.obj scale=-1 -1 1; visual mesh filename=package://jodell_description/meshes/srs/RG75/finger.obj scale=-1 -1 1
- link left_right_finger_pad: geometry collision mesh filename=package://jodell_description/meshes/srs/RG75/pad_fiveages.o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 scale=1 -1 1; visual mesh filename=package://jodell_description/meshes/srs/RG75/pad_fiveages.o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 scale=1 -1 1
- link right_base_link: geometry collision cylinder length=0.105 radius=0.045; visual mesh filename=package://rokae_ar5_description/meshes/srs/base.obj scale=1 -1 1
- link right_flange: geometry collision mesh filename=package://jodell_description/meshes/srs/RG75/flange.obj; visual mesh filename=package://jodell_description/meshes/srs/RG75/flange.obj
- link right_gripper_base: geometry collision mesh filename=package://jodell_description/meshes/srs/RG75/base.obj; visual mesh filename=package://jodell_description/meshes/srs/RG75/base.obj
- link right_left_finger: geometry collision mesh filename=package://jodell_description/meshes/srs/RG75/finger.obj; visual mesh filename=package://jodell_description/meshes/srs/RG75/finger.obj
- link right_left_finger_pad: geometry collision mesh filename=package://jodell_description/meshes/srs/RG75/pad_fiveages.o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; visual mesh filename=package://jodell_description/meshes/srs/RG75/pad_fiveages.o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
- link right_link1: geometry collision cylinder length=0.1354 radius=0.0560; visual mesh filename=package://rokae_ar5_description/meshes/srs/link1.obj scale=1 -1 1
- link right_link2: geometry collision cylinder length=0.11413 radius=0.053; visual mesh filename=package://rokae_ar5_description/meshes/srs/link2.obj scale=1 -1 1
- link right_link3: geometry collision cylinder length=0.096 radius=0.053; collision cylinder length=0.1284 radius=0.0484
- link right_link4: geometry collision cylinder length=0.10 radius=0.03789; visual mesh filename=package://rokae_ar5_description/meshes/srs/link4.obj scale=1 -1 1
- link right_link5: geometry collision cylinder length=0.107 radius=0.0383; visual mesh filename=package://rokae_ar5_description/meshes/srs/link5.obj scale=1 -1 1
- link right_link6: geometry collision cylinder length=0.1238 radius=0.04; visual mesh filename=package://rokae_ar5_description/meshes/srs/link6.obj scale=1 -1 1
- link right_link7: geometry visual mesh filename=package://rokae_ar5_description/meshes/srs/link7.obj scale=1 -1 1
- link right_right_finger: geometry collision mesh filename=package://jodell_description/meshes/srs/RG75/finger.obj scale=-1 -1 1; visual mesh filename=package://jodell_description/meshes/srs/RG75/finger.obj scale=-1 -1 1
- link right_right_finger_pad: geometry collision mesh filename=package://jodell_description/meshes/srs/RG75/pad_fiveages.o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 scale=1 -1 1; visual mesh filename=package://jodell_description/meshes/srs/RG75/pad_fiveages.o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 scale=1 -1 1
