Commit message: update mesh to glb

File: rokae_ar5_description/urdf/rokae_ar5.urdf (robot description, URDF)
Before this commit: robot RokaeAR5, 8 links, 7 joints
Links:
- link base_link: geometry collision cylinder length=0.105 radius=0.045; visual mesh filename=package://rokae_ar5_description/meshes/srs/base.glb scale=1 1 1
- link link1: geometry collision cylinder length=0.1354 radius=0.0560; visual mesh filename=package://rokae_ar5_description/meshes/srs/link1.glb scale=1 1 1
- link link2: geometry collision cylinder length=0.11413 radius=0.053; visual mesh filename=package://rokae_ar5_description/meshes/srs/link2.glb scale=1 1 1
- link link3: geometry collision cylinder length=0.096 radius=0.053; collision cylinder length=0.1284 radius=0.0484
- link link4: geometry collision cylinder length=0.10 radius=0.03789; visual mesh filename=package://rokae_ar5_description/meshes/srs/link4.glb scale=1 1 1
- link link5: geometry collision cylinder length=0.107 radius=0.0383; visual mesh filename=package://rokae_ar5_description/meshes/srs/link5.glb scale=1 1 1
- link link6: geometry collision cylinder length=0.1238 radius=0.04; visual mesh filename=package://rokae_ar5_description/meshes/srs/link6.glb scale=1 1 1
- link link7: geometry visual mesh filename=package://rokae_ar5_description/meshes/srs/link7.glb scale=1 1 1

File: rokae_ar5_description/urdf/rokae_ar5_ccs_left.urdf (robot description, URDF)
Before this commit: robot RokaeAR5, 9 links, 8 joints
Links:
- link base_link: geometry collision mesh filename=package://rokae_ar5_description/meshes/ccs/base.glb; visual mesh filename=package://rokae_ar5_description/meshes/ccs/base.glb
- link link1: geometry collision mesh filename=package://rokae_ar5_description/meshes/ccs/link1.glb scale=1 1 1; visual mesh filename=package://rokae_ar5_description/meshes/ccs/link1.glb scale=1 1 1
- link link2: geometry collision mesh filename=package://rokae_ar5_description/meshes/ccs/link2.glb scale=1 1 1; visual mesh filename=package://rokae_ar5_description/meshes/ccs/link2.glb scale=1 1 1
- link link3: geometry collision mesh filename=package://rokae_ar5_description/meshes/ccs/link3.glb scale=1 1 1; visual mesh filename=package://rokae_ar5_description/meshes/ccs/link3.glb scale=1 1 1
- link link4: geometry collision mesh filename=package://rokae_ar5_description/meshes/ccs/link4.glb scale=1 1 1; visual mesh filename=package://rokae_ar5_description/meshes/ccs/link4.glb scale=1 1 1
- link link5: geometry collision mesh filename=package://rokae_ar5_description/meshes/ccs/link5.glb scale=1 1 1; visual mesh filename=package://rokae_ar5_description/meshes/ccs/link5.glb scale=1 1 1
- link link6: geometry collision mesh filename=package://rokae_ar5_description/meshes/ccs/link6.glb scale=1 1 1; visual mesh filename=package://rokae_ar5_description/meshes/ccs/link6.glb scale=1 1 1
- link link7: geometry collision mesh filename=package://rokae_ar5_description/meshes/ccs/link7.glb scale=1 1 1; visual mesh filename=package://rokae_ar5_description/meshes/ccs/link7.glb scale=1 1 1

File: rokae_ar5_description/urdf/rokae_ar5_ccs_right.urdf (robot description, URDF)
Before this commit: robot RokaeAR5, 9 links, 8 joints
Links:
- link base_link: geometry collision mesh filename=package://rokae_ar5_description/meshes/ccs/base.glb; visual mesh filename=package://rokae_ar5_description/meshes/ccs/base.glb
- link link1: geometry collision mesh filename=package://rokae_ar5_description/meshes/ccs/link1.glb scale=1 -1 1; visual mesh filename=package://rokae_ar5_description/meshes/ccs/link1.glb scale=1 -1 1
- link link2: geometry collision mesh filename=package://rokae_ar5_description/meshes/ccs/link2.glb scale=1 -1 1; visual mesh filename=package://rokae_ar5_description/meshes/ccs/link2.glb scale=1 -1 1
- link link3: geometry collision mesh filename=package://rokae_ar5_description/meshes/ccs/link3.glb scale=1 -1 1; visual mesh filename=package://rokae_ar5_description/meshes/ccs/link3.glb scale=1 -1 1
- link link4: geometry collision mesh filename=package://rokae_ar5_description/meshes/ccs/link4.glb scale=1 -1 1; visual mesh filename=package://rokae_ar5_description/meshes/ccs/link4.glb scale=1 -1 1
- link link5: geometry collision mesh filename=package://rokae_ar5_description/meshes/ccs/link5.glb scale=1 -1 1; visual mesh filename=package://rokae_ar5_description/meshes/ccs/link5.glb scale=1 -1 1
- link link6: geometry collision mesh filename=package://rokae_ar5_description/meshes/ccs/link6.glb scale=1 -1 1; visual mesh filename=package://rokae_ar5_description/meshes/ccs/link6.glb scale=1 -1 1
- link link7: geometry collision mesh filename=package://rokae_ar5_description/meshes/ccs/link7.glb scale=-1 1 1; visual mesh filename=package://rokae_ar5_description/meshes/ccs/link7.glb scale=-1 1 1

File: rokae_ar5_description/urdf/rokae_ar5_dual.urdf (robot description, URDF)
Before this commit: robot RokaeAR5, 20 links, 19 joints
Links:
- link left_base_link: geometry collision cylinder length=0.105 radius=0.045; visual mesh filename=package://rokae_ar5_description/meshes/srs/base.glb scale=1 1 1
- link left_link1: geometry collision cylinder length=0.1354 radius=0.0560; visual mesh filename=package://rokae_ar5_description/meshes/srs/link1.glb scale=1 1 1
- link left_link2: geometry collision cylinder length=0.11413 radius=0.053; visual mesh filename=package://rokae_ar5_description/meshes/srs/link2.glb scale=1 1 1
- link left_link3: geometry collision cylinder length=0.096 radius=0.053; collision cylinder length=0.1284 radius=0.0484
- link left_link4: geometry collision cylinder length=0.10 radius=0.03789; visual mesh filename=package://rokae_ar5_description/meshes/srs/link4.glb scale=1 1 1
- link left_link5: geometry collision cylinder length=0.107 radius=0.0383; visual mesh filename=package://rokae_ar5_description/meshes/srs/link5.glb scale=1 1 1
- link left_link6: geometry collision cylinder length=0.1238 radius=0.04; visual mesh filename=package://rokae_ar5_description/meshes/srs/link6.glb scale=1 1 1
- link left_link7: geometry collision mesh filename=package://rokae_ar5_description/meshes/srs/link7.glb scale=1 1 1; visual mesh filename=package://rokae_ar5_description/meshes/srs/link7.glb scale=1 1 1
- link right_base_link: geometry collision cylinder length=0.105 radius=0.045; visual mesh filename=package://rokae_ar5_description/meshes/srs/base.glb scale=1 -1 1
- link right_link1: geometry collision cylinder length=0.1354 radius=0.0560; visual mesh filename=package://rokae_ar5_description/meshes/srs/link1.glb scale=1 -1 1
- link right_link2: geometry collision cylinder length=0.11413 radius=0.053; visual mesh filename=package://rokae_ar5_description/meshes/srs/link2.glb scale=1 -1 1
- link right_link3: geometry collision cylinder length=0.096 radius=0.053; collision cylinder length=0.1284 radius=0.0484
- link right_link4: geometry collision cylinder length=0.10 radius=0.03789; visual mesh filename=package://rokae_ar5_description/meshes/srs/link4.glb scale=1 -1 1
- link right_link5: geometry collision cylinder length=0.107 radius=0.0383; visual mesh filename=package://rokae_ar5_description/meshes/srs/link5.glb scale=1 -1 1
- link right_link6: geometry collision cylinder length=0.1238 radius=0.04; visual mesh filename=package://rokae_ar5_description/meshes/srs/link6.glb scale=1 -1 1
- link right_link7: geometry visual mesh filename=package://rokae_ar5_description/meshes/srs/link7.glb scale=1 -1 1

File: rokae_ar5_description/urdf/rokae_ar5_dual_ccs.urdf (robot description, URDF)
Before this commit: robot RokaeAR5, 22 links, 21 joints
Links:
- link left_base_link: geometry collision cylinder length=0.105 radius=0.045; visual mesh filename=package://rokae_ar5_description/meshes/ccs/base.glb
- link left_link1: geometry visual mesh filename=package://rokae_ar5_description/meshes/ccs/link1.glb scale=1 1 1
- link left_link2: geometry collision cylinder length=0.12413 radius=0.053; collision cylinder length=0.1354 radius=0.0560
- link left_link3: geometry collision cylinder length=0.096 radius=0.053; collision cylinder length=0.1284 radius=0.0484
- link left_link4: geometry collision cylinder length=0.10 radius=0.03789; visual mesh filename=package://rokae_ar5_description/meshes/ccs/link4.glb scale=1 1 1
- link left_link5: geometry collision cylinder length=0.11 radius=0.042766; visual mesh filename=package://rokae_ar5_description/meshes/ccs/link5.glb scale=1 1 1
- link left_link6: geometry collision cylinder length=0.11772 radius=0.044145; visual mesh filename=package://rokae_ar5_description/meshes/ccs/link6.glb scale=1 1 1
- link left_link7: geometry collision cylinder length=0.038669 radius=0.03559; visual mesh filename=package://rokae_ar5_description/meshes/ccs/link7.glb scale=1 1 1
- link right_base_link: geometry collision cylinder length=0.105 radius=0.045; visual mesh filename=package://rokae_ar5_description/meshes/ccs/base.glb
- link right_link1: geometry visual mesh filename=package://rokae_ar5_description/meshes/ccs/link1.glb scale=1 -1 1
- link right_link2: geometry collision cylinder length=0.12413 radius=0.053; collision cylinder length=0.1354 radius=0.0560
- link right_link3: geometry collision cylinder length=0.096 radius=0.053; collision cylinder length=0.1284 radius=0.0484
- link right_link4: geometry collision cylinder length=0.10 radius=0.03789; visual mesh filename=package://rokae_ar5_description/meshes/ccs/link4.glb scale=1 -1 1
- link right_link5: geometry collision cylinder length=0.11 radius=0.042766; visual mesh filename=package://rokae_ar5_description/meshes/ccs/link5.glb scale=1 -1 1
- link right_link6: geometry collision cylinder length=0.11772 radius=0.044145; visual mesh filename=package://rokae_ar5_description/meshes/ccs/link6.glb scale=1 -1 1
- link right_link7: geometry collision cylinder length=0.038669 radius=0.03559; visual mesh filename=package://rokae_ar5_description/meshes/ccs/link7.glb scale=-1 1 1

File: rokae_ar5_description/urdf/rokae_ar5_dual_ccs_rg75.urdf (robot description, URDF)
Before this commit: robot RokaeAR5, 34 links, 33 joints
Links:
- link left_base_link: geometry collision cylinder length=0.105 radius=0.045; visual mesh filename=package://rokae_ar5_description/meshes/ccs/base.glb
- link left_flange: geometry collision mesh filename=package://jodell_description/meshes/RG75/flange.glb; visual mesh filename=package://jodell_description/meshes/RG75/flange.glb
- link left_gripper_base: geometry collision mesh filename=package://jodell_description/meshes/RG75/base.glb; visual mesh filename=package://jodell_description/meshes/RG75/base.glb
- link left_left_finger: geometry collision mesh filename=package://jodell_description/meshes/RG75/finger.glb; visual mesh filename=package://jodell_description/meshes/RG75/finger.glb
- link left_left_finger_pad: geometry collision mesh filename=package://jodell_description/meshes/RG75/pad_fiveages.glb; visual mesh filename=package://jodell_description/meshes/RG75/pad_fiveages.glb
- link left_link1: geometry visual mesh filename=package://rokae_ar5_description/meshes/ccs/link1.glb scale=1 1 1
- link left_link2: geometry collision cylinder length=0.12413 radius=0.053; collision cylinder length=0.1354 radius=0.0560
- link left_link3: geometry collision cylinder length=0.096 radius=0.053; collision cylinder length=0.1284 radius=0.0484
- link left_link4: geometry collision cylinder length=0.10 radius=0.03789; visual mesh filename=package://rokae_ar5_description/meshes/ccs/link4.glb scale=1 1 1
- link left_link5: geometry collision cylinder length=0.11 radius=0.042766; visual mesh filename=package://rokae_ar5_description/meshes/ccs/link5.glb scale=1 1 1
- link left_link6: geometry collision cylinder length=0.11772 radius=0.044145; visual mesh filename=package://rokae_ar5_description/meshes/ccs/link6.glb scale=1 1 1
- link left_link7: geometry collision cylinder length=0.038669 radius=0.03559; visual mesh filename=package://rokae_ar5_description/meshes/ccs/link7.glb scale=1 1 1
- link left_right_finger: geometry collision mesh filename=package://jodell_description/meshes/RG75/finger.glb scale=-1 -1 1; visual mesh filename=package://jodell_description/meshes/RG75/finger.glb scale=-1 -1 1
- link left_right_finger_pad: geometry collision mesh filename=package://jodell_description/meshes/RG75/pad_fiveages.glb scale=1 -1 1; visual mesh filename=package://jodell_description/meshes/RG75/pad_fiveages.glb scale=1 -1 1
- link right_base_link: geometry collision cylinder length=0.105 radius=0.045; visual mesh filename=package://rokae_ar5_description/meshes/ccs/base.glb
- link right_flange: geometry collision mesh filename=package://jodell_description/meshes/RG75/flange.glb; visual mesh filename=package://jodell_description/meshes/RG75/flange.glb
- link right_gripper_base: geometry collision mesh filename=package://jodell_description/meshes/RG75/base.glb; visual mesh filename=package://jodell_description/meshes/RG75/base.glb
- link right_left_finger: geometry collision mesh filename=package://jodell_description/meshes/RG75/finger.glb; visual mesh filename=package://jodell_description/meshes/RG75/finger.glb
- link right_left_finger_pad: geometry collision mesh filename=package://jodell_description/meshes/RG75/pad_fiveages.glb; visual mesh filename=package://jodell_description/meshes/RG75/pad_fiveages.glb
- link right_link1: geometry visual mesh filename=package://rokae_ar5_description/meshes/ccs/link1.glb scale=1 -1 1
- link right_link2: geometry collision cylinder length=0.12413 radius=0.053; collision cylinder length=0.1354 radius=0.0560
- link right_link3: geometry collision cylinder length=0.096 radius=0.053; collision cylinder length=0.1284 radius=0.0484
- link right_link4: geometry collision cylinder length=0.10 radius=0.03789; visual mesh filename=package://rokae_ar5_description/meshes/ccs/link4.glb scale=1 -1 1
- link right_link5: geometry collision cylinder length=0.11 radius=0.042766; visual mesh filename=package://rokae_ar5_description/meshes/ccs/link5.glb scale=1 -1 1
- link right_link6: geometry collision cylinder length=0.11772 radius=0.044145; visual mesh filename=package://rokae_ar5_description/meshes/ccs/link6.glb scale=1 -1 1
- link right_link7: geometry collision cylinder length=0.038669 radius=0.03559; visual mesh filename=package://rokae_ar5_description/meshes/ccs/link7.glb scale=-1 1 1
- link right_right_finger: geometry collision mesh filename=package://jodell_description/meshes/RG75/finger.glb scale=-1 -1 1; visual mesh filename=package://jodell_description/meshes/RG75/finger.glb scale=-1 -1 1
- link right_right_finger_pad: geometry collision mesh filename=package://jodell_description/meshes/RG75/pad_fiveages.glb scale=1 -1 1; visual mesh filename=package://jodell_description/meshes/RG75/pad_fiveages.glb scale=1 -1 1

File: rokae_ar5_description/urdf/rokae_ar5_dual_rg75.urdf (robot description, URDF)
Before this commit: robot RokaeAR5, 32 links, 31 joints
Links:
- link left_base_link: geometry collision cylinder length=0.105 radius=0.045; visual mesh filename=package://rokae_ar5_description/meshes/srs/base.glb scale=1 1 1
- link left_flange: geometry collision mesh filename=package://jodell_description/meshes/RG75/flange.glb; visual mesh filename=package://jodell_description/meshes/RG75/flange.glb
- link left_gripper_base: geometry collision mesh filename=package://jodell_description/meshes/RG75/base.glb; visual mesh filename=package://jodell_description/meshes/RG75/base.glb
- link left_left_finger: geometry collision mesh filename=package://jodell_description/meshes/RG75/finger.glb; visual mesh filename=package://jodell_description/meshes/RG75/finger.glb
- link left_left_finger_pad: geometry collision mesh filename=package://jodell_description/meshes/RG75/pad_fiveages.glb; visual mesh filename=package://jodell_description/meshes/RG75/pad_fiveages.glb
- link left_link1: geometry collision cylinder length=0.1354 radius=0.0560; visual mesh filename=package://rokae_ar5_description/meshes/srs/link1.glb scale=1 1 1
- link left_link2: geometry collision cylinder length=0.11413 radius=0.053; visual mesh filename=package://rokae_ar5_description/meshes/srs/link2.glb scale=1 1 1
- link left_link3: geometry collision cylinder length=0.096 radius=0.053; collision cylinder length=0.1284 radius=0.0484
- link left_link4: geometry collision cylinder length=0.10 radius=0.03789; visual mesh filename=package://rokae_ar5_description/meshes/srs/link4.glb scale=1 1 1
- link left_link5: geometry collision cylinder length=0.107 radius=0.0383; visual mesh filename=package://rokae_ar5_description/meshes/srs/link5.glb scale=1 1 1
- link left_link6: geometry collision cylinder length=0.1238 radius=0.04; visual mesh filename=package://rokae_ar5_description/meshes/srs/link6.glb scale=1 1 1
- link left_link7: geometry visual mesh filename=package://rokae_ar5_description/meshes/srs/link7.glb scale=1 1 1
- link left_right_finger: geometry collision mesh filename=package://jodell_description/meshes/RG75/finger.glb scale=-1 -1 1; visual mesh filename=package://jodell_description/meshes/RG75/finger.glb scale=-1 -1 1
- link left_right_finger_pad: geometry collision mesh filename=package://jodell_description/meshes/RG75/pad_fiveages.glb scale=1 -1 1; visual mesh filename=package://jodell_description/meshes/RG75/pad_fiveages.glb scale=1 -1 1
- link right_base_link: geometry collision cylinder length=0.105 radius=0.045; visual mesh filename=package://rokae_ar5_description/meshes/srs/base.glb scale=1 -1 1
- link right_flange: geometry collision mesh filename=package://jodell_description/meshes/RG75/flange.glb; visual mesh filename=package://jodell_description/meshes/RG75/flange.glb
- link right_gripper_base: geometry collision mesh filename=package://jodell_description/meshes/RG75/base.glb; visual mesh filename=package://jodell_description/meshes/RG75/base.glb
- link right_left_finger: geometry collision mesh filename=package://jodell_description/meshes/RG75/finger.glb; visual mesh filename=package://jodell_description/meshes/RG75/finger.glb
- link right_left_finger_pad: geometry collision mesh filename=package://jodell_description/meshes/RG75/pad_fiveages.glb; visual mesh filename=package://jodell_description/meshes/RG75/pad_fiveages.glb
- link right_link1: geometry collision cylinder length=0.1354 radius=0.0560; visual mesh filename=package://rokae_ar5_description/meshes/srs/link1.glb scale=1 -1 1
- link right_link2: geometry collision cylinder length=0.11413 radius=0.053; visual mesh filename=package://rokae_ar5_description/meshes/srs/link2.glb scale=1 -1 1
- link right_link3: geometry collision cylinder length=0.096 radius=0.053; collision cylinder length=0.1284 radius=0.0484
- link right_link4: geometry collision cylinder length=0.10 radius=0.03789; visual mesh filename=package://rokae_ar5_description/meshes/srs/link4.glb scale=1 -1 1
- link right_link5: geometry collision cylinder length=0.107 radius=0.0383; visual mesh filename=package://rokae_ar5_description/meshes/srs/link5.glb scale=1 -1 1
- link right_link6: geometry collision cylinder length=0.1238 radius=0.04; visual mesh filename=package://rokae_ar5_description/meshes/srs/link6.glb scale=1 -1 1
- link right_link7: geometry visual mesh filename=package://rokae_ar5_description/meshes/srs/link7.glb scale=1 -1 1
- link right_right_finger: geometry collision mesh filename=package://jodell_description/meshes/RG75/finger.glb scale=-1 -1 1; visual mesh filename=package://jodell_description/meshes/RG75/finger.glb scale=-1 -1 1
- link right_right_finger_pad: geometry collision mesh filename=package://jodell_description/meshes/RG75/pad_fiveages.glb scale=1 -1 1; visual mesh filename=package://jodell_description/meshes/RG75/pad_fiveages.glb scale=1 -1 1
