Commit message: update mesh to glb

File: rokae_ar5_description/xacro/arm_ccs.xacro (robot description, xacro)
@@ -12,11 +12,11 @@
 			<visual>
 				<geometry>
-					<mesh filename="file://$(find rokae_ar5_description)/meshes/ccs/base.obj"/>
-				</geometry>
-			</visual>
-			<xacro:if value="${collider == 'convex'}">
-				<collision>
-					<geometry>
-						<mesh filename="file://$(find rokae_ar5_description)/meshes/ccs/base.obj"/>
+					<mesh filename="file://$(find rokae_ar5_description)/meshes/ccs/base.glb"/>
+				</geometry>
+			</visual>
+			<xacro:if value="${collider == 'convex'}">
+				<collision>
+					<geometry>
+						<mesh filename="file://$(find rokae_ar5_description)/meshes/ccs/base.glb"/>
 					</geometry>
 				</collision>
@@ -48,11 +48,11 @@
 			<visual>
 				<geometry>
-					<mesh filename="file://$(find rokae_ar5_description)/meshes/ccs/link1.obj" scale="1 ${direction} 1"/>
-				</geometry>
-			</visual>
-			<xacro:if value="${collider == 'convex'}">
-				<collision>
-					<geometry>
-						<mesh filename="file://$(find rokae_ar5_description)/meshes/ccs/link1.obj" scale="1 ${direction} 1"/>
+					<mesh filename="file://$(find rokae_ar5_description)/meshes/ccs/link1.glb" scale="1 ${direction} 1"/>
+				</geometry>
+			</visual>
+			<xacro:if value="${collider == 'convex'}">
+				<collision>
+					<geometry>
+						<mesh filename="file://$(find rokae_ar5_description)/meshes/ccs/link1.glb" scale="1 ${direction} 1"/>
 					</geometry>
 				</collision>
@@ -77,11 +77,11 @@
 			<visual>
 				<geometry>
-					<mesh filename="file://$(find rokae_ar5_description)/meshes/ccs/link2.obj" scale="1 ${direction} 1"/>
-				</geometry>
-			</visual>
-			<xacro:if value="${collider == 'convex'}">
-				<collision>
-					<geometry>
-						<mesh filename="file://$(find rokae_ar5_description)/meshes/ccs/link2.obj" scale="1 ${direction} 1"/>
+					<mesh filename="file://$(find rokae_ar5_description)/meshes/ccs/link2.glb" scale="1 ${direction} 1"/>
+				</geometry>
+			</visual>
+			<xacro:if value="${collider == 'convex'}">
+				<collision>
+					<geometry>
+						<mesh filename="file://$(find rokae_ar5_description)/meshes/ccs/link2.glb" scale="1 ${direction} 1"/>
 					</geometry>
 				</collision>
@@ -120,11 +120,11 @@
 			<visual>
 				<geometry>
-					<mesh filename="file://$(find rokae_ar5_description)/meshes/ccs/link3.obj" scale="1 ${direction} 1"/>
-				</geometry>
-			</visual>
-			<xacro:if value="${collider == 'convex'}">
-				<collision>
-					<geometry>
-						<mesh filename="file://$(find rokae_ar5_description)/meshes/ccs/link3.obj" scale="1 ${direction} 1"/>
+					<mesh filename="file://$(find rokae_ar5_description)/meshes/ccs/link3.glb" scale="1 ${direction} 1"/>
+				</geometry>
+			</visual>
+			<xacro:if value="${collider == 'convex'}">
+				<collision>
+					<geometry>
+						<mesh filename="file://$(find rokae_ar5_description)/meshes/ccs/link3.glb" scale="1 ${direction} 1"/>
 					</geometry>
 				</collision>
@@ -163,11 +163,11 @@
 			<visual>
 				<geometry>
-					<mesh filename="file://$(find rokae_ar5_description)/meshes/ccs/link4.obj" scale="1 ${direction} 1"/>
-				</geometry>
-			</visual>
-			<xacro:if value="${collider == 'convex'}">
-				<collision>
-					<geometry>
-						<mesh filename="file://$(find rokae_ar5_description)/meshes/ccs/link4.obj" scale="1 ${direction} 1"/>
+					<mesh filename="file://$(find rokae_ar5_description)/meshes/ccs/link4.glb" scale="1 ${direction} 1"/>
+				</geometry>
+			</visual>
+			<xacro:if value="${collider == 'convex'}">
+				<collision>
+					<geometry>
+						<mesh filename="file://$(find rokae_ar5_description)/meshes/ccs/link4.glb" scale="1 ${direction} 1"/>
 					</geometry>
 				</collision>
@@ -200,11 +200,11 @@
 			<visual>
 				<geometry>
-					<mesh filename="file://$(find rokae_ar5_description)/meshes/ccs/link5.obj" scale="1 ${direction} 1"/>
-				</geometry>
-			</visual>
-			<xacro:if value="${collider == 'convex'}">
-				<collision>
-					<geometry>
-						<mesh filename="file://$(find rokae_ar5_description)/meshes/ccs/link5.obj" scale="1 ${direction} 1"/>
+					<mesh filename="file://$(find rokae_ar5_description)/meshes/ccs/link5.glb" scale="1 ${direction} 1"/>
+				</geometry>
+			</visual>
+			<xacro:if value="${collider == 'convex'}">
+				<collision>
+					<geometry>
+						<mesh filename="file://$(find rokae_ar5_description)/meshes/ccs/link5.glb" scale="1 ${direction} 1"/>
 					</geometry>
 				</collision>
@@ -236,11 +236,11 @@
 			<visual>
 				<geometry>
-					<mesh filename="file://$(find rokae_ar5_description)/meshes/ccs/link6.obj" scale="1 ${direction} 1"/>
-				</geometry>
-			</visual>
-			<xacro:if value="${collider == 'convex'}">
-				<collision>
-					<geometry>
-						<mesh filename="file://$(find rokae_ar5_description)/meshes/ccs/link6.obj" scale="1 ${direction} 1"/>
+					<mesh filename="file://$(find rokae_ar5_description)/meshes/ccs/link6.glb" scale="1 ${direction} 1"/>
+				</geometry>
+			</visual>
+			<xacro:if value="${collider == 'convex'}">
+				<collision>
+					<geometry>
+						<mesh filename="file://$(find rokae_ar5_description)/meshes/ccs/link6.glb" scale="1 ${direction} 1"/>
 					</geometry>
 				</collision>
@@ -272,11 +272,11 @@
 			<visual>
 				<geometry>
-					<mesh filename="file://$(find rokae_ar5_description)/meshes/ccs/link7.obj" scale="${direction} 1 1"/>
-				</geometry>
-			</visual>
-			<xacro:if value="${collider == 'convex'}">
-				<collision>
-					<geometry>
-						<mesh filename="file://$(find rokae_ar5_description)/meshes/ccs/link7.obj" scale=" ${direction} 1 1"/>
+					<mesh filename="file://$(find rokae_ar5_description)/meshes/ccs/link7.glb" scale="${direction} 1 1"/>
+				</geometry>
+			</visual>
+			<xacro:if value="${collider == 'convex'}">
+				<collision>
+					<geometry>
+						<mesh filename="file://$(find rokae_ar5_description)/meshes/ccs/link7.glb" scale=" ${direction} 1 1"/>
 					</geometry>
 				</collision>

File: rokae_ar5_description/xacro/arm_srs.xacro (robot description, xacro)
@@ -13,11 +13,11 @@
 			<visual>
 				<geometry>
-					<mesh filename="file://$(find rokae_ar5_description)/meshes/srs/base.obj" scale="1 ${direction} 1"/>
-				</geometry>
-			</visual>
-			<xacro:if value="${collider == 'convex'}">
-				<collision>
-					<geometry>
-						<mesh filename="file://$(find rokae_ar5_description)/meshes/srs/base.obj" scale="1 ${direction} 1"/>
+					<mesh filename="file://$(find rokae_ar5_description)/meshes/srs/base.glb" scale="1 ${direction} 1"/>
+				</geometry>
+			</visual>
+			<xacro:if value="${collider == 'convex'}">
+				<collision>
+					<geometry>
+						<mesh filename="file://$(find rokae_ar5_description)/meshes/srs/base.glb" scale="1 ${direction} 1"/>
 					</geometry>
 				</collision>
@@ -49,11 +49,11 @@
 			<visual>
 				<geometry>
-					<mesh filename="file://$(find rokae_ar5_description)/meshes/srs/link1.obj" scale="1 ${direction} 1"/>
-				</geometry>
-			</visual>
-			<xacro:if value="${collider == 'convex'}">
-				<collision>
-					<geometry>
-						<mesh filename="file://$(find rokae_ar5_description)/meshes/srs/link1.obj" scale="1 ${direction} 1"/>
+					<mesh filename="file://$(find rokae_ar5_description)/meshes/srs/link1.glb" scale="1 ${direction} 1"/>
+				</geometry>
+			</visual>
+			<xacro:if value="${collider == 'convex'}">
+				<collision>
+					<geometry>
+						<mesh filename="file://$(find rokae_ar5_description)/meshes/srs/link1.glb" scale="1 ${direction} 1"/>
 					</geometry>
 				</collision>
@@ -85,11 +85,11 @@
 			<visual>
 				<geometry>
-					<mesh filename="file://$(find rokae_ar5_description)/meshes/srs/link2.obj" scale="1 ${direction} 1"/>
-				</geometry>
-			</visual>
-			<xacro:if value="${collider == 'convex'}">
-				<collision>
-					<geometry>
-						<mesh filename="file://$(find rokae_ar5_description)/meshes/srs/link2.obj" scale="1 ${direction} 1"/>
+					<mesh filename="file://$(find rokae_ar5_description)/meshes/srs/link2.glb" scale="1 ${direction} 1"/>
+				</geometry>
+			</visual>
+			<xacro:if value="${collider == 'convex'}">
+				<collision>
+					<geometry>
+						<mesh filename="file://$(find rokae_ar5_description)/meshes/srs/link2.glb" scale="1 ${direction} 1"/>
 					</geometry>
 				</collision>
@@ -121,11 +121,11 @@
 			<visual>
 				<geometry>
-					<mesh filename="file://$(find rokae_ar5_description)/meshes/srs/link3.obj" scale="1 ${direction} 1"/>
-				</geometry>
-			</visual>
-			<xacro:if value="${collider == 'convex'}">
-				<collision>
-					<geometry>
-						<mesh filename="file://$(find rokae_ar5_description)/meshes/srs/link3.obj" scale="1 ${direction} 1"/>
+					<mesh filename="file://$(find rokae_ar5_description)/meshes/srs/link3.glb" scale="1 ${direction} 1"/>
+				</geometry>
+			</visual>
+			<xacro:if value="${collider == 'convex'}">
+				<collision>
+					<geometry>
+						<mesh filename="file://$(find rokae_ar5_description)/meshes/srs/link3.glb" scale="1 ${direction} 1"/>
 					</geometry>
 				</collision>
@@ -164,11 +164,11 @@
 			<visual>
 				<geometry>
-					<mesh filename="file://$(find rokae_ar5_description)/meshes/srs/link4.obj" scale="1 ${direction} 1"/>
-				</geometry>
-			</visual>
-			<xacro:if value="${collider == 'convex'}">
-				<collision>
-					<geometry>
-						<mesh filename="file://$(find rokae_ar5_description)/meshes/srs/link4.obj" scale="1 ${direction} 1"/>
+					<mesh filename="file://$(find rokae_ar5_description)/meshes/srs/link4.glb" scale="1 ${direction} 1"/>
+				</geometry>
+			</visual>
+			<xacro:if value="${collider == 'convex'}">
+				<collision>
+					<geometry>
+						<mesh filename="file://$(find rokae_ar5_description)/meshes/srs/link4.glb" scale="1 ${direction} 1"/>
 					</geometry>
 				</collision>
@@ -200,11 +200,11 @@
 			<visual>
 				<geometry>
-					<mesh filename="file://$(find rokae_ar5_description)/meshes/srs/link5.obj" scale="1 ${direction} 1"/>
-				</geometry>
-			</visual>
-			<xacro:if value="${collider == 'convex'}">
-				<collision>
-					<geometry>
-						<mesh filename="file://$(find rokae_ar5_description)/meshes/srs/link5.obj" scale="1 ${direction} 1"/>
+					<mesh filename="file://$(find rokae_ar5_description)/meshes/srs/link5.glb" scale="1 ${direction} 1"/>
+				</geometry>
+			</visual>
+			<xacro:if value="${collider == 'convex'}">
+				<collision>
+					<geometry>
+						<mesh filename="file://$(find rokae_ar5_description)/meshes/srs/link5.glb" scale="1 ${direction} 1"/>
 					</geometry>
 				</collision>
@@ -236,11 +236,11 @@
 			<visual>
 				<geometry>
-					<mesh filename="file://$(find rokae_ar5_description)/meshes/srs/link6.obj" scale="1 ${direction} 1"/>
-				</geometry>
-			</visual>
-			<xacro:if value="${collider == 'convex'}">
-				<collision>
-					<geometry>
-						<mesh filename="file://$(find rokae_ar5_description)/meshes/srs/link6.obj" scale="1 ${direction} 1"/>
+					<mesh filename="file://$(find rokae_ar5_description)/meshes/srs/link6.glb" scale="1 ${direction} 1"/>
+				</geometry>
+			</visual>
+			<xacro:if value="${collider == 'convex'}">
+				<collision>
+					<geometry>
+						<mesh filename="file://$(find rokae_ar5_description)/meshes/srs/link6.glb" scale="1 ${direction} 1"/>
 					</geometry>
 				</collision>
@@ -272,5 +272,5 @@
 			<visual>
 				<geometry>
-					<mesh filename="file://$(find rokae_ar5_description)/meshes/srs/link7.obj" scale="1 ${direction} 1"/>
+					<mesh filename="file://$(find rokae_ar5_description)/meshes/srs/link7.glb" scale="1 ${direction} 1"/>
 				</geometry>
 			</visual>
