Commit message: Add new URDF and mesh files for AR5 SRS robot configuration

File: ar5_srs_description/urdf/ar5_srs_dual.urdf (robot description, URDF)
Before this commit: robot RokaeAR5, 20 links, 19 joints
Links:
- removed link left_eef
- removed link right_eef
- added link left_tcp
- added link right_tcp
- link left_base_link: geometry collision cylinder length=0.105 radius=0.045; visual mesh filename=package://ar5_srs_description/meshes/base.glb scale=1 1 1
- link left_link1: geometry collision cylinder length=0.1354 radius=0.0560; visual mesh filename=package://ar5_srs_description/meshes/link1.glb scale=1 1 1
- link left_link2: geometry collision cylinder length=0.11413 radius=0.053; visual mesh filename=package://ar5_srs_description/meshes/link2.glb scale=1 1 1
- link left_link3: geometry collision cylinder length=0.096 radius=0.053; collision cylinder length=0.1284 radius=0.0484
- link left_link4: geometry collision cylinder length=0.10 radius=0.03789; visual mesh filename=package://ar5_srs_description/meshes/link4.glb scale=1 1 1
- link left_link5: geometry collision cylinder length=0.107 radius=0.0383; visual mesh filename=package://ar5_srs_description/meshes/link5.glb scale=1 1 1
- link left_link6: geometry collision cylinder length=0.1238 radius=0.04; visual mesh filename=package://ar5_srs_description/meshes/link6.glb scale=1 1 1
- link left_link7: geometry visual mesh filename=package://ar5_srs_description/meshes/link7.glb scale=1 1 1
- link right_base_link: geometry collision cylinder length=0.105 radius=0.045; visual mesh filename=package://ar5_srs_description/meshes/base.glb scale=1 -1 1
- link right_link1: geometry collision cylinder length=0.1354 radius=0.0560; visual mesh filename=package://ar5_srs_description/meshes/link1.glb scale=1 -1 1
- link right_link2: geometry collision cylinder length=0.11413 radius=0.053; visual mesh filename=package://ar5_srs_description/meshes/link2.glb scale=1 -1 1
- link right_link3: geometry collision cylinder length=0.096 radius=0.053; collision cylinder length=0.1284 radius=0.0484
- link right_link4: geometry collision cylinder length=0.10 radius=0.03789; visual mesh filename=package://ar5_srs_description/meshes/link4.glb scale=1 -1 1
- link right_link5: geometry collision cylinder length=0.107 radius=0.0383; visual mesh filename=package://ar5_srs_description/meshes/link5.glb scale=1 -1 1
- link right_link6: geometry collision cylinder length=0.1238 radius=0.04; visual mesh filename=package://ar5_srs_description/meshes/link6.glb scale=1 -1 1
- link right_link7: geometry visual mesh filename=package://ar5_srs_description/meshes/link7.glb scale=1 -1 1
Joints:
- removed joint left_eef_joint
- removed joint right_eef_joint
- added joint left_tcp_joint: type fixed, parent left_link7, child left_tcp
- added joint right_tcp_joint: type fixed, parent right_link7, child right_tcp

File: ar5_srs_description/urdf/ar5_srs_dual_rg75.urdf (robot description, URDF)
Before this commit: robot RokaeAR5, 34 links, 33 joints
Links:
- link left_base_link: geometry collision cylinder length=0.105 radius=0.045; visual mesh filename=package://ar5_srs_description/meshes/base.glb scale=1 1 1
- link left_flange: geometry visual mesh filename=package://jodell_description/meshes/RG75/flange.glb
- link left_gripper_base: geometry visual mesh filename=package://jodell_description/meshes/RG75/base.glb
- link left_left_finger: geometry visual mesh filename=package://jodell_description/meshes/RG75/finger.glb; visual mesh filename=package://jodell_description/meshes/RG75/finger_support.glb
- link left_left_finger_pad: geometry visual mesh filename=package://jodell_description/meshes/RG75/pad_fiveages.glb
- link left_link1: mass 2.683 -> 2.4; geometry collision cylinder length=0.1354 radius=0.0560; visual mesh filename=package://ar5_srs_description/meshes/link1.glb scale=1 1 1
- link left_link2: mass 2.3 -> 2.26; geometry collision cylinder length=0.11413 radius=0.053; visual mesh filename=package://ar5_srs_description/meshes/link2.glb scale=1 1 1
- link left_link3: mass 1.862 -> 1.85; geometry collision cylinder length=0.096 radius=0.053; collision cylinder length=0.1284 radius=0.0484
- link left_link4: mass 1.234 -> 1.19; geometry collision cylinder length=0.10 radius=0.03789; visual mesh filename=package://ar5_srs_description/meshes/link4.glb scale=1 1 1
- link left_link5: mass 1.329 -> 0.95; geometry collision cylinder length=0.107 radius=0.0383; visual mesh filename=package://ar5_srs_description/meshes/link5.glb scale=1 1 1
- link left_link6: mass 0.93 -> 1.06; geometry collision cylinder length=0.1238 radius=0.04; visual mesh filename=package://ar5_srs_description/meshes/link6.glb scale=1 1 1
- link left_link7: mass 0.33 -> 0.18; geometry visual mesh filename=package://ar5_srs_description/meshes/link7.glb scale=1 1 1
- link left_right_finger: geometry visual mesh filename=package://jodell_description/meshes/RG75/finger.glb; visual mesh filename=package://jodell_description/meshes/RG75/finger_support.glb
- link left_right_finger_pad: geometry visual mesh filename=package://jodell_description/meshes/RG75/pad_fiveages.glb scale=1 -1 1
- link left_tcp: mass 0.0 -> None
- link right_base_link: geometry collision cylinder length=0.105 radius=0.045; visual mesh filename=package://ar5_srs_description/meshes/base.glb scale=1 -1 1
- link right_flange: geometry visual mesh filename=package://jodell_description/meshes/RG75/flange.glb
- link right_gripper_base: geometry visual mesh filename=package://jodell_description/meshes/RG75/base.glb
- link right_left_finger: geometry visual mesh filename=package://jodell_description/meshes/RG75/finger.glb; visual mesh filename=package://jodell_description/meshes/RG75/finger_support.glb
- link right_left_finger_pad: geometry visual mesh filename=package://jodell_description/meshes/RG75/pad_fiveages.glb
- link right_link1: mass 2.683 -> 2.4; geometry collision cylinder length=0.1354 radius=0.0560; visual mesh filename=package://ar5_srs_description/meshes/link1.glb scale=1 -1 1
- link right_link2: mass 2.3 -> 2.26; geometry collision cylinder length=0.11413 radius=0.053; visual mesh filename=package://ar5_srs_description/meshes/link2.glb scale=1 -1 1
- link right_link3: mass 1.862 -> 1.85; geometry collision cylinder length=0.096 radius=0.053; collision cylinder length=0.1284 radius=0.0484
- link right_link4: mass 1.234 -> 1.19; geometry collision cylinder length=0.10 radius=0.03789; visual mesh filename=package://ar5_srs_description/meshes/link4.glb scale=1 -1 1
- link right_link5: mass 1.329 -> 0.95; geometry collision cylinder length=0.107 radius=0.0383; visual mesh filename=package://ar5_srs_description/meshes/link5.glb scale=1 -1 1
- link right_link6: mass 0.93 -> 1.06; geometry collision cylinder length=0.1238 radius=0.04; visual mesh filename=package://ar5_srs_description/meshes/link6.glb scale=1 -1 1
- link right_link7: mass 0.33 -> 0.18; geometry visual mesh filename=package://ar5_srs_description/meshes/link7.glb scale=1 -1 1
- link right_right_finger: geometry visual mesh filename=package://jodell_description/meshes/RG75/finger.glb; visual mesh filename=package://jodell_description/meshes/RG75/finger_support.glb
- link right_right_finger_pad: geometry visual mesh filename=package://jodell_description/meshes/RG75/pad_fiveages.glb scale=1 -1 1
- link right_tcp: mass 0.0 -> None
Joints:
- joint left_joint1: limit lower=-3.1067 upper=3.1067 effort=108 velocity=3.0543261909900763 -> lower=-3.14 upper=3.14 effort=108 velocity=3.9269908169872414; origin (none) -> xyz=0.0 0.0 0.1745 rpy=0 0 -3.14159
- joint left_joint2: axis 0 1 0 -> 0 -1 0; limit lower=-2.0944 upper=2.0944 effort=108 velocity=3.0543261909900763 -> lower=-2.12 upper=2.12 effort=108 velocity=3.9269908169872414; origin xyz=0.0 0.0 0.1745 -> (none)
- joint left_joint3: limit lower=-3.1067 upper=3.1067 effort=66 velocity=4.71238898038469 -> lower=-3.14 upper=3.14 effort=66 velocity=5.235987755982989; origin xyz=0.0 0.0 0.314 -> xyz=0.0 0.0 0.305 rpy=0 0 3.1415926535
- joint left_joint4: limit lower=-1.0472 upper=2.5307 effort=66 velocity=5.235987755982989 -> lower=-1.39 upper=2.50 effort=66 velocity=5.235987755982989
- joint left_joint5: limit lower=-3.1067 upper=3.1067 effort=19 velocity=4.1887902047863905 -> lower=-3.14 upper=3.14 effort=19 velocity=4.1887902047863905; origin xyz=-0.01 0.0 0.272 -> xyz=-0.01 0.0 0.179
- joint left_joint6: limit lower=-1.0472 upper=1.0472 effort=19 velocity=4.1887902047863905 -> lower=-1.96 upper=1.96 effort=19 velocity=4.1887902047863905
- joint left_joint7: axis 1 0 0 -> 0 0 1; limit lower=-1.0472 upper=1.0472 effort=19 velocity=4.1887902047863905 -> lower=-3.14 upper=3.14 effort=19 velocity=4.1887902047863905; origin (none) -> xyz=0.0 0.0 0.166
- joint left_left_finger_pad_joint: origin xyz=-0.014715 0.011478 0.0315 -> xyz=-0.014785 0.011478 0.0315
- joint left_right_finger_pad_joint: origin xyz=0.014785 -0.011478 0.03175 -> xyz=0.014785 -0.011478 0.0315
- joint left_tcp_joint: origin xyz=0.0 0.0 0.097 -> (none)
- joint right_joint1: limit lower=-3.1067 upper=3.1067 effort=108 velocity=3.0543261909900763 -> lower=-3.14 upper=3.14 effort=108 velocity=3.9269908169872414; origin (none) -> xyz=0.0 0.0 0.1745 rpy=0 0 -3.14159
- joint right_joint2: axis 0 1 0 -> 0 -1 0; limit lower=-2.0944 upper=2.0944 effort=108 velocity=3.0543261909900763 -> lower=-2.12 upper=2.12 effort=108 velocity=3.9269908169872414; origin xyz=0.0 0.0 0.1745 -> (none)
- joint right_joint3: limit lower=-3.1067 upper=3.1067 effort=66 velocity=4.71238898038469 -> lower=-3.14 upper=3.14 effort=66 velocity=5.235987755982989; origin xyz=0.0 0.0 0.314 -> xyz=0.0 0.0 0.305 rpy=0 0 3.1415926535
- joint right_joint4: limit lower=-1.0472 upper=2.5307 effort=66 velocity=5.235987755982989 -> lower=-1.39 upper=2.50 effort=66 velocity=5.235987755982989
- joint right_joint5: limit lower=-3.1067 upper=3.1067 effort=19 velocity=4.1887902047863905 -> lower=-3.14 upper=3.14 effort=19 velocity=4.1887902047863905; origin xyz=-0.01 0.0 0.272 -> xyz=-0.01 0.0 0.179
- joint right_joint6: limit lower=-1.0472 upper=1.0472 effort=19 velocity=4.1887902047863905 -> lower=-1.96 upper=1.96 effort=19 velocity=4.1887902047863905
- joint right_joint7: axis 1 0 0 -> 0 0 1; limit lower=-1.0472 upper=1.0472 effort=19 velocity=4.1887902047863905 -> lower=-3.14 upper=3.14 effort=19 velocity=4.1887902047863905; origin (none) -> xyz=0.0 0.0 0.166
- joint right_left_finger_pad_joint: origin xyz=-0.014715 0.011478 0.0315 -> xyz=-0.014785 0.011478 0.0315
- joint right_right_finger_pad_joint: origin xyz=0.014785 -0.011478 0.03175 -> xyz=0.014785 -0.011478 0.0315
- joint right_tcp_joint: origin xyz=0.0 0.0 0.097 -> (none)

File: ar5_srs_description/urdf/ar5_srs_left.urdf (robot description, URDF)
Before this commit: robot RokaeAR5, 8 links, 7 joints
Links:
- added link tcp
- link base_link: geometry collision cylinder length=0.105 radius=0.045; visual mesh filename=package://ar5_srs_description/meshes/base.glb scale=1 1 1
- link link1: geometry collision cylinder length=0.1354 radius=0.0560; visual mesh filename=package://ar5_srs_description/meshes/link1.glb scale=1 1 1
- link link2: geometry collision cylinder length=0.11413 radius=0.053; visual mesh filename=package://ar5_srs_description/meshes/link2.glb scale=1 1 1
- link link3: geometry collision cylinder length=0.096 radius=0.053; collision cylinder length=0.1284 radius=0.0484
- link link4: geometry collision cylinder length=0.10 radius=0.03789; visual mesh filename=package://ar5_srs_description/meshes/link4.glb scale=1 1 1
- link link5: geometry collision cylinder length=0.107 radius=0.0383; visual mesh filename=package://ar5_srs_description/meshes/link5.glb scale=1 1 1
- link link6: geometry collision cylinder length=0.1238 radius=0.04; visual mesh filename=package://ar5_srs_description/meshes/link6.glb scale=1 1 1
- link link7: geometry visual mesh filename=package://ar5_srs_description/meshes/link7.glb scale=1 1 1
Joints:
- added joint tcp_joint: type fixed, parent link7, child tcp

File: ar5_srs_description/xacro/arm_srs.xacro (robot description, xacro)
@@ -13,11 +13,11 @@
 			<visual>
 				<geometry>
-					<mesh filename="file://$(find rokae_ar5_description)/meshes/srs/base.glb" scale="1 ${direction} 1"/>
-				</geometry>
-			</visual>
-			<xacro:if value="${collider == 'convex'}">
-				<collision>
-					<geometry>
-						<mesh filename="file://$(find rokae_ar5_description)/meshes/srs/base.glb" scale="1 ${direction} 1"/>
+					<mesh filename="package://ar5_srs_description/meshes/base.glb" scale="1 ${direction} 1"/>
+				</geometry>
+			</visual>
+			<xacro:if value="${collider == 'convex'}">
+				<collision>
+					<geometry>
+						<mesh filename="file://$(find ar5_srs_description)/meshes/base.glb" scale="1 ${direction} 1"/>
 					</geometry>
 				</collision>
@@ -49,11 +49,11 @@
 			<visual>
 				<geometry>
-					<mesh filename="file://$(find rokae_ar5_description)/meshes/srs/link1.glb" scale="1 ${direction} 1"/>
-				</geometry>
-			</visual>
-			<xacro:if value="${collider == 'convex'}">
-				<collision>
-					<geometry>
-						<mesh filename="file://$(find rokae_ar5_description)/meshes/srs/link1.glb" scale="1 ${direction} 1"/>
+					<mesh filename="file://$(find ar5_srs_description)/meshes/link1.glb" scale="1 ${direction} 1"/>
+				</geometry>
+			</visual>
+			<xacro:if value="${collider == 'convex'}">
+				<collision>
+					<geometry>
+						<mesh filename="file://$(find ar5_srs_description)/meshes/link1.glb" scale="1 ${direction} 1"/>
 					</geometry>
 				</collision>
@@ -85,11 +85,11 @@
 			<visual>
 				<geometry>
-					<mesh filename="file://$(find rokae_ar5_description)/meshes/srs/link2.glb" scale="1 ${direction} 1"/>
-				</geometry>
-			</visual>
-			<xacro:if value="${collider == 'convex'}">
-				<collision>
-					<geometry>
-						<mesh filename="file://$(find rokae_ar5_description)/meshes/srs/link2.glb" scale="1 ${direction} 1"/>
+					<mesh filename="file://$(find ar5_srs_description)/meshes/link2.glb" scale="1 ${direction} 1"/>
+				</geometry>
+			</visual>
+			<xacro:if value="${collider == 'convex'}">
+				<collision>
+					<geometry>
+						<mesh filename="file://$(find ar5_srs_description)/meshes/link2.glb" scale="1 ${direction} 1"/>
 					</geometry>
 				</collision>
@@ -121,11 +121,11 @@
 			<visual>
 				<geometry>
-					<mesh filename="file://$(find rokae_ar5_description)/meshes/srs/link3.glb" scale="1 ${direction} 1"/>
-				</geometry>
-			</visual>
-			<xacro:if value="${collider == 'convex'}">
-				<collision>
-					<geometry>
-						<mesh filename="file://$(find rokae_ar5_description)/meshes/srs/link3.glb" scale="1 ${direction} 1"/>
+					<mesh filename="file://$(find ar5_srs_description)/meshes/link3.glb" scale="1 ${direction} 1"/>
+				</geometry>
+			</visual>
+			<xacro:if value="${collider == 'convex'}">
+				<collision>
+					<geometry>
+						<mesh filename="file://$(find ar5_srs_description)/meshes/link3.glb" scale="1 ${direction} 1"/>
 					</geometry>
 				</collision>
@@ -164,11 +164,11 @@
 			<visual>
 				<geometry>
-					<mesh filename="file://$(find rokae_ar5_description)/meshes/srs/link4.glb" scale="1 ${direction} 1"/>
-				</geometry>
-			</visual>
-			<xacro:if value="${collider == 'convex'}">
-				<collision>
-					<geometry>
-						<mesh filename="file://$(find rokae_ar5_description)/meshes/srs/link4.glb" scale="1 ${direction} 1"/>
+					<mesh filename="file://$(find ar5_srs_description)/meshes/link4.glb" scale="1 ${direction} 1"/>
+				</geometry>
+			</visual>
+			<xacro:if value="${collider == 'convex'}">
+				<collision>
+					<geometry>
+						<mesh filename="file://$(find ar5_srs_description)/meshes/link4.glb" scale="1 ${direction} 1"/>
 					</geometry>
 				</collision>
@@ -200,11 +200,11 @@
 			<visual>
 				<geometry>
-					<mesh filename="file://$(find rokae_ar5_description)/meshes/srs/link5.glb" scale="1 ${direction} 1"/>
-				</geometry>
-			</visual>
-			<xacro:if value="${collider == 'convex'}">
-				<collision>
-					<geometry>
-						<mesh filename="file://$(find rokae_ar5_description)/meshes/srs/link5.glb" scale="1 ${direction} 1"/>
+					<mesh filename="file://$(find ar5_srs_description)/meshes/link5.glb" scale="1 ${direction} 1"/>
+				</geometry>
+			</visual>
+			<xacro:if value="${collider == 'convex'}">
+				<collision>
+					<geometry>
+						<mesh filename="file://$(find ar5_srs_description)/meshes/link5.glb" scale="1 ${direction} 1"/>
 					</geometry>
 				</collision>
@@ -236,11 +236,11 @@
 			<visual>
 				<geometry>
-					<mesh filename="file://$(find rokae_ar5_description)/meshes/srs/link6.glb" scale="1 ${direction} 1"/>
-				</geometry>
-			</visual>
-			<xacro:if value="${collider == 'convex'}">
-				<collision>
-					<geometry>
-						<mesh filename="file://$(find rokae_ar5_description)/meshes/srs/link6.glb" scale="1 ${direction} 1"/>
+					<mesh filename="file://$(find ar5_srs_description)/meshes/link6.glb" scale="1 ${direction} 1"/>
+				</geometry>
+			</visual>
+			<xacro:if value="${collider == 'convex'}">
+				<collision>
+					<geometry>
+						<mesh filename="file://$(find ar5_srs_description)/meshes/link6.glb" scale="1 ${direction} 1"/>
 					</geometry>
 				</collision>
@@ -272,5 +272,5 @@
 			<visual>
 				<geometry>
-					<mesh filename="file://$(find rokae_ar5_description)/meshes/srs/link7.glb" scale="1 ${direction} 1"/>
+					<mesh filename="file://$(find ar5_srs_description)/meshes/link7.glb" scale="1 ${direction} 1"/>
 				</geometry>
 			</visual>

File: ar5_srs_description/xacro/grippers.xacro (robot description, xacro)
@@ -9,9 +9,9 @@
         type: 夹爪类型 ('rg75', 'leapmotor', '' 等)
         arm_config: 配置方式 ('left', 'right', 'dual')
-        注意：现在 SRS 和 CCS 都使用 tcp 作为连接点，所以不需要 arm_type 参数了
+        注意：使用 tcp 作为夹爪连接点
         -->
         <xacro:if value="${type == 'rg75'}">
             <xacro:include filename="$(find jodell_description)/xacro/RG75-300.xacro"/>
-            <!-- 统一使用 tcp 作为连接点（SRS 和 CCS 都已支持） -->
+            <!-- 统一使用 tcp 作为连接点 -->
             <xacro:if value="${arm_config == 'left'}">
                 <xacro:RG75-300 name="" use_flange="true"/>

File: ar5_srs_description/xacro/robot.xacro (robot description, xacro)
@@ -1,4 +1,4 @@
 <?xml version="1.0"?>
-<robot name="RokaeAR5" xmlns:xacro="http://www.ros.org/wiki/xacro">
+<robot name="AR5_SRS" xmlns:xacro="http://www.ros.org/wiki/xacro">
 	<xacro:arg name="collider" default="convex"/>
 	<xacro:arg name="type" default="left"/>
@@ -6,40 +6,7 @@
 	<xacro:property name="type_arg" value="$(arg type)"/>
 	<!-- 默认值 -->
-	<xacro:property name="selected_arm_type" value="srs"/>      <!-- srs 或 ccs -->
 	<xacro:property name="selected_arm_config" value="left"/>    <!-- left, right, dual -->
 	<xacro:property name="selected_gripper_type" value=""/>     <!-- 空字符串或 rg75 -->
 	<!-- 解析 type 参数 - 使用显式匹配 -->
-	<!-- 处理 CCS 类型 -->
-	<xacro:if value="${type_arg == 'ccs_left'}">
-		<xacro:property name="selected_arm_type" value="ccs"/>
-		<xacro:property name="selected_arm_config" value="left"/>
-		<xacro:property name="selected_gripper_type" value=""/>
-	</xacro:if>
-	<xacro:if value="${type_arg == 'ccs_right'}">
-		<xacro:property name="selected_arm_type" value="ccs"/>
-		<xacro:property name="selected_arm_config" value="right"/>
-		<xacro:property name="selected_gripper_type" value=""/>
-	</xacro:if>
-	<xacro:if value="${type_arg == 'dual_ccs'}">
-		<xacro:property name="selected_arm_type" value="ccs"/>
-		<xacro:property name="selected_arm_config" value="dual"/>
-		<xacro:property name="selected_gripper_type" value=""/>
-	</xacro:if>
-	<xacro:if value="${type_arg == 'ccs_left_rg75'}">
-		<xacro:property name="selected_arm_type" value="ccs"/>
-		<xacro:property name="selected_arm_config" value="left"/>
-		<xacro:property name="selected_gripper_type" value="rg75"/>
-	</xacro:if>
-	<xacro:if value="${type_arg == 'ccs_right_rg75'}">
-		<xacro:property name="selected_arm_type" value="ccs"/>
-		<xacro:property name="selected_arm_config" value="right"/>
-		<xacro:property name="selected_gripper_type" value="rg75"/>
-	</xacro:if>
-	<xacro:if value="${type_arg == 'dual_ccs_rg75'}">
-		<xacro:property name="selected_arm_type" value="ccs"/>
-		<xacro:property name="selected_arm_config" value="dual"/>
-		<xacro:property name="selected_gripper_type" value="rg75"/>
-	</xacro:if>
-	<!-- 处理 SRS 类型（默认） -->
 	<xacro:if value="${type_arg == 'left'}">
 		<xacro:property name="selected_arm_config" value="left"/>
@@ -67,11 +34,6 @@
 	</xacro:if>
 	<!-- Include Component Macros -->
-	<xacro:if value="${selected_arm_type == 'srs'}">
-		<xacro:include filename="$(find rokae_ar5_description)/xacro/arm_srs.xacro"/>
-	</xacro:if>
-	<xacro:if value="${selected_arm_type == 'ccs'}">
-		<xacro:include filename="$(find rokae_ar5_description)/xacro/arm_ccs.xacro"/>
-	</xacro:if>
-	<xacro:include filename="$(find rokae_ar5_description)/xacro/grippers.xacro"/>
+	<xacro:include filename="$(find ar5_srs_description)/xacro/arm_srs.xacro"/>
+	<xacro:include filename="$(find ar5_srs_description)/xacro/grippers.xacro"/>
 	<!-- 根据 arm_config 创建机械臂 -->
 	<xacro:if value="${selected_arm_config == 'left'}">

File: ar5_srs_description/xacro/ros2_control/robot.xacro (robot description, xacro)
@@ -8,6 +8,6 @@
 		<origin/>
 	</joint>
-	<xacro:include filename="$(find rokae_ar5_description)/xacro/robot.xacro"/>
-	<xacro:include filename="$(find rokae_ar5_description)/xacro/ros2_control/interfaces.xacro"/>
+	<xacro:include filename="$(find ar5_srs_description)/xacro/robot.xacro"/>
+	<xacro:include filename="$(find ar5_srs_description)/xacro/ros2_control/interfaces.xacro"/>
 	<!-- 使用 robot.xacro 中已定义的 property 来判断 -->
 	<!-- selected_arm_config: left, right, dual -->
@@ -140,11 +140,11 @@
 			<plugin filename="gz_ros2_control-system" name="gz_ros2_control::GazeboSimROS2ControlPlugin">
 				<xacro:if value="${selected_arm_config == 'left'}">
-					<parameters>$(find rokae_ar5_description)/config/ros2_control/ros2_controllers.yaml</parameters>
+					<parameters>$(find ar5_srs_description)/config/ros2_control/ros2_controllers.yaml</parameters>
 				</xacro:if>
 				<xacro:if value="${selected_arm_config == 'right'}">
-					<parameters>$(find rokae_ar5_description)/config/ros2_control/right.yaml</parameters>
+					<parameters>$(find ar5_srs_description)/config/ros2_control/right.yaml</parameters>
 				</xacro:if>
 				<xacro:if value="${selected_arm_config == 'dual'}">
-					<parameters>$(find rokae_ar5_description)/config/ros2_control/dual.yaml</parameters>
+					<parameters>$(find ar5_srs_description)/config/ros2_control/dual.yaml</parameters>
 				</xacro:if>
 			</plugin>
