Commit message: Enhance gripper configuration for AR5 robot by adding support for 'ag2f90' type and updating related parameters in Xacro files.

File: ar5_ccs_description/xacro/grippers.xacro (robot description, xacro)
@@ -7,5 +7,5 @@
     <xacro:macro name="Grippers" params="type arm_config">
         <!--
-        type: 夹爪类型 ('rg75', 'leapmotor', '' 等)
+        type: 夹爪类型 ('rg75', 'ag2f90', 'leapmotor', '' 等)
         arm_config: 配置方式 ('left', 'right', 'dual')
         注意：现在 SRS 和 CCS 都使用 tcp 作为连接点，所以不需要 arm_type 参数了
@@ -45,4 +45,37 @@
             </xacro:if>
         </xacro:if>
+        <xacro:if value="${type == 'ag2f90'}">
+            <xacro:include filename="$(find changingtek_description)/xacro/AG2F90-C.xacro"/>
+            <xacro:if value="${arm_config == 'left'}">
+                <xacro:AG2F90-C name="" use_flange="true" pad="none"/>
+                <joint name="gripper_base_joint" type="fixed">
+                    <origin xyz="0 0 0" rpy="0 0 -1.5708"/>
+                    <parent link="tcp"/>
+                    <child link="flange"/>
+                </joint>
+            </xacro:if>
+            <xacro:if value="${arm_config == 'right'}">
+                <xacro:AG2F90-C name="" use_flange="true" pad="none"/>
+                <joint name="gripper_base_joint" type="fixed">
+                    <origin xyz="0 0 0" rpy="0 0 1.5708"/>
+                    <parent link="tcp"/>
+                    <child link="flange"/>
+                </joint>
+            </xacro:if>
+            <xacro:if value="${arm_config == 'dual'}">
+                <xacro:AG2F90-C name="left" use_flange="true" pad="none"/>
+                <xacro:AG2F90-C name="right" use_flange="true" pad="none"/>
+                <joint name="left_gripper_base_joint" type="fixed">
+                    <origin xyz="0 0 0"/>
+                    <parent link="left_tcp"/>
+                    <child link="left_flange"/>
+                </joint>
+                <joint name="right_gripper_base_joint" type="fixed">
+                    <origin xyz="0 0 0"/>
+                    <parent link="right_tcp"/>
+                    <child link="right_flange"/>
+                </joint>
+            </xacro:if>
+        </xacro:if>
         <!-- 可以在这里添加其他夹爪类型，如 leapmotor -->
         <xacro:if value="${type == 'leapmotor'}">

File: ar5_ccs_description/xacro/robot.xacro (robot description, xacro)
@@ -7,5 +7,5 @@
 	<!-- 默认值 -->
 	<xacro:property name="selected_arm_config" value="dual"/>    <!-- left, right, dual -->
-	<xacro:property name="selected_gripper_type" value=""/>     <!-- 空字符串或 rg75 -->
+	<xacro:property name="selected_gripper_type" value=""/>     <!-- 空字符串, rg75, ag2f90 -->
 	<!-- 解析 type 参数 - 使用显式匹配 -->
 	<!-- 处理 CCS 类型 -->
@@ -28,4 +28,15 @@
 	<xacro:if value="${type_arg == 'rg75'}">
 		<xacro:property name="selected_gripper_type" value="rg75"/>
+	</xacro:if>
+	<xacro:if value="${type_arg == 'left_ag2f90'}">
+		<xacro:property name="selected_arm_config" value="left"/>
+		<xacro:property name="selected_gripper_type" value="ag2f90"/>
+	</xacro:if>
+	<xacro:if value="${type_arg == 'right_ag2f90'}">
+		<xacro:property name="selected_arm_config" value="right"/>
+		<xacro:property name="selected_gripper_type" value="ag2f90"/>
+	</xacro:if>
+	<xacro:if value="${type_arg == 'ag2f90'}">
+		<xacro:property name="selected_gripper_type" value="ag2f90"/>
 	</xacro:if>
 	<!-- Include Component Macros -->

File: ar5_ccs_description/xacro/ros2_control/robot.xacro (robot description, xacro)
@@ -22,4 +22,14 @@
 					<param name="joint_impedance">200,200,200,200,20,20,20</param>
 					<param name="local_ip">192.168.1.233</param>
+					<xacro:if value="${selected_gripper_type == 'rg75'}">
+						<param name="gripper_type">jodell</param>
+					</xacro:if>
+					<xacro:if value="${selected_gripper_type == 'ag2f90'}">
+						<param name="gripper_type">ag2f90d</param>
+						<param name="gripper_slave_id">1</param>
+						<param name="gripper_close_pos">9000</param>
+						<param name="gripper_max_opening_distance">1.0</param>
+						<param name="gripper_configure_xpanel">false</param>
+					</xacro:if>
 				</hardware>
 				<xacro:ar5_interfaces name="left"/>
@@ -40,4 +50,14 @@
 					<param name="joint_impedance">200,200,200,200,20,20,20</param>
 					<param name="local_ip">192.168.1.233</param>
+					<xacro:if value="${selected_gripper_type == 'rg75'}">
+						<param name="gripper_type">jodell</param>
+					</xacro:if>
+					<xacro:if value="${selected_gripper_type == 'ag2f90'}">
+						<param name="gripper_type">ag2f90d</param>
+						<param name="gripper_slave_id">1</param>
+						<param name="gripper_close_pos">9000</param>
+						<param name="gripper_max_opening_distance">1.0</param>
+						<param name="gripper_configure_xpanel">false</param>
+					</xacro:if>
 				</hardware>
 				<xacro:ar5_interfaces name="right"/>
@@ -66,4 +86,14 @@
 					<param name="joint_impedance">200,200,200,200,20,20,20</param>
 					<param name="local_ip">192.168.1.233</param>
+					<xacro:if value="${selected_gripper_type == 'rg75'}">
+						<param name="gripper_type">jodell</param>
+					</xacro:if>
+					<xacro:if value="${selected_gripper_type == 'ag2f90'}">
+						<param name="gripper_type">ag2f90d</param>
+						<param name="gripper_slave_id">1</param>
+						<param name="gripper_close_pos">9000</param>
+						<param name="gripper_max_opening_distance">1.0</param>
+						<param name="gripper_configure_xpanel">false</param>
+					</xacro:if>
 				</hardware>
 				<xacro:ar5_interfaces name=""/>

File: ar5_srs_description/xacro/grippers.xacro (robot description, xacro)
@@ -7,5 +7,5 @@
     <xacro:macro name="Grippers" params="type arm_config">
         <!--
-        type: 夹爪类型 ('rg75', 'leapmotor', '' 等)
+        type: 夹爪类型 ('rg75', 'ag2f90', 'leapmotor', '' 等)
         arm_config: 配置方式 ('left', 'right', 'dual')
         注意：使用 tcp 作为夹爪连接点
@@ -45,4 +45,37 @@
             </xacro:if>
         </xacro:if>
+        <xacro:if value="${type == 'ag2f90'}">
+            <xacro:include filename="$(find changingtek_description)/xacro/AG2F90-C.xacro"/>
+            <xacro:if value="${arm_config == 'left'}">
+                <xacro:AG2F90-C name="" use_flange="true" pad="none"/>
+                <joint name="gripper_base_joint" type="fixed">
+                    <origin xyz="0 0 0" rpy="0 0 -1.5708"/>
+                    <parent link="tcp"/>
+                    <child link="flange"/>
+                </joint>
+            </xacro:if>
+            <xacro:if value="${arm_config == 'right'}">
+                <xacro:AG2F90-C name="" use_flange="true" pad="none"/>
+                <joint name="gripper_base_joint" type="fixed">
+                    <origin xyz="0 0 0" rpy="0 0 1.5708"/>
+                    <parent link="tcp"/>
+                    <child link="flange"/>
+                </joint>
+            </xacro:if>
+            <xacro:if value="${arm_config == 'dual'}">
+                <xacro:AG2F90-C name="left" use_flange="true" pad="none"/>
+                <xacro:AG2F90-C name="right" use_flange="true" pad="none"/>
+                <joint name="left_gripper_base_joint" type="fixed">
+                    <origin xyz="0 0 0"/>
+                    <parent link="left_tcp"/>
+                    <child link="left_flange"/>
+                </joint>
+                <joint name="right_gripper_base_joint" type="fixed">
+                    <origin xyz="0 0 0"/>
+                    <parent link="right_tcp"/>
+                    <child link="right_flange"/>
+                </joint>
+            </xacro:if>
+        </xacro:if>
         <!-- 可以在这里添加其他夹爪类型，如 leapmotor -->
         <xacro:if value="${type == 'leapmotor'}">

File: ar5_srs_description/xacro/robot.xacro (robot description, xacro)
@@ -7,5 +7,5 @@
 	<!-- 默认值 -->
 	<xacro:property name="selected_arm_config" value="dual"/>    <!-- left, right, dual -->
-	<xacro:property name="selected_gripper_type" value=""/>     <!-- 空字符串或 rg75 -->
+	<xacro:property name="selected_gripper_type" value=""/>     <!-- 空字符串, rg75, ag2f90 -->
 	<!-- 解析 type 参数 - 使用显式匹配 -->
 	<xacro:if value="${type_arg == 'left'}">
@@ -27,4 +27,15 @@
 	<xacro:if value="${type_arg == 'rg75'}">
 		<xacro:property name="selected_gripper_type" value="rg75"/>
+	</xacro:if>
+	<xacro:if value="${type_arg == 'left_ag2f90'}">
+		<xacro:property name="selected_arm_config" value="left"/>
+		<xacro:property name="selected_gripper_type" value="ag2f90"/>
+	</xacro:if>
+	<xacro:if value="${type_arg == 'right_ag2f90'}">
+		<xacro:property name="selected_arm_config" value="right"/>
+		<xacro:property name="selected_gripper_type" value="ag2f90"/>
+	</xacro:if>
+	<xacro:if value="${type_arg == 'ag2f90'}">
+		<xacro:property name="selected_gripper_type" value="ag2f90"/>
 	</xacro:if>
 	<!-- Include Component Macros -->

File: ar5_srs_description/xacro/ros2_control/robot.xacro (robot description, xacro)
@@ -24,4 +24,14 @@
 <!--					<param name="joint_impedance">500,500,500,500,50,50,50</param>-->
 					<param name="local_ip">192.168.1.233</param>
+					<xacro:if value="${selected_gripper_type == 'rg75'}">
+						<param name="gripper_type">jodell</param>
+					</xacro:if>
+					<xacro:if value="${selected_gripper_type == 'ag2f90'}">
+						<param name="gripper_type">ag2f90d</param>
+						<param name="gripper_slave_id">1</param>
+						<param name="gripper_close_pos">9000</param>
+						<param name="gripper_max_opening_distance">1.0</param>
+						<param name="gripper_configure_xpanel">false</param>
+					</xacro:if>
 				</hardware>
 				<xacro:ar5_interfaces name="left"/>
@@ -44,4 +54,14 @@
 <!--					<param name="joint_impedance">500,500,500,500,50,50,50</param>-->
 					<param name="local_ip">192.168.1.233</param>
+					<xacro:if value="${selected_gripper_type == 'rg75'}">
+						<param name="gripper_type">jodell</param>
+					</xacro:if>
+					<xacro:if value="${selected_gripper_type == 'ag2f90'}">
+						<param name="gripper_type">ag2f90d</param>
+						<param name="gripper_slave_id">1</param>
+						<param name="gripper_close_pos">9000</param>
+						<param name="gripper_max_opening_distance">1.0</param>
+						<param name="gripper_configure_xpanel">false</param>
+					</xacro:if>
 				</hardware>
 				<xacro:ar5_interfaces name="right"/>
@@ -74,4 +94,14 @@
 					</xacro:if>
 					<param name="local_ip">192.168.1.233</param>
+					<xacro:if value="${selected_gripper_type == 'rg75'}">
+						<param name="gripper_type">jodell</param>
+					</xacro:if>
+					<xacro:if value="${selected_gripper_type == 'ag2f90'}">
+						<param name="gripper_type">ag2f90d</param>
+						<param name="gripper_slave_id">1</param>
+						<param name="gripper_close_pos">9000</param>
+						<param name="gripper_max_opening_distance">1.0</param>
+						<param name="gripper_configure_xpanel">false</param>
+					</xacro:if>
 				</hardware>
 				<xacro:ar5_interfaces name=""/>

Commit message: Update gripper type references from 'ag2f90' to 'ag2f90_d' across Xacro files for consistency

File: ar5_ccs_description/xacro/grippers.xacro (robot description, xacro)
@@ -45,5 +45,5 @@
             </xacro:if>
         </xacro:if>
-        <xacro:if value="${type == 'ag2f90'}">
+        <xacro:if value="${type == 'ag2f90_d'}">
             <xacro:include filename="$(find changingtek_description)/xacro/AG2F90-C.xacro"/>
             <xacro:if value="${arm_config == 'left'}">

File: ar5_ccs_description/xacro/robot.xacro (robot description, xacro)
@@ -7,5 +7,5 @@
 	<!-- 默认值 -->
 	<xacro:property name="selected_arm_config" value="dual"/>    <!-- left, right, dual -->
-	<xacro:property name="selected_gripper_type" value=""/>     <!-- 空字符串, rg75, ag2f90 -->
+	<xacro:property name="selected_gripper_type" value=""/>     <!-- 空字符串, rg75, ag2f90_d -->
 	<!-- 解析 type 参数 - 使用显式匹配 -->
 	<!-- 处理 CCS 类型 -->
@@ -29,14 +29,14 @@
 		<xacro:property name="selected_gripper_type" value="rg75"/>
 	</xacro:if>
-	<xacro:if value="${type_arg == 'left_ag2f90'}">
+	<xacro:if value="${type_arg == 'left_ag2f90_d'}">
 		<xacro:property name="selected_arm_config" value="left"/>
-		<xacro:property name="selected_gripper_type" value="ag2f90"/>
+		<xacro:property name="selected_gripper_type" value="ag2f90_d"/>
 	</xacro:if>
-	<xacro:if value="${type_arg == 'right_ag2f90'}">
+	<xacro:if value="${type_arg == 'right_ag2f90_d'}">
 		<xacro:property name="selected_arm_config" value="right"/>
-		<xacro:property name="selected_gripper_type" value="ag2f90"/>
+		<xacro:property name="selected_gripper_type" value="ag2f90_d"/>
 	</xacro:if>
-	<xacro:if value="${type_arg == 'ag2f90'}">
-		<xacro:property name="selected_gripper_type" value="ag2f90"/>
+	<xacro:if value="${type_arg == 'ag2f90_d'}">
+		<xacro:property name="selected_gripper_type" value="ag2f90_d"/>
 	</xacro:if>
 	<!-- Include Component Macros -->

File: ar5_ccs_description/xacro/ros2_control/robot.xacro (robot description, xacro)
@@ -25,6 +25,6 @@
 						<param name="gripper_type">jodell</param>
 					</xacro:if>
-					<xacro:if value="${selected_gripper_type == 'ag2f90'}">
-						<param name="gripper_type">ag2f90d</param>
+					<xacro:if value="${selected_gripper_type == 'ag2f90_d'}">
+						<param name="gripper_type">ag2f90_d</param>
 						<param name="gripper_slave_id">1</param>
 						<param name="gripper_close_pos">9000</param>
@@ -53,6 +53,6 @@
 						<param name="gripper_type">jodell</param>
 					</xacro:if>
-					<xacro:if value="${selected_gripper_type == 'ag2f90'}">
-						<param name="gripper_type">ag2f90d</param>
+					<xacro:if value="${selected_gripper_type == 'ag2f90_d'}">
+						<param name="gripper_type">ag2f90_d</param>
 						<param name="gripper_slave_id">1</param>
 						<param name="gripper_close_pos">9000</param>
@@ -89,6 +89,6 @@
 						<param name="gripper_type">jodell</param>
 					</xacro:if>
-					<xacro:if value="${selected_gripper_type == 'ag2f90'}">
-						<param name="gripper_type">ag2f90d</param>
+					<xacro:if value="${selected_gripper_type == 'ag2f90_d'}">
+						<param name="gripper_type">ag2f90_d</param>
 						<param name="gripper_slave_id">1</param>
 						<param name="gripper_close_pos">9000</param>

File: ar5_srs_description/xacro/grippers.xacro (robot description, xacro)
@@ -45,5 +45,5 @@
             </xacro:if>
         </xacro:if>
-        <xacro:if value="${type == 'ag2f90'}">
+        <xacro:if value="${type == 'ag2f90_d'}">
             <xacro:include filename="$(find changingtek_description)/xacro/AG2F90-C.xacro"/>
             <xacro:if value="${arm_config == 'left'}">

File: ar5_srs_description/xacro/robot.xacro (robot description, xacro)
@@ -7,5 +7,5 @@
 	<!-- 默认值 -->
 	<xacro:property name="selected_arm_config" value="dual"/>    <!-- left, right, dual -->
-	<xacro:property name="selected_gripper_type" value=""/>     <!-- 空字符串, rg75, ag2f90 -->
+	<xacro:property name="selected_gripper_type" value=""/>     <!-- 空字符串, rg75, ag2f90_d -->
 	<!-- 解析 type 参数 - 使用显式匹配 -->
 	<xacro:if value="${type_arg == 'left'}">
@@ -28,14 +28,14 @@
 		<xacro:property name="selected_gripper_type" value="rg75"/>
 	</xacro:if>
-	<xacro:if value="${type_arg == 'left_ag2f90'}">
+	<xacro:if value="${type_arg == 'left_ag2f90_d'}">
 		<xacro:property name="selected_arm_config" value="left"/>
-		<xacro:property name="selected_gripper_type" value="ag2f90"/>
+		<xacro:property name="selected_gripper_type" value="ag2f90_d"/>
 	</xacro:if>
-	<xacro:if value="${type_arg == 'right_ag2f90'}">
+	<xacro:if value="${type_arg == 'right_ag2f90_d'}">
 		<xacro:property name="selected_arm_config" value="right"/>
-		<xacro:property name="selected_gripper_type" value="ag2f90"/>
+		<xacro:property name="selected_gripper_type" value="ag2f90_d"/>
 	</xacro:if>
-	<xacro:if value="${type_arg == 'ag2f90'}">
-		<xacro:property name="selected_gripper_type" value="ag2f90"/>
+	<xacro:if value="${type_arg == 'ag2f90_d'}">
+		<xacro:property name="selected_gripper_type" value="ag2f90_d"/>
 	</xacro:if>
 	<!-- Include Component Macros -->

File: ar5_srs_description/xacro/ros2_control/robot.xacro (robot description, xacro)
@@ -27,6 +27,6 @@
 						<param name="gripper_type">jodell</param>
 					</xacro:if>
-					<xacro:if value="${selected_gripper_type == 'ag2f90'}">
-						<param name="gripper_type">ag2f90d</param>
+					<xacro:if value="${selected_gripper_type == 'ag2f90_d'}">
+						<param name="gripper_type">ag2f90_d</param>
 						<param name="gripper_slave_id">1</param>
 						<param name="gripper_close_pos">9000</param>
@@ -57,6 +57,6 @@
 						<param name="gripper_type">jodell</param>
 					</xacro:if>
-					<xacro:if value="${selected_gripper_type == 'ag2f90'}">
-						<param name="gripper_type">ag2f90d</param>
+					<xacro:if value="${selected_gripper_type == 'ag2f90_d'}">
+						<param name="gripper_type">ag2f90_d</param>
 						<param name="gripper_slave_id">1</param>
 						<param name="gripper_close_pos">9000</param>
@@ -97,6 +97,6 @@
 						<param name="gripper_type">jodell</param>
 					</xacro:if>
-					<xacro:if value="${selected_gripper_type == 'ag2f90'}">
-						<param name="gripper_type">ag2f90d</param>
+					<xacro:if value="${selected_gripper_type == 'ag2f90_d'}">
+						<param name="gripper_type">ag2f90_d</param>
 						<param name="gripper_slave_id">1</param>
 						<param name="gripper_close_pos">9000</param>
