Commit message: Add linkerhand support in robot.xacro and related files

File: ar5_ccs_description/xacro/eefs.xacro (robot description, xacro)
@@ -4,4 +4,5 @@
     <xacro:include filename="$(find jodell_description)/xacro/RG75-300.xacro"/>
     <xacro:include filename="$(find changingtek_description)/xacro/AG2F90-C.xacro"/>
+    <xacro:include filename="$(find linkerhand_description)/xacro/l6.xacro"/>
     <xacro:macro name="Ocs2SideEefFrame" params="side parent_link">
         <link name="${side}_eef"/>
@@ -32,4 +33,12 @@
             </joint>
         </xacro:if>
+        <xacro:if value="${hand_type == 'linkerhand_l6'}">
+            <xacro:LinkerHandL6 name="${side}_hand" direction="${1 if side == 'left' else -1}"
+                                use_flange="true" fixed_joints="${eef_fixed_joints}"/>
+            <joint name="${side}_hand_base_joint" type="fixed">
+                <parent link="${side}_tcp"/>
+                <child link="${side}_hand_flange"/>
+            </joint>
+        </xacro:if>
     </xacro:macro>
     <xacro:macro name="EndEffectors"

File: ar5_ccs_description/xacro/robot.xacro (robot description, xacro)
@@ -106,3 +106,15 @@
 		<xacro:Grippers type="${selected_gripper_type}" arm_config="${selected_arm_config}"/>
 	</xacro:if>
+	<xacro:if value="${selected_arm_config != 'dual'}">
+		<xacro:include filename="$(find linkerhand_description)/xacro/l6.xacro"/>
+		<xacro:if value="${(left_hand_type if selected_arm_config == 'left' else right_hand_type) == 'linkerhand_l6'}">
+			<xacro:LinkerHandL6 name="${'left_hand' if selected_arm_config == 'left' else 'right_hand'}"
+							direction="${1 if selected_arm_config == 'left' else -1}"
+							use_flange="true" fixed_joints="$(arg eef_fixed_joints)"/>
+			<joint name="hand_base_joint" type="fixed">
+				<parent link="tcp"/>
+				<child link="${'left_hand_flange' if selected_arm_config == 'left' else 'right_hand_flange'}"/>
+			</joint>
+		</xacro:if>
+	</xacro:if>
 </robot>

File: ar5_ccs_description/xacro/ros2_control/robot.xacro (robot description, xacro)
@@ -28,4 +28,5 @@
 	<xacro:include filename="$(find ar5_ccs_description)/xacro/robot.xacro"/>
 	<xacro:include filename="$(find ar5_ccs_description)/xacro/ros2_control/interfaces.xacro"/>
+	<xacro:include filename="$(find linkerhand_description)/xacro/ros2_control/o6.xacro"/>
 	<!--
 		Default Rokae tool load table by gripper/pad.
@@ -128,5 +129,5 @@
 						<param name="left_tool_velocity">1.0</param>
 					</xacro:if>
-					<xacro:if value="${left_gripper_type in ('ag2f90_c', 'ag2f90_d')}">
+						<xacro:if value="${left_gripper_type in ('ag2f90_c', 'ag2f90_d')}">
 						<param name="gripper_type">${left_gripper_type}</param>
 						<param name="gripper_slave_id">1</param>
@@ -136,5 +137,12 @@
 						<param name="left_tool_torque">1.0</param>
 						<param name="left_tool_velocity">1.0</param>
-					</xacro:if>
+						</xacro:if>
+						<xacro:if value="${left_hand_type == 'linkerhand_l6'}">
+							<param name="gripper_type">linkerhand_l6</param>
+							<param name="hand_slave_id">40</param>
+							<param name="hand_configure_xpanel">false</param>
+							<param name="left_tool_torque">1.0</param>
+							<param name="left_tool_velocity">1.0</param>
+						</xacro:if>
 					<xacro:if value="${left_gripper_type != ''}">
 						<xacro:rokae_tool_load_params_with_override side="left" gripper_type="${left_gripper_type}" gripper_pad="${left_gripper_pad}"
@@ -143,4 +151,7 @@
 				</hardware>
 				<xacro:ar5_interfaces name="left"/>
+				<xacro:if value="${left_hand_type == 'linkerhand_l6'}">
+					<xacro:linkerhand_o6_interfaces name="left_hand"/>
+				</xacro:if>
 				<xacro:if value="${left_gripper_type != ''}">
 					<joint name="left_gripper_joint">
@@ -171,5 +182,5 @@
 						<param name="right_tool_velocity">1.0</param>
 					</xacro:if>
-					<xacro:if value="${right_gripper_type in ('ag2f90_c', 'ag2f90_d')}">
+						<xacro:if value="${right_gripper_type in ('ag2f90_c', 'ag2f90_d')}">
 						<param name="gripper_type">${right_gripper_type}</param>
 						<param name="gripper_slave_id">1</param>
@@ -179,5 +190,12 @@
 						<param name="right_tool_torque">1.0</param>
 						<param name="right_tool_velocity">1.0</param>
-					</xacro:if>
+						</xacro:if>
+						<xacro:if value="${right_hand_type == 'linkerhand_l6'}">
+							<param name="gripper_type">linkerhand_l6</param>
+							<param name="hand_slave_id">39</param>
+							<param name="hand_configure_xpanel">false</param>
+							<param name="right_tool_torque">1.0</param>
+							<param name="right_tool_velocity">1.0</param>
+						</xacro:if>
 					<xacro:if value="${right_gripper_type != ''}">
 						<xacro:rokae_tool_load_params_with_override side="right" gripper_type="${right_gripper_type}" gripper_pad="${right_gripper_pad}"
@@ -186,4 +204,7 @@
 				</hardware>
 				<xacro:ar5_interfaces name="right"/>
+				<xacro:if value="${right_hand_type == 'linkerhand_l6'}">
+					<xacro:linkerhand_o6_interfaces name="right_hand"/>
+				</xacro:if>
 				<xacro:if value="${right_gripper_type != ''}">
 					<joint name="right_gripper_joint">
@@ -227,5 +248,5 @@
 						<param name="${'left' if selected_arm_config == 'left' else 'right'}_tool_velocity">1.0</param>
 					</xacro:if>
-					<xacro:if value="${selected_gripper_type in ('ag2f90_c', 'ag2f90_d')}">
+						<xacro:if value="${selected_gripper_type in ('ag2f90_c', 'ag2f90_d')}">
 						<param name="gripper_type">${selected_gripper_type}</param>
 						<param name="gripper_slave_id">1</param>
@@ -235,5 +256,12 @@
 						<param name="${'left' if selected_arm_config == 'left' else 'right'}_tool_torque">1.0</param>
 						<param name="${'left' if selected_arm_config == 'left' else 'right'}_tool_velocity">1.0</param>
-					</xacro:if>
+						</xacro:if>
+						<xacro:if value="${(left_hand_type if selected_arm_config == 'left' else right_hand_type) == 'linkerhand_l6'}">
+							<param name="gripper_type">linkerhand_l6</param>
+							<param name="hand_slave_id">${40 if selected_arm_config == 'left' else 39}</param>
+							<param name="hand_configure_xpanel">false</param>
+							<param name="${'left' if selected_arm_config == 'left' else 'right'}_tool_torque">1.0</param>
+							<param name="${'left' if selected_arm_config == 'left' else 'right'}_tool_velocity">1.0</param>
+						</xacro:if>
 					<xacro:if value="${selected_gripper_type != ''}">
 						<xacro:rokae_tool_load_params_with_override side="${'left' if selected_arm_config == 'left' else 'right'}" gripper_type="${selected_gripper_type}" gripper_pad="${selected_gripper_pad}"
@@ -244,4 +272,7 @@
 				</hardware>
 				<xacro:ar5_interfaces name=""/>
+				<xacro:if value="${(left_hand_type if selected_arm_config == 'left' else right_hand_type) == 'linkerhand_l6'}">
+					<xacro:linkerhand_o6_interfaces name="${'left_hand' if selected_arm_config == 'left' else 'right_hand'}"/>
+				</xacro:if>
 				<xacro:if value="${selected_gripper_type != ''}">
 					<joint name="gripper_joint">
@@ -274,7 +305,13 @@
 				</xacro:if>
 			</hardware>
-			<xacro:if value="${selected_arm_config == 'dual'}">
-				<xacro:ar5_interfaces name="left"/>
-				<xacro:ar5_interfaces name="right"/>
+				<xacro:if value="${selected_arm_config == 'dual'}">
+					<xacro:ar5_interfaces name="left"/>
+					<xacro:ar5_interfaces name="right"/>
+					<xacro:if value="${left_hand_type == 'linkerhand_l6'}">
+						<xacro:linkerhand_o6_interfaces name="left_hand"/>
+					</xacro:if>
+					<xacro:if value="${right_hand_type == 'linkerhand_l6'}">
+						<xacro:linkerhand_o6_interfaces name="right_hand"/>
+					</xacro:if>
 				<xacro:if value="${left_gripper_type != ''}">
 					<joint name="left_gripper_joint">
@@ -298,6 +335,9 @@
 				</xacro:if>
 			</xacro:if>
-			<xacro:unless value="${selected_arm_config == 'dual'}">
-				<xacro:ar5_interfaces name=""/>
+				<xacro:unless value="${selected_arm_config == 'dual'}">
+					<xacro:ar5_interfaces name=""/>
+					<xacro:if value="${(left_hand_type if selected_arm_config == 'left' else right_hand_type) == 'linkerhand_l6'}">
+						<xacro:linkerhand_o6_interfaces name="${'left_hand' if selected_arm_config == 'left' else 'right_hand'}"/>
+					</xacro:if>
 				<xacro:if value="${selected_gripper_type != ''}">
 					<joint name="gripper_joint">

Commit message: Add origin element to hand base joints for left and right configurations

File: ar5_ccs_description/xacro/eefs.xacro (robot description, xacro)
@@ -37,4 +37,5 @@
                                 use_flange="true" fixed_joints="${eef_fixed_joints}"/>
             <joint name="${side}_hand_base_joint" type="fixed">
+                <origin rpy="0 0 ${3.141592653589793 if side == 'left' else 0}"/>
                 <parent link="${side}_tcp"/>
                 <child link="${side}_hand_flange"/>

File: ar5_ccs_description/xacro/robot.xacro (robot description, xacro)
@@ -113,4 +113,5 @@
 							use_flange="true" fixed_joints="$(arg eef_fixed_joints)"/>
 			<joint name="hand_base_joint" type="fixed">
+				<origin rpy="0 0 ${3.141592653589793 if selected_arm_config == 'left' else 0}"/>
 				<parent link="tcp"/>
 				<child link="${'left_hand_flange' if selected_arm_config == 'left' else 'right_hand_flange'}"/>
