Commit message: add rviz config

File: ar5_ccs_description/xacro/eefs.xacro (robot description, xacro)
@@ -72,6 +72,5 @@
             <xacro:unless value="${hand_type == 'linkerhand_o6' or hand_type == 'linkerhand_o7' or hand_type == 'linkerhand_l6'}">
                 <xacro:if value="${gripper_type == 'ag2f90_c' or gripper_type == 'ag2f90_d'}">
-                    <xacro:property name="ag2f90_pad" value="${'none' if gripper_type == 'ag2f90_d' else gripper_pad}"/>
-                    <xacro:AG2F90-C name="${side}" use_flange="true" pad="${ag2f90_pad}" kinematic_only="true"/>
+                    <xacro:AG2F90-C name="${side}" use_flange="true" pad="${gripper_pad}" kinematic_only="true"/>
                     <joint name="${side}_gripper_base_joint" type="fixed">
                         <origin xyz="0 0 0"/>
@@ -122,6 +121,5 @@
             </xacro:if>
             <xacro:if value="${gripper_type == 'ag2f90_c' or gripper_type == 'ag2f90_d'}">
-                <xacro:property name="ag2f90_pad" value="${'none' if gripper_type == 'ag2f90_d' else gripper_pad}"/>
-                <xacro:AG2F90-C name="${side}" use_flange="true" pad="${ag2f90_pad}" kinematic_only="false"/>
+                <xacro:AG2F90-C name="${side}" use_flange="true" pad="${gripper_pad}" kinematic_only="false"/>
                 <joint name="${side}_gripper_base_joint" type="fixed">
                     <origin xyz="0 0 0"/>

File: ar5_srs_description/xacro/arm_srs.xacro (robot description, xacro)
@@ -13,5 +13,5 @@
 			<visual>
 				<geometry>
-					<mesh filename="package://ar5_srs_description/meshes/base.glb" scale="1 ${direction} 1"/>
+					<mesh filename="file://$(find ar5_srs_description)/meshes/base.glb" scale="1 ${direction} 1"/>
 				</geometry>
 			</visual>

Commit message: add xhand option

File: ar5_ccs_description/xacro/eefs.xacro (robot description, xacro)
@@ -96,9 +96,14 @@
         </xacro:if>
         <xacro:if value="${hand_type == 'xhand1'}">
-            <xacro:XHand1 name="${side}_hand" direction="${1 if side == 'left' else -1}" fixed_joints="${eef_fixed_joints}"/>
-            <joint name="${side}_hand_base_joint" type="fixed">
-                <origin rpy="0 0 ${PI}"/>
-                <parent link="${side}_tcp"/>
-                <child link="${side}_hand_hand_base"/>
+            <xacro:XHand1 name="${side}_hand" direction="${1 if side == 'left' else -1}" use_flange="true" fixed_joints="${eef_fixed_joints}"/>
+            <joint name="${side}_hand_base_joint" type="fixed">
+                <xacro:if value="${side == 'left'}">
+                    <origin xyz="0 0 0.0045" rpy="0 0 ${PI/2}"/>
+                </xacro:if>
+                <xacro:if value="${side == 'right'}">
+                    <origin xyz="0 0 0.0045" rpy="0 0 ${-PI/2}"/>
+                </xacro:if>
+                <parent link="${side}_tcp"/>
+                <child link="${side}_hand_flange"/>
             </joint>
         </xacro:if>
@@ -111,5 +116,12 @@
             </joint>
         </xacro:if>
-        <xacro:if value="${hand_type in ('linkerhand_o6', 'linkerhand_l6', 'linkerhand_o7', 'freedom_v1', 'freedom_v2', 'inspire_e2', 'inspire_f2', 'xhand1', 'theohand_std16a')}">
+        <xacro:if value="${hand_type == 'xhand1'}">
+            <link name="${side}_eef"/>
+            <joint name="${side}_eef_joint" type="fixed">
+                <parent link="${side}_hand_hand_ee_link"/>
+                <child link="${side}_eef"/>
+            </joint>
+        </xacro:if>
+        <xacro:if value="${hand_type in ('linkerhand_o6', 'linkerhand_l6', 'linkerhand_o7', 'freedom_v1', 'freedom_v2', 'inspire_e2', 'inspire_f2', 'theohand_std16a')}">
             <link name="${side}_eef"/>
             <joint name="${side}_eef_joint" type="fixed">

File: ar5_ccs_description/xacro/ros2_control/end_effector_interfaces.xacro (robot description, xacro)
@@ -8,4 +8,5 @@
     <xacro:include filename="$(find linkerhand_description)/xacro/ros2_control/o6.xacro"/>
     <xacro:include filename="$(find linkerhand_description)/xacro/ros2_control/o7.xacro"/>
+    <xacro:include filename="$(find xhand1_description)/xacro/ros2_control/side_systems.xacro"/>
     <xacro:macro name="side_gripper_joint" params="side">
         <joint name="${side}_gripper_joint">
@@ -41,4 +42,7 @@
         <xacro:if value="${hand_type == 'linkerhand_o7'}">
             <xacro:linkerhand_o7_interfaces name="${side}_hand"/>
+        </xacro:if>
+        <xacro:if value="${hand_type == 'xhand1'}">
+            <xacro:xhand1_interfaces name="${side}_hand"/>
         </xacro:if>
     </xacro:macro>
