Commit message: update

File: ar5_ccs_description/xacro/robot.xacro (robot description, xacro)
@@ -2,9 +2,9 @@
 <robot name="AR5_CCS" xmlns:xacro="http://www.ros.org/wiki/xacro">
 	<xacro:arg name="collider" default="convex"/>
-	<xacro:arg name="type" default="left"/>
+	<xacro:arg name="type" default="dual"/>
 	<!-- 拆解 type 参数为三个独立属性 -->
 	<xacro:property name="type_arg" value="$(arg type)"/>
 	<!-- 默认值 -->
-	<xacro:property name="selected_arm_config" value="left"/>    <!-- left, right, dual -->
+	<xacro:property name="selected_arm_config" value="dual"/>    <!-- left, right, dual -->
 	<xacro:property name="selected_gripper_type" value=""/>     <!-- 空字符串或 rg75 -->
 	<!-- 解析 type 参数 - 使用显式匹配 -->
@@ -18,8 +18,4 @@
 		<xacro:property name="selected_gripper_type" value=""/>
 	</xacro:if>
-	<xacro:if value="${type_arg == 'dual'}">
-		<xacro:property name="selected_arm_config" value="dual"/>
-		<xacro:property name="selected_gripper_type" value=""/>
-	</xacro:if>
 	<xacro:if value="${type_arg == 'left_rg75'}">
 		<xacro:property name="selected_arm_config" value="left"/>
@@ -30,6 +26,5 @@
 		<xacro:property name="selected_gripper_type" value="rg75"/>
 	</xacro:if>
-	<xacro:if value="${type_arg == 'dual_rg75'}">
-		<xacro:property name="selected_arm_config" value="dual"/>
+	<xacro:if value="${type_arg == 'rg75'}">
 		<xacro:property name="selected_gripper_type" value="rg75"/>
 	</xacro:if>

File: ar5_srs_description/xacro/robot.xacro (robot description, xacro)
@@ -2,9 +2,9 @@
 <robot name="AR5_SRS" xmlns:xacro="http://www.ros.org/wiki/xacro">
 	<xacro:arg name="collider" default="convex"/>
-	<xacro:arg name="type" default="left"/>
+	<xacro:arg name="type" default="dual"/>
 	<!-- 拆解 type 参数为三个独立属性 -->
 	<xacro:property name="type_arg" value="$(arg type)"/>
 	<!-- 默认值 -->
-	<xacro:property name="selected_arm_config" value="left"/>    <!-- left, right, dual -->
+	<xacro:property name="selected_arm_config" value="dual"/>    <!-- left, right, dual -->
 	<xacro:property name="selected_gripper_type" value=""/>     <!-- 空字符串或 rg75 -->
 	<!-- 解析 type 参数 - 使用显式匹配 -->
@@ -17,8 +17,4 @@
 		<xacro:property name="selected_gripper_type" value=""/>
 	</xacro:if>
-	<xacro:if value="${type_arg == 'dual'}">
-		<xacro:property name="selected_arm_config" value="dual"/>
-		<xacro:property name="selected_gripper_type" value=""/>
-	</xacro:if>
 	<xacro:if value="${type_arg == 'left_rg75'}">
 		<xacro:property name="selected_arm_config" value="left"/>
@@ -29,6 +25,5 @@
 		<xacro:property name="selected_gripper_type" value="rg75"/>
 	</xacro:if>
-	<xacro:if value="${type_arg == 'dual_rg75'}">
-		<xacro:property name="selected_arm_config" value="dual"/>
+	<xacro:if value="${type_arg == 'rg75'}">
 		<xacro:property name="selected_gripper_type" value="rg75"/>
 	</xacro:if>

File: ar5_srs_description/xacro/ros2_control/robot.xacro (robot description, xacro)
@@ -140,5 +140,5 @@
 			<plugin filename="gz_ros2_control-system" name="gz_ros2_control::GazeboSimROS2ControlPlugin">
 				<xacro:if value="${selected_arm_config == 'left'}">
-					<parameters>$(find ar5_srs_description)/config/ros2_control/ros2_controllers.yaml</parameters>
+					<parameters>$(find ar5_srs_description)/config/ros2_control/left.yaml</parameters>
 				</xacro:if>
 				<xacro:if value="${selected_arm_config == 'right'}">
@@ -146,5 +146,5 @@
 				</xacro:if>
 				<xacro:if value="${selected_arm_config == 'dual'}">
-					<parameters>$(find ar5_srs_description)/config/ros2_control/dual.yaml</parameters>
+					<parameters>$(find ar5_srs_description)/config/ros2_control/ros2_controllers.yaml</parameters>
 				</xacro:if>
 			</plugin>

Commit message: Refactor AR5 CCS URDF and Xacro files for end effector configuration
- Deleted outdated URDF files for right arm configurations: ar5_ccs_right.urdf and ar5_ccs_right_rg75.urdf.
- Introduced new Xacro files: eef_type_resolver.xacro and eefs.xacro to manage end effector types and configurations.
- Updated robot.xacro to support separate left and right end effector types, enhancing configurability for dual-arm setups.
- Modified ros2_control/robot.xacro to accommodate changes in gripper type handling for both arms, ensuring proper integration with control interfaces.

File: ar5_ccs_description/xacro/robot.xacro (robot description, xacro)
@@ -3,6 +3,11 @@
 	<xacro:arg name="collider" default="convex"/>
 	<xacro:arg name="type" default="dual"/>
+	<xacro:arg name="left_type" default=""/>
+	<xacro:arg name="right_type" default=""/>
+	<xacro:arg name="eef_fixed_joints" default="false"/>
 	<!-- 拆解 type 参数为三个独立属性 -->
 	<xacro:property name="type_arg" value="$(arg type)"/>
+	<xacro:property name="left_type_arg" value="$(arg left_type)"/>
+	<xacro:property name="right_type_arg" value="$(arg right_type)"/>
 	<!-- 默认值 -->
 	<xacro:property name="selected_arm_config" value="dual"/>    <!-- left, right, dual -->
@@ -39,4 +44,13 @@
 	<xacro:if value="${type_arg == 'ag2f90_d'}">
 		<xacro:property name="selected_gripper_type" value="ag2f90_d"/>
+	</xacro:if>
+	<!-- 双臂末端支持 left_type/right_type；未指定时沿用对称 type。 -->
+	<xacro:property name="effective_left_type" value="${left_type_arg if left_type_arg != '' else type_arg}"/>
+	<xacro:property name="effective_right_type" value="${right_type_arg if right_type_arg != '' else type_arg}"/>
+	<xacro:include filename="$(find ar5_ccs_description)/xacro/eef_type_resolver.xacro"/>
+	<xacro:set_side_eef_types side="left" type_key="${effective_left_type}"/>
+	<xacro:set_side_eef_types side="right" type_key="${effective_right_type}"/>
+	<xacro:if value="${selected_arm_config == 'dual'}">
+		<xacro:property name="selected_gripper_type" value="${left_gripper_type if left_gripper_type == right_gripper_type else ''}"/>
 	</xacro:if>
 	<!-- Include Component Macros -->
@@ -76,7 +90,16 @@
 		<xacro:Arm name="left" collider="$(arg collider)" direction="1"/>
 		<xacro:Arm name="right" collider="$(arg collider)" direction="-1"/>
+		<xacro:include filename="$(find ar5_ccs_description)/xacro/eefs.xacro"/>
+		<xacro:EndEffectors
+			eef_fixed_joints="$(arg eef_fixed_joints)"
+			left_hand_type="${left_hand_type}"
+			left_gripper_type="${left_gripper_type}"
+			left_gripper_pad="${left_gripper_pad}"
+			right_hand_type="${right_hand_type}"
+			right_gripper_type="${right_gripper_type}"
+			right_gripper_pad="${right_gripper_pad}"/>
 	</xacro:if>
-	<!-- 根据 gripper_type 添加夹爪 -->
-	<xacro:if value="${selected_gripper_type != ''}">
+	<!-- 单臂配置沿用旧夹爪宏。双臂末端由 EndEffectors 按侧生成。 -->
+	<xacro:if value="${selected_arm_config != 'dual' and selected_gripper_type != ''}">
 		<xacro:Grippers type="${selected_gripper_type}" arm_config="${selected_arm_config}"/>
 	</xacro:if>

File: ar5_ccs_description/xacro/ros2_control/robot.xacro (robot description, xacro)
@@ -22,8 +22,8 @@
 					<param name="joint_impedance">200,200,200,200,20,20,20</param>
 					<param name="local_ip">192.168.1.233</param>
-					<xacro:if value="${selected_gripper_type == 'rg75'}">
+					<xacro:if value="${left_gripper_type == 'rg75'}">
 						<param name="gripper_type">jodell</param>
 					</xacro:if>
-					<xacro:if value="${selected_gripper_type == 'ag2f90_d'}">
+					<xacro:if value="${left_gripper_type == 'ag2f90_d'}">
 						<param name="gripper_type">ag2f90_d</param>
 						<param name="gripper_slave_id">1</param>
@@ -34,5 +34,5 @@
 				</hardware>
 				<xacro:ar5_interfaces name="left"/>
-				<xacro:if value="${selected_gripper_type != ''}">
+				<xacro:if value="${left_gripper_type != ''}">
 					<joint name="left_gripper_joint">
 						<command_interface name="position"/>
@@ -40,4 +40,6 @@
 							<param name="initial_value">0</param>
 						</state_interface>
+						<state_interface name="velocity"/>
+						<state_interface name="effort"/>
 					</joint>
 				</xacro:if>
@@ -50,8 +52,8 @@
 					<param name="joint_impedance">200,200,200,200,20,20,20</param>
 					<param name="local_ip">192.168.1.233</param>
-					<xacro:if value="${selected_gripper_type == 'rg75'}">
+					<xacro:if value="${right_gripper_type == 'rg75'}">
 						<param name="gripper_type">jodell</param>
 					</xacro:if>
-					<xacro:if value="${selected_gripper_type == 'ag2f90_d'}">
+					<xacro:if value="${right_gripper_type == 'ag2f90_d'}">
 						<param name="gripper_type">ag2f90_d</param>
 						<param name="gripper_slave_id">1</param>
@@ -62,5 +64,5 @@
 				</hardware>
 				<xacro:ar5_interfaces name="right"/>
-				<xacro:if value="${selected_gripper_type != ''}">
+				<xacro:if value="${right_gripper_type != ''}">
 					<joint name="right_gripper_joint">
 						<command_interface name="position"/>
@@ -68,4 +70,6 @@
 							<param name="initial_value">0</param>
 						</state_interface>
+						<state_interface name="velocity"/>
+						<state_interface name="effort"/>
 					</joint>
 				</xacro:if>
@@ -104,4 +108,6 @@
 							<param name="initial_value">0</param>
 						</state_interface>
+						<state_interface name="velocity"/>
+						<state_interface name="effort"/>
 					</joint>
 				</xacro:if>
@@ -129,5 +135,5 @@
 				<xacro:ar5_interfaces name="left"/>
 				<xacro:ar5_interfaces name="right"/>
-				<xacro:if value="${selected_gripper_type != ''}">
+				<xacro:if value="${left_gripper_type != ''}">
 					<joint name="left_gripper_joint">
 						<command_interface name="position"/>
@@ -135,5 +141,9 @@
 							<param name="initial_value">0</param>
 						</state_interface>
+						<state_interface name="velocity"/>
+						<state_interface name="effort"/>
 					</joint>
+				</xacro:if>
+				<xacro:if value="${right_gripper_type != ''}">
 					<joint name="right_gripper_joint">
 						<command_interface name="position"/>
@@ -141,4 +151,6 @@
 							<param name="initial_value">0</param>
 						</state_interface>
+						<state_interface name="velocity"/>
+						<state_interface name="effort"/>
 					</joint>
 				</xacro:if>
@@ -152,4 +164,6 @@
 							<param name="initial_value">0</param>
 						</state_interface>
+						<state_interface name="velocity"/>
+						<state_interface name="effort"/>
 					</joint>
 				</xacro:if>

Commit message: Update tool load parameters and add gripper pad selection for AR5 robot

File: ar5_ccs_description/xacro/robot.xacro (robot description, xacro)
@@ -13,4 +13,5 @@
 	<xacro:property name="selected_arm_config" value="dual"/>    <!-- left, right, dual -->
 	<xacro:property name="selected_gripper_type" value=""/>     <!-- 空字符串, rg75, ag2f90_d -->
+	<xacro:property name="selected_gripper_pad" value="default"/>
 	<!-- 解析 type 参数 - 使用显式匹配 -->
 	<!-- 处理 CCS 类型 -->
@@ -53,4 +54,5 @@
 	<xacro:if value="${selected_arm_config == 'dual'}">
 		<xacro:property name="selected_gripper_type" value="${left_gripper_type if left_gripper_type == right_gripper_type else ''}"/>
+		<xacro:property name="selected_gripper_pad" value="${left_gripper_pad if left_gripper_pad == right_gripper_pad else 'default'}"/>
 	</xacro:if>
 	<!-- Include Component Macros -->

File: ar5_ccs_description/xacro/ros2_control/robot.xacro (robot description, xacro)
@@ -21,4 +21,71 @@
 	<xacro:include filename="$(find ar5_ccs_description)/xacro/robot.xacro"/>
 	<xacro:include filename="$(find ar5_ccs_description)/xacro/ros2_control/interfaces.xacro"/>
+	<!--
+		Default Rokae tool load table by gripper/pad.
+		All values are intentionally zero placeholders. Fill the real values here
+		when the measured mass/CoG/inertia for each end effector is available.
+	-->
+	<xacro:macro name="rokae_tool_load_params" params="side gripper_type gripper_pad">
+		<!-- Left RG75, default pad: TODO fill measured load. -->
+		<xacro:if value="${side == 'left' and gripper_type == 'rg75' and gripper_pad != 'heavy_carry'}">
+			<param name="load_mass">0.0</param>
+			<param name="load_cog">[0.0, 0.0, 0.0]</param>
+			<param name="load_inertia">[0.0, 0.0, 0.0]</param>
+		</xacro:if>
+		<!-- Left RG75, heavy_carry pad: TODO fill measured load. -->
+		<xacro:if value="${side == 'left' and gripper_type == 'rg75' and gripper_pad == 'heavy_carry'}">
+			<param name="load_mass">0.0</param>
+			<param name="load_cog">[0.0, 0.0, 0.0]</param>
+			<param name="load_inertia">[0.0, 0.0, 0.0]</param>
+		</xacro:if>
+		<!-- Left AG2F90-C, default pad: TODO fill measured load. -->
+		<xacro:if value="${side == 'left' and gripper_type == 'ag2f90_c' and gripper_pad != 'soft'}">
+			<param name="load_mass">0.0</param>
+			<param name="load_cog">[0.0, 0.0, 0.0]</param>
+			<param name="load_inertia">[0.0, 0.0, 0.0]</param>
+		</xacro:if>
+		<!-- Left AG2F90-C, soft pad: TODO fill measured load. -->
+		<xacro:if value="${side == 'left' and gripper_type == 'ag2f90_c' and gripper_pad == 'soft'}">
+			<param name="load_mass">0.0</param>
+			<param name="load_cog">[0.0, 0.0, 0.0]</param>
+			<param name="load_inertia">[0.0, 0.0, 0.0]</param>
+		</xacro:if>
+		<!-- Left AG2F90-D, pad is ignored by the model: TODO fill measured load. -->
+		<xacro:if value="${side == 'left' and gripper_type == 'ag2f90_d'}">
+			<param name="load_mass">0.0</param>
+			<param name="load_cog">[0.0, 0.0, 0.0]</param>
+			<param name="load_inertia">[0.0, 0.0, 0.0]</param>
+		</xacro:if>
+		<!-- Right RG75, default pad. -->
+		<xacro:if value="${side == 'right' and gripper_type == 'rg75' and gripper_pad != 'heavy_carry'}">
+			<param name="load_mass">1.62</param>
+			<param name="load_cog">[-0.0014285, 0.000579, 0.10439]</param>
+			<param name="load_inertia">[0.04874, 0.001, 0.001936]</param>
+		</xacro:if>
+		<!-- Right RG75, heavy_carry pad: TODO fill measured load. -->
+		<xacro:if value="${side == 'right' and gripper_type == 'rg75' and gripper_pad == 'heavy_carry'}">
+			<param name="load_mass">0.0</param>
+			<param name="load_cog">[0.0, 0.0, 0.0]</param>
+			<param name="load_inertia">[0.0, 0.0, 0.0]</param>
+		</xacro:if>
+		<!-- Right AG2F90-C, default pad: TODO fill measured load. -->
+		<xacro:if value="${side == 'right' and gripper_type == 'ag2f90_c' and gripper_pad != 'soft'}">
+			<param name="load_mass">0.0</param>
+			<param name="load_cog">[0.0, 0.0, 0.0]</param>
+			<param name="load_inertia">[0.0, 0.0, 0.0]</param>
+		</xacro:if>
+		<!-- Right AG2F90-C, soft pad: TODO fill measured load. -->
+		<xacro:if value="${side == 'right' and gripper_type == 'ag2f90_c' and gripper_pad == 'soft'}">
+			<param name="load_mass">0.0</param>
+			<param name="load_cog">[0.0, 0.0, 0.0]</param>
+			<param name="load_inertia">[0.0, 0.0, 0.0]</param>
+		</xacro:if>
+		<!-- Right AG2F90-D, pad is ignored by the model: TODO fill measured load. -->
+		<xacro:if value="${side == 'right' and gripper_type == 'ag2f90_d'}">
+			<param name="load_mass">0.0</param>
+			<param name="load_cog">[0.0, 0.0, 0.0]</param>
+			<param name="load_inertia">[0.0, 0.0, 0.0]</param>
+		</xacro:if>
+	</xacro:macro>
 	<!-- 使用 robot.xacro 中已定义的 property 来判断 -->
 	<!-- selected_arm_config: left, right, dual -->
@@ -57,4 +124,7 @@
 						<param name="left_tool_velocity">1.0</param>
 					</xacro:if>
+					<xacro:if value="${left_gripper_type != ''}">
+						<xacro:rokae_tool_load_params side="left" gripper_type="${left_gripper_type}" gripper_pad="${left_gripper_pad}"/>
+					</xacro:if>
 				</hardware>
 				<xacro:ar5_interfaces name="left"/>
@@ -101,4 +171,7 @@
 						<param name="right_tool_velocity">1.0</param>
 					</xacro:if>
+					<xacro:if value="${right_gripper_type != ''}">
+						<xacro:rokae_tool_load_params side="right" gripper_type="${right_gripper_type}" gripper_pad="${right_gripper_pad}"/>
+					</xacro:if>
 				</hardware>
 				<xacro:ar5_interfaces name="right"/>
@@ -158,4 +231,7 @@
 						<param name="${'left' if selected_arm_config == 'left' else 'right'}_tool_velocity">1.0</param>
 					</xacro:if>
+					<xacro:if value="${selected_gripper_type != ''}">
+						<xacro:rokae_tool_load_params side="${'left' if selected_arm_config == 'left' else 'right'}" gripper_type="${selected_gripper_type}" gripper_pad="${selected_gripper_pad}"/>
+					</xacro:if>
 				</hardware>
 				<xacro:ar5_interfaces name=""/>

Commit message: Update end-effector frames and joint origins in robot configuration

File: ar5_ccs_description/xacro/robot.xacro (robot description, xacro)
@@ -83,10 +83,10 @@
 			<parent link="arm_base"/>
 			<child link="left_base_link"/>
-			<origin xyz="0.0 0.12 0" rpy="-1.57 1.57 0"/>
+			<origin xyz="0.0 0.062 0" rpy="-1.57 1.57 0"/>
 		</joint>
 		<joint name="right_arm_mount" type="fixed">
 			<parent link="arm_base"/>
 			<child link="right_base_link"/>
-			<origin xyz="0.0 -0.12 0" rpy="1.57 1.57 0"/>
+			<origin xyz="0.0 -0.062 0" rpy="1.57 1.57 0"/>
 		</joint>
 		<xacro:Arm name="left" collider="$(arg collider)" direction="1"/>

Commit message: 修改 ar5_ccs 的 arm base 碰撞体

File: ar5_ccs_description/xacro/robot.xacro (robot description, xacro)
@@ -70,7 +70,7 @@
 		<link name="arm_base">
 			<collision>
-				<origin xyz="0.0091 0 -0.086"/>
+				<origin xyz="0.0091 0 -0.096"/>
 				<geometry>
-					<box size="0.2509 0.35 0.5029"/>
+					<box size="0.33 0.30 0.5029"/>
 				</geometry>
 			</collision>
