Commit message: Fix collision geometry and position for arm_base in AR5_CCS and AR5_SRS

File: ar5_ccs_description/xacro/robot.xacro (robot description, xacro)
@@ -73,7 +73,7 @@
 		<link name="arm_base">
 			<collision>
-				<origin xyz="0.0091 0 -0.2"/>
+				<origin xyz="0.0091 0 -0.25"/>
 				<geometry>
-					<box size="0.33 0.30 0.5029"/>
+					<box size="0.2000 0.3 0.4029"/>
 				</geometry>
 			</collision>

File: ar5_srs_description/xacro/robot.xacro (robot description, xacro)
@@ -53,7 +53,7 @@
 		<link name="arm_base">
 			<collision>
-				<origin xyz="0.0091 0 -0.2"/>
+				<origin xyz="0.0091 0 -0.25"/>
 				<geometry>
-					<box size="0.2509 0.35 0.5029"/>
+					<box size="0.2000 0.3 0.4029"/>
 				</geometry>
 			</collision>

Commit message: Add TCP offset arguments and joints for AR5_CCS and AR5_SRS

File: ar5_ccs_description/xacro/robot.xacro (robot description, xacro)
@@ -8,4 +8,8 @@
 	<xacro:arg name="right_type" default=""/>
 	<xacro:arg name="eef_fixed_joints" default="false"/>
+	<xacro:arg name="left_tcp_offset_xyz" default="$(optenv FA_W2R_LEFT_TCP_OFFSET_XYZ 0 0 0)"/>
+	<xacro:arg name="left_tcp_offset_rpy" default="$(optenv FA_W2R_LEFT_TCP_OFFSET_RPY 0 0 0)"/>
+	<xacro:arg name="right_tcp_offset_xyz" default="$(optenv FA_W2R_RIGHT_TCP_OFFSET_XYZ 0 0 0)"/>
+	<xacro:arg name="right_tcp_offset_rpy" default="$(optenv FA_W2R_RIGHT_TCP_OFFSET_RPY 0 0 0)"/>
 	<!-- 从 type 参数解析 arm_config / 对称末端 -->
 	<xacro:property name="type_arg" value="$(arg type)"/>
@@ -86,4 +90,16 @@
 		<xacro:SelectedAR5CCS name="left" collider="$(arg collider)" direction="1"/>
 		<xacro:SelectedAR5CCS name="right" collider="$(arg collider)" direction="-1"/>
+		<link name="left_tcp_offset"/>
+		<joint name="left_tcp_offset_joint" type="fixed">
+			<parent link="left_tcp"/>
+			<child link="left_tcp_offset"/>
+			<origin xyz="$(arg left_tcp_offset_xyz)" rpy="$(arg left_tcp_offset_rpy)"/>
+		</joint>
+		<link name="right_tcp_offset"/>
+		<joint name="right_tcp_offset_joint" type="fixed">
+			<parent link="right_tcp"/>
+			<child link="right_tcp_offset"/>
+			<origin xyz="$(arg right_tcp_offset_xyz)" rpy="$(arg right_tcp_offset_rpy)"/>
+		</joint>
 		<xacro:include filename="$(find ar5_ccs_description)/xacro/eef_type_resolver.xacro"/>
 		<xacro:set_side_eef_types side="left" type_key="${effective_left_type}"/>

File: ar5_srs_description/xacro/robot.xacro (robot description, xacro)
@@ -3,4 +3,8 @@
 	<xacro:arg name="collider" default="convex"/>
 	<xacro:arg name="type" default="dual"/>
+	<xacro:arg name="left_tcp_offset_xyz" default="$(optenv FA_W2R_LEFT_TCP_OFFSET_XYZ 0 0 0)"/>
+	<xacro:arg name="left_tcp_offset_rpy" default="$(optenv FA_W2R_LEFT_TCP_OFFSET_RPY 0 0 0)"/>
+	<xacro:arg name="right_tcp_offset_xyz" default="$(optenv FA_W2R_RIGHT_TCP_OFFSET_XYZ 0 0 0)"/>
+	<xacro:arg name="right_tcp_offset_rpy" default="$(optenv FA_W2R_RIGHT_TCP_OFFSET_RPY 0 0 0)"/>
 	<!-- 拆解 type 参数为三个独立属性 -->
 	<xacro:property name="type_arg" value="$(arg type)"/>
@@ -75,4 +79,16 @@
 		<xacro:Arm name="left" collider="$(arg collider)" direction="1"/>
 		<xacro:Arm name="right" collider="$(arg collider)" direction="-1"/>
+		<link name="left_tcp_offset"/>
+		<joint name="left_tcp_offset_joint" type="fixed">
+			<parent link="left_tcp"/>
+			<child link="left_tcp_offset"/>
+			<origin xyz="$(arg left_tcp_offset_xyz)" rpy="$(arg left_tcp_offset_rpy)"/>
+		</joint>
+		<link name="right_tcp_offset"/>
+		<joint name="right_tcp_offset_joint" type="fixed">
+			<parent link="right_tcp"/>
+			<child link="right_tcp_offset"/>
+			<origin xyz="$(arg right_tcp_offset_xyz)" rpy="$(arg right_tcp_offset_rpy)"/>
+		</joint>
 	</xacro:if>
 	<!-- 根据 gripper_type 添加夹爪 -->

Commit message: fix: update parameter naming from 'variant' to 'arms' in AR5-CCS and AR5-SRS descriptions

File: ar5_ccs_description/xacro/robot.xacro (robot description, xacro)
@@ -3,5 +3,5 @@
 	<xacro:arg name="collider" default="convex"/>
 	<xacro:arg name="skin" default="default"/>
-	<xacro:arg name="variant" default="ar5_ccs"/>
+	<xacro:arg name="arms" default="ar5_ccs"/>
 	<xacro:arg name="type" default="dual"/>
 	<xacro:arg name="left_type" default=""/>
@@ -14,5 +14,4 @@
 	<!-- 从 type 参数解析 arm_config / 对称末端 -->
 	<xacro:property name="type_arg" value="$(arg type)"/>
-	<xacro:property name="variant_arg" value="$(arg variant)"/>
 	<xacro:property name="left_type_arg" value="$(arg left_type)"/>
 	<xacro:property name="right_type_arg" value="$(arg right_type)"/>
@@ -49,15 +48,15 @@
 	</xacro:if>
 	<!-- Select the CCS generation while keeping one public description package. -->
-	<xacro:if value="${'$(arg variant)' == 'ar5_ccs'}">
+	<xacro:if value="${'$(arg arms)' == 'ar5_ccs'}">
 		<xacro:include filename="$(find ar5_ccs_description)/xacro/arm_ccs.xacro"/>
 	</xacro:if>
-	<xacro:if value="${'$(arg variant)' == 'ar5_ccs_v2'}">
+	<xacro:if value="${'$(arg arms)' == 'ar5_ccs_v2'}">
 		<xacro:include filename="$(find ar5_ccs_description)/xacro/arm_ccs_v2.xacro"/>
 	</xacro:if>
 	<xacro:macro name="SelectedAR5CCS" params="name direction collider">
-		<xacro:if value="${'$(arg variant)' == 'ar5_ccs'}">
+		<xacro:if value="${'$(arg arms)' == 'ar5_ccs'}">
 			<xacro:AR5_CCS name="${name}" direction="${direction}" collider="${collider}"/>
 		</xacro:if>
-		<xacro:if value="${'$(arg variant)' == 'ar5_ccs_v2'}">
+		<xacro:if value="${'$(arg arms)' == 'ar5_ccs_v2'}">
 			<xacro:AR5_CCS_V2 name="${name}" direction="${direction}" collider="${collider}" skin="$(arg skin)"/>
 		</xacro:if>

Commit message: fix: adjust collision geometry and origins for arm_base link

File: ar5_ccs_description/xacro/robot.xacro (robot description, xacro)
@@ -76,7 +76,13 @@
 		<link name="arm_base">
 			<collision>
-				<origin xyz="0.0091 0 -0.25"/>
+				<origin xyz="0.0091 0 -0.05"/>
 				<geometry>
-					<box size="0.2000 0.3 0.4029"/>
+					<box size="0.20 0.32 0.20"/>
+				</geometry>
+			</collision>
+			<collision>
+				<origin xyz="0.0091 0 -0.30"/>
+				<geometry>
+					<box size="0.16 0.26 0.30"/>
 				</geometry>
 			</collision>

Commit message: feat: update skin handling for AR5_CCS robot configuration

File: ar5_ccs_description/xacro/robot.xacro (robot description, xacro)
@@ -3,4 +3,8 @@
 	<xacro:arg name="collider" default="convex"/>
 	<xacro:arg name="skin" default="default"/>
+	<xacro:arg name="variant" default=""/>
+	<!-- auto is used by W2R profiles; standalone AR5 retains its default skin. -->
+	<xacro:property name="skin_arg" value="$(arg skin)"/>
+	<xacro:property name="arm_skin" value="${('default' if '$(arg variant)' == 'white' else 'fiveages') if skin_arg in ('', 'auto') else skin_arg}"/>
 	<xacro:arg name="arms" default="ar5_ccs"/>
 	<xacro:arg name="type" default="dual"/>
@@ -59,5 +63,5 @@
 		</xacro:if>
 		<xacro:if value="${'$(arg arms)' == 'ar5_ccs_v2'}">
-			<xacro:AR5_CCS_V2 name="${name}" direction="${direction}" collider="${collider}" skin="$(arg skin)"/>
+			<xacro:AR5_CCS_V2 name="${name}" direction="${direction}" collider="${collider}" skin="${arm_skin}"/>
 		</xacro:if>
 	</xacro:macro>
