Commit message: 使用ar5_ccs的末端工具

File: ar5_ccs_description/xacro/eef_type_resolver.xacro (robot description, xacro)
@@ -1,4 +1,10 @@
 <?xml version="1.0"?>
 <robot xmlns:xacro="http://www.ros.org/wiki/xacro">
+<!--
+  Shared AR5/W2R end-effector type resolver.
+  Supported keys:
+    grippers: rg75, rg75_heavy, ag2f90/ag2f90_d, ag2f90_c, ag2f90_c_soft
+    hands: linkerhand_o6, linkerhand_l6, linkerhand_o7
+-->
     <!-- Map a type key (rg75, linkerhand_o7, ...) to per-side hand/gripper/pad properties. -->
     <xacro:macro name="set_side_eef_types" params="side type_key">

File: ar5_ccs_description/xacro/eefs.xacro (robot description, xacro)
@@ -2,7 +2,7 @@
 <robot xmlns:xacro="http://www.ros.org/wiki/xacro">
     <xacro:arg name="collider" default="simple"/>
+    <xacro:property name="PI" value="3.1415926535897931"/>
     <xacro:include filename="$(find jodell_description)/xacro/RG75-300.xacro"/>
     <xacro:include filename="$(find changingtek_description)/xacro/AG2F90-C.xacro"/>
-    <xacro:include filename="$(find linkerhand_description)/xacro/l6.xacro"/>
     <xacro:macro name="Ocs2SideEefFrame" params="side parent_link">
         <link name="${side}_eef"/>
@@ -12,34 +12,108 @@
         </joint>
     </xacro:macro>
-    <xacro:macro name="SideEndEffector" params="side hand_type gripper_type gripper_pad eef_fixed_joints:=false">
-        <xacro:if value="${gripper_type == '' and hand_type == ''}">
-            <xacro:Ocs2SideEefFrame side="${side}" parent_link="${side}_tcp"/>
-        </xacro:if>
-        <xacro:if value="${gripper_type == 'rg75'}">
-            <xacro:RG75-300 name="${side}" use_flange="true" pad="${gripper_pad}" kinematic_only="${eef_fixed_joints}"/>
-            <joint name="${side}_gripper_base_joint" type="fixed">
-                <origin xyz="0 0 -0.0045"/>
-                <parent link="${side}_tcp"/>
-                <child link="${side}_flange"/>
-            </joint>
-        </xacro:if>
-        <xacro:if value="${gripper_type == 'ag2f90_c' or gripper_type == 'ag2f90_d'}">
-            <xacro:property name="ag2f90_pad" value="${'none' if gripper_type == 'ag2f90_d' else gripper_pad}"/>
-            <xacro:AG2F90-C name="${side}" use_flange="true" pad="${ag2f90_pad}" kinematic_only="${eef_fixed_joints}"/>
-            <joint name="${side}_gripper_base_joint" type="fixed">
-                <origin xyz="0 0 0"/>
-                <parent link="${side}_tcp"/>
-                <child link="${side}_flange"/>
-            </joint>
-        </xacro:if>
-        <xacro:if value="${hand_type == 'linkerhand_l6'}">
-            <xacro:LinkerHandL6 name="${side}_hand" direction="${1 if side == 'left' else -1}"
-                                use_flange="true" fixed_joints="${eef_fixed_joints}"/>
+    <xacro:macro name="SideEndEffectorLinkerHand" params="side hand_type eef_fixed_joints">
+        <xacro:if value="${hand_type == 'linkerhand_o6'}">
+            <xacro:include filename="$(find linkerhand_description)/xacro/o6.xacro"/>
+            <xacro:LinkerHandO6 name="${side}_hand" direction="${1 if side == 'left' else -1}" use_flange="true" fixed_joints="${eef_fixed_joints}"/>
             <joint name="${side}_hand_base_joint" type="fixed">
-                <origin rpy="0 0 ${3.141592653589793 if side == 'left' else 0}"/>
+                <xacro:if value="${side == 'left'}">
+                    <origin xyz="0 0 0.0045" rpy="0 0 ${PI}"/>
+                </xacro:if>
+                <xacro:if value="${side == 'right'}">
+                    <origin xyz="0 0 0.0045"/>
+                </xacro:if>
                 <parent link="${side}_tcp"/>
                 <child link="${side}_hand_flange"/>
             </joint>
         </xacro:if>
+        <xacro:if value="${hand_type == 'linkerhand_l6'}">
+            <xacro:include filename="$(find linkerhand_description)/xacro/l6.xacro"/>
+            <xacro:LinkerHandL6 name="${side}_hand" direction="${1 if side == 'left' else -1}" use_flange="true" fixed_joints="${eef_fixed_joints}"/>
+            <joint name="${side}_hand_base_joint" type="fixed">
+                <xacro:if value="${side == 'left'}">
+                    <origin xyz="0 0 0.0045" rpy="0 0 ${PI}"/>
+                </xacro:if>
+                <xacro:if value="${side == 'right'}">
+                    <origin xyz="0 0 0.0045"/>
+                </xacro:if>
+                <parent link="${side}_tcp"/>
+                <child link="${side}_hand_flange"/>
+            </joint>
+        </xacro:if>
+        <xacro:if value="${hand_type == 'linkerhand_o7'}">
+            <xacro:include filename="$(find linkerhand_description)/xacro/o7.xacro"/>
+            <xacro:LinkerHandO7 name="${side}_hand" direction="${1 if side == 'left' else -1}" use_flange="true" fixed_joints="${eef_fixed_joints}"/>
+            <joint name="${side}_hand_base_joint" type="fixed">
+                <xacro:if value="${side == 'left'}">
+                    <origin rpy="0 0 ${PI/2}"/>
+                </xacro:if>
+                <xacro:if value="${side == 'right'}">
+                    <origin rpy="0 0 ${-PI/2}"/>
+                </xacro:if>
+                <parent link="${side}_tcp"/>
+                <child link="${side}_hand_flange"/>
+            </joint>
+        </xacro:if>
+        <xacro:if value="${hand_type == 'linkerhand_o6' or hand_type == 'linkerhand_l6' or hand_type == 'linkerhand_o7'}">
+            <link name="${side}_eef"/>
+            <joint name="${side}_eef_joint" type="fixed">
+                <parent link="${side}_hand_eef"/>
+                <child link="${side}_eef"/>
+            </joint>
+        </xacro:if>
+    </xacro:macro>
+    <xacro:macro name="SideEndEffector" params="side hand_type gripper_type gripper_pad eef_fixed_joints:=false">
+        <xacro:if value="${eef_fixed_joints}">
+            <xacro:if value="${hand_type == 'linkerhand_o6' or hand_type == 'linkerhand_o7' or hand_type == 'linkerhand_l6'}">
+                <xacro:SideEndEffectorLinkerHand side="${side}" hand_type="${hand_type}" eef_fixed_joints="true"/>
+            </xacro:if>
+            <xacro:unless value="${hand_type == 'linkerhand_o6' or hand_type == 'linkerhand_o7' or hand_type == 'linkerhand_l6'}">
+                <xacro:if value="${gripper_type == 'ag2f90_c' or gripper_type == 'ag2f90_d'}">
+                    <xacro:property name="ag2f90_pad" value="${'none' if gripper_type == 'ag2f90_d' else gripper_pad}"/>
+                    <xacro:AG2F90-C name="${side}" use_flange="true" pad="${ag2f90_pad}" kinematic_only="true"/>
+                    <joint name="${side}_gripper_base_joint" type="fixed">
+                        <origin xyz="0 0 0"/>
+                        <parent link="${side}_tcp"/>
+                        <child link="${side}_flange"/>
+                    </joint>
+                </xacro:if>
+                <xacro:if value="${gripper_type == 'rg75'}">
+                    <xacro:RG75-300 name="${side}" use_flange="true" pad="${gripper_pad}" kinematic_only="true"/>
+                    <joint name="${side}_gripper_base_joint" type="fixed">
+                        <origin xyz="0 0 -0.0045"/>
+                        <parent link="${side}_tcp"/>
+                        <child link="${side}_flange"/>
+                    </joint>
+                </xacro:if>
+                <xacro:if value="${gripper_type == '' and hand_type == ''}">
+                    <xacro:Ocs2SideEefFrame side="${side}" parent_link="${side}_tcp"/>
+                </xacro:if>
+            </xacro:unless>
+        </xacro:if>
+        <xacro:unless value="${eef_fixed_joints}">
+            <xacro:if value="${gripper_type == '' and hand_type == ''}">
+                <xacro:Ocs2SideEefFrame side="${side}" parent_link="${side}_tcp"/>
+            </xacro:if>
+            <xacro:if value="${gripper_type == 'rg75'}">
+                <xacro:RG75-300 name="${side}" use_flange="true" pad="${gripper_pad}" kinematic_only="false"/>
+                <joint name="${side}_gripper_base_joint" type="fixed">
+                    <origin xyz="0 0 -0.0045"/>
+                    <parent link="${side}_tcp"/>
+                    <child link="${side}_flange"/>
+                </joint>
+            </xacro:if>
+            <xacro:if value="${gripper_type == 'ag2f90_c' or gripper_type == 'ag2f90_d'}">
+                <xacro:property name="ag2f90_pad" value="${'none' if gripper_type == 'ag2f90_d' else gripper_pad}"/>
+                <xacro:AG2F90-C name="${side}" use_flange="true" pad="${ag2f90_pad}" kinematic_only="false"/>
+                <joint name="${side}_gripper_base_joint" type="fixed">
+                    <origin xyz="0 0 0"/>
+                    <parent link="${side}_tcp"/>
+                    <child link="${side}_flange"/>
+                </joint>
+            </xacro:if>
+            <xacro:if value="${hand_type == 'linkerhand_o6' or hand_type == 'linkerhand_o7' or hand_type == 'linkerhand_l6'}">
+                <xacro:SideEndEffectorLinkerHand side="${side}" hand_type="${hand_type}" eef_fixed_joints="false"/>
+            </xacro:if>
+        </xacro:unless>
     </xacro:macro>
     <xacro:macro name="EndEffectors"

File: ar5_ccs_description/xacro/robot.xacro (robot description, xacro)
@@ -102,20 +102,7 @@
 			right_gripper_pad="${right_gripper_pad}"/>
 	</xacro:if>
-	<!-- 单臂配置沿用旧夹爪宏。双臂末端由 EndEffectors 按侧生成。 -->
+	<!-- 单臂配置沿用旧夹爪宏（无前缀）。双臂末端由 EndEffectors 按侧生成。 -->
 	<xacro:if value="${selected_arm_config != 'dual' and selected_gripper_type != ''}">
 		<xacro:Grippers type="${selected_gripper_type}" arm_config="${selected_arm_config}"/>
 	</xacro:if>
-	<xacro:if value="${selected_arm_config != 'dual'}">
-		<xacro:include filename="$(find linkerhand_description)/xacro/l6.xacro"/>
-		<xacro:if value="${(left_hand_type if selected_arm_config == 'left' else right_hand_type) == 'linkerhand_l6'}">
-			<xacro:LinkerHandL6 name="${'left_hand' if selected_arm_config == 'left' else 'right_hand'}"
-							direction="${1 if selected_arm_config == 'left' else -1}"
-							use_flange="true" fixed_joints="$(arg eef_fixed_joints)"/>
-			<joint name="hand_base_joint" type="fixed">
-				<origin rpy="0 0 ${3.141592653589793 if selected_arm_config == 'left' else 0}"/>
-				<parent link="tcp"/>
-				<child link="${'left_hand_flange' if selected_arm_config == 'left' else 'right_hand_flange'}"/>
-			</joint>
-		</xacro:if>
-	</xacro:if>
 </robot>
