Commit message: 增加erg32/120s/120sd 加爪

File: ar5_ccs_description/xacro/eef_type_resolver.xacro (robot description, xacro)
@@ -4,5 +4,5 @@
   Shared AR5/W2R end-effector type resolver.
   Supported keys:
-    grippers: rg75, rg75_heavy, ag2f90/ag2f90_d, ag2f90_c, ag2f90_c_soft
+    grippers: rg75, rg75_heavy, erg32/ERG32, ag2f90/ag2f90_d, ag2f90_c, ag2f90_c_soft, ag2f120s, ag2f120s_d
     hands: linkerhand_o6, linkerhand_l6, linkerhand_o7
 -->
@@ -19,4 +19,7 @@
             <xacro:property name="${side}_gripper_pad" value="heavy_carry" scope="parent"/>
         </xacro:if>
+        <xacro:if value="${type_key == 'erg32' or type_key == 'ERG32'}">
+            <xacro:property name="${side}_gripper_type" value="erg32" scope="parent"/>
+        </xacro:if>
         <xacro:if value="${type_key == 'ag2f90' or type_key == 'ag2f90_d'}">
             <xacro:property name="${side}_gripper_type" value="ag2f90_d" scope="parent"/>
@@ -28,4 +31,10 @@
             <xacro:property name="${side}_gripper_type" value="ag2f90_c" scope="parent"/>
             <xacro:property name="${side}_gripper_pad" value="soft" scope="parent"/>
+        </xacro:if>
+        <xacro:if value="${type_key == 'ag2f120s' or type_key == 'AG2F120S'}">
+            <xacro:property name="${side}_gripper_type" value="ag2f120s" scope="parent"/>
+        </xacro:if>
+        <xacro:if value="${type_key == 'ag2f120s_d' or type_key == 'AG2F120S_D'}">
+            <xacro:property name="${side}_gripper_type" value="ag2f120s_d" scope="parent"/>
         </xacro:if>
         <xacro:if value="${type_key == 'linkerhand_o6'}">

File: ar5_ccs_description/xacro/eefs.xacro (robot description, xacro)
@@ -4,5 +4,7 @@
     <xacro:property name="PI" value="3.1415926535897931"/>
     <xacro:include filename="$(find jodell_description)/xacro/RG75-300.xacro"/>
+    <xacro:include filename="$(find jodell_description)/xacro/ERG32.xacro"/>
     <xacro:include filename="$(find changingtek_description)/xacro/AG2F90-C.xacro"/>
+    <xacro:include filename="$(find changingtek_description)/xacro/AG2F120S.xacro"/>
     <xacro:macro name="Ocs2SideEefFrame" params="side parent_link">
         <link name="${side}_eef"/>
@@ -86,4 +88,19 @@
                     </joint>
                 </xacro:if>
+            <xacro:if value="${gripper_type == 'erg32'}">
+                <xacro:ERG32 name="${side}_hand" use_flange="true" kinematic_only="true"/>
+                <joint name="${side}_hand_base_joint" type="fixed">
+                    <parent link="${side}_tcp"/>
+                    <child link="${side}_hand_flange"/>
+                </joint>
+            </xacro:if>
+            <xacro:if value="${gripper_type == 'ag2f120s' or gripper_type == 'ag2f120s_d'}">
+                <xacro:AG2F120S name="${side}" use_flange="true" kinematic_only="true"/>
+                <joint name="${side}_gripper_base_joint" type="fixed">
+                    <origin xyz="0 0 0"/>
+                    <parent link="${side}_tcp"/>
+                    <child link="${side}_flange"/>
+                </joint>
+            </xacro:if>
                 <xacro:if value="${gripper_type == '' and hand_type == ''}">
                     <xacro:Ocs2SideEefFrame side="${side}" parent_link="${side}_tcp"/>
@@ -106,4 +123,19 @@
                 <xacro:property name="ag2f90_pad" value="${'none' if gripper_type == 'ag2f90_d' else gripper_pad}"/>
                 <xacro:AG2F90-C name="${side}" use_flange="true" pad="${ag2f90_pad}" kinematic_only="false"/>
+                <joint name="${side}_gripper_base_joint" type="fixed">
+                    <origin xyz="0 0 0"/>
+                    <parent link="${side}_tcp"/>
+                    <child link="${side}_flange"/>
+                </joint>
+            </xacro:if>
+            <xacro:if value="${gripper_type == 'erg32'}">
+                <xacro:ERG32 name="${side}_hand" use_flange="true" kinematic_only="false"/>
+                <joint name="${side}_hand_base_joint" type="fixed">
+                    <parent link="${side}_tcp"/>
+                    <child link="${side}_hand_flange"/>
+                </joint>
+            </xacro:if>
+            <xacro:if value="${gripper_type == 'ag2f120s' or gripper_type == 'ag2f120s_d'}">
+                <xacro:AG2F120S name="${side}" use_flange="true" kinematic_only="false"/>
                 <joint name="${side}_gripper_base_joint" type="fixed">
                     <origin xyz="0 0 0"/>

File: ar5_ccs_description/xacro/ros2_control/end_effector_interfaces.xacro (robot description, xacro)
@@ -3,5 +3,7 @@
     <xacro:include filename="$(find ar5_ccs_description)/xacro/ros2_control/interfaces.xacro"/>
     <xacro:include filename="$(find jodell_description)/xacro/ros2_control/RG75-300.xacro"/>
+    <xacro:include filename="$(find jodell_description)/xacro/ros2_control/ERG32.xacro"/>
     <xacro:include filename="$(find changingtek_description)/xacro/ros2_control/AG2F90-C.xacro"/>
+    <xacro:include filename="$(find changingtek_description)/xacro/ros2_control/AG2F120S.xacro"/>
     <xacro:include filename="$(find linkerhand_description)/xacro/ros2_control/o6.xacro"/>
     <xacro:include filename="$(find linkerhand_description)/xacro/ros2_control/o7.xacro"/>
@@ -17,4 +19,7 @@
     </xacro:macro>
     <xacro:macro name="side_gripper_interfaces_sim" params="side gripper_type">
+        <xacro:if value="${gripper_type == 'erg32'}">
+            <xacro:erg32_interfaces name="${side}_hand"/>
+        </xacro:if>
         <xacro:if value="${gripper_type == 'rg75'}">
             <xacro:rg75_interfaces name="${side}"/>
@@ -23,4 +28,10 @@
             <xacro:ag2f90c_interfaces name="${side}"/>
         </xacro:if>
+        <xacro:if value="${gripper_type == 'ag2f120s' or gripper_type == 'ag2f120s_d'}">
+            <xacro:ag2f120s_interfaces name="${side}"/>
+        </xacro:if>
+    </xacro:macro>
+    <xacro:macro name="side_erg32_interfaces" params="side">
+        <xacro:erg32_interfaces name="${side}_hand"/>
     </xacro:macro>
     <xacro:macro name="side_hand_interfaces" params="side hand_type">
@@ -43,5 +54,8 @@
         </xacro:if>
         <xacro:if value="${mode == 'real'}">
-            <xacro:if value="${gripper_type != ''}">
+            <xacro:if value="${gripper_type == 'erg32'}">
+                <xacro:side_erg32_interfaces side="${side}"/>
+            </xacro:if>
+            <xacro:if value="${gripper_type != '' and gripper_type != 'erg32'}">
                 <xacro:side_gripper_joint side="${side}"/>
             </xacro:if>
@@ -70,8 +84,14 @@
         </xacro:if>
         <xacro:if value="${mode == 'real'}">
-            <xacro:if value="${left_gripper_type != ''}">
+            <xacro:if value="${left_gripper_type == 'erg32'}">
+                <xacro:side_erg32_interfaces side="left"/>
+            </xacro:if>
+            <xacro:if value="${left_gripper_type != '' and left_gripper_type != 'erg32'}">
                 <xacro:side_gripper_joint side="left"/>
             </xacro:if>
-            <xacro:if value="${right_gripper_type != ''}">
+            <xacro:if value="${right_gripper_type == 'erg32'}">
+                <xacro:side_erg32_interfaces side="right"/>
+            </xacro:if>
+            <xacro:if value="${right_gripper_type != '' and right_gripper_type != 'erg32'}">
                 <xacro:side_gripper_joint side="right"/>
             </xacro:if>
@@ -93,5 +113,8 @@
         </xacro:if>
         <xacro:if value="${mode == 'real'}">
-            <xacro:if value="${gripper_type != ''}">
+            <xacro:if value="${gripper_type == 'erg32'}">
+                <xacro:erg32_interfaces name=""/>
+            </xacro:if>
+            <xacro:if value="${gripper_type != '' and gripper_type != 'erg32'}">
                 <xacro:side_gripper_joint side=""/>
             </xacro:if>

File: ar5_ccs_description/xacro/ros2_control/rokae_hardware.xacro (robot description, xacro)
@@ -110,4 +110,9 @@
             <param name="${side}_tool_velocity">1.0</param>
         </xacro:if>
+        <xacro:if value="${gripper_type == 'erg32'}">
+            <param name="gripper_type">erg32</param>
+            <param name="${side}_tool_torque">1.0</param>
+            <param name="${side}_tool_velocity">1.0</param>
+        </xacro:if>
         <xacro:if value="${gripper_type == 'ag2f90_c' or gripper_type == 'ag2f90_d'}">
             <param name="gripper_type">${gripper_type}</param>
@@ -115,4 +120,22 @@
             <param name="gripper_close_pos">9000</param>
             <param name="gripper_max_opening_distance">1.0</param>
+            <param name="gripper_configure_xpanel">false</param>
+            <param name="${side}_tool_torque">1.0</param>
+            <param name="${side}_tool_velocity">1.0</param>
+        </xacro:if>
+        <xacro:if value="${gripper_type == 'ag2f120s'}">
+            <param name="gripper_type">ag2f120s</param>
+            <param name="gripper_slave_id">1</param>
+            <param name="gripper_close_pos">12000</param>
+            <param name="gripper_max_opening_distance">0.12</param>
+            <param name="gripper_configure_xpanel">false</param>
+            <param name="${side}_tool_torque">1.0</param>
+            <param name="${side}_tool_velocity">1.0</param>
+        </xacro:if>
+        <xacro:if value="${gripper_type == 'ag2f120s_d'}">
+            <param name="gripper_type">ag2f120s_d</param>
+            <param name="gripper_slave_id">1</param>
+            <param name="gripper_close_pos">1000</param>
+            <param name="gripper_max_opening_distance">0.10</param>
             <param name="gripper_configure_xpanel">false</param>
             <param name="${side}_tool_torque">1.0</param>

Commit message: update rokae ros2 control

File: ar5_ccs_description/xacro/eef_type_resolver.xacro (robot description, xacro)
@@ -4,5 +4,5 @@
   Shared AR5/W2R end-effector type resolver.
   Supported keys:
-    grippers: rg75, rg75_heavy, erg32/ERG32, ag2f90/ag2f90_d, ag2f90_c, ag2f90_c_soft, ag2f120s, ag2f120s_d
+    grippers: rg75, rg75_heavy, leapmotor, erg32/ERG32, ag2f90/ag2f90_d, ag2f90_c/AG2F90-C, ag2f90_c_soft, ag2f120s, ag2f120s_d
     hands: linkerhand_o6, linkerhand_l6, linkerhand_o7
 -->
@@ -19,4 +19,8 @@
             <xacro:property name="${side}_gripper_pad" value="heavy_carry" scope="parent"/>
         </xacro:if>
+        <xacro:if value="${type_key == 'leapmotor'}">
+            <xacro:property name="${side}_gripper_type" value="rg75" scope="parent"/>
+            <xacro:property name="${side}_gripper_pad" value="leapmotor" scope="parent"/>
+        </xacro:if>
         <xacro:if value="${type_key == 'erg32' or type_key == 'ERG32'}">
             <xacro:property name="${side}_gripper_type" value="erg32" scope="parent"/>
@@ -25,5 +29,5 @@
             <xacro:property name="${side}_gripper_type" value="ag2f90_d" scope="parent"/>
         </xacro:if>
-        <xacro:if value="${type_key == 'ag2f90_c'}">
+        <xacro:if value="${type_key == 'ag2f90_c' or type_key == 'AG2F90-C'}">
             <xacro:property name="${side}_gripper_type" value="ag2f90_c" scope="parent"/>
         </xacro:if>

File: ar5_ccs_description/xacro/robot.xacro (robot description, xacro)
@@ -3,5 +3,5 @@
 	<xacro:arg name="collider" default="convex"/>
 	<xacro:arg name="skin" default="default"/>
-	<xacro:arg name="variant" default="base_ar5_ccs"/>
+	<xacro:arg name="variant" default="ar5_ccs"/>
 	<xacro:arg name="type" default="dual"/>
 	<xacro:arg name="left_type" default=""/>
@@ -49,15 +49,15 @@
 	</xacro:if>
 	<!-- Select the CCS generation while keeping one public description package. -->
-	<xacro:if value="${'$(arg variant)' != 'base_ar5_ccs_v2' and '$(arg variant)' != 'base_ar5_srs'}">
+	<xacro:if value="${'$(arg variant)' == 'ar5_ccs'}">
 		<xacro:include filename="$(find ar5_ccs_description)/xacro/arm_ccs.xacro"/>
 	</xacro:if>
-	<xacro:if value="${'$(arg variant)' == 'base_ar5_ccs_v2'}">
+	<xacro:if value="${'$(arg variant)' == 'ar5_ccs_v2'}">
 		<xacro:include filename="$(find ar5_ccs_description)/xacro/arm_ccs_v2.xacro"/>
 	</xacro:if>
 	<xacro:macro name="SelectedAR5CCS" params="name direction collider">
-		<xacro:if value="${'$(arg variant)' != 'base_ar5_ccs_v2' and '$(arg variant)' != 'base_ar5_srs'}">
+		<xacro:if value="${'$(arg variant)' == 'ar5_ccs'}">
 			<xacro:AR5_CCS name="${name}" direction="${direction}" collider="${collider}"/>
 		</xacro:if>
-		<xacro:if value="${'$(arg variant)' == 'base_ar5_ccs_v2'}">
+		<xacro:if value="${'$(arg variant)' == 'ar5_ccs_v2'}">
 			<xacro:AR5_CCS_V2 name="${name}" direction="${direction}" collider="${collider}"/>
 		</xacro:if>
