Commit message: feat: add support for additional end-effectors and external systems in AR5 CCS description

File: ar5_ccs_description/xacro/eef_type_resolver.xacro (robot description, xacro)
@@ -5,5 +5,6 @@
   Supported keys:
     grippers: rg75, rg75_heavy, leapmotor, erg32/ERG32, ag2f90/ag2f90_d, ag2f90_c/AG2F90-C, ag2f90_c_soft, ag2f120s, ag2f120s_d
-    hands: linkerhand_o6, linkerhand_l6, linkerhand_o7
+    hands: linkerhand_o6, linkerhand_l6, linkerhand_o7, freedom_v1, freedom_v2,
+           inspire_e2, inspire_f2, xhand1, theohand_std16a
 -->
     <!-- Map a type key (rg75, linkerhand_o7, ...) to per-side hand/gripper/pad properties. -->
@@ -51,4 +52,7 @@
             <xacro:property name="${side}_hand_type" value="linkerhand_o7" scope="parent"/>
         </xacro:if>
+        <xacro:if value="${type_key in ('freedom_v1', 'freedom_v2', 'inspire_e2', 'inspire_f2', 'xhand1', 'theohand_std16a')}">
+            <xacro:property name="${side}_hand_type" value="${type_key}" scope="parent"/>
+        </xacro:if>
     </xacro:macro>
 </robot>

File: ar5_ccs_description/xacro/eefs.xacro (robot description, xacro)
@@ -7,4 +7,10 @@
     <xacro:include filename="$(find changingtek_description)/xacro/AG2F90-C.xacro"/>
     <xacro:include filename="$(find changingtek_description)/xacro/AG2F120S.xacro"/>
+    <xacro:include filename="$(find freedom_description)/xacro/freedomv1.xacro"/>
+    <xacro:include filename="$(find freedom_description)/xacro/freedomv2.xacro"/>
+    <xacro:include filename="$(find inspire_description)/xacro/hands/RH56E2.xacro"/>
+    <xacro:include filename="$(find inspire_description)/xacro/hands/RH56F2.xacro"/>
+    <xacro:include filename="$(find xhand1_description)/xacro/xhand1.xacro"/>
+    <xacro:include filename="$(find theohand_description)/xacro/std16a.xacro"/>
     <xacro:macro name="Ocs2SideEefFrame" params="side parent_link">
         <link name="${side}_eef"/>
@@ -57,5 +63,53 @@
             </joint>
         </xacro:if>
-        <xacro:if value="${hand_type == 'linkerhand_o6' or hand_type == 'linkerhand_l6' or hand_type == 'linkerhand_o7'}">
+        <xacro:if value="${hand_type == 'freedom_v1'}">
+            <xacro:FreedomHand name="${side}_hand" direction="${1 if side == 'left' else -1}" fixed_joints="${eef_fixed_joints}"/>
+            <joint name="${side}_hand_base_joint" type="fixed">
+                <origin xyz="0 0 0.0045" rpy="${PI/2} 0 ${PI if side == 'left' else 0}"/>
+                <parent link="${side}_tcp"/>
+                <child link="${side}_hand_hand_base"/>
+            </joint>
+        </xacro:if>
+        <xacro:if value="${hand_type == 'freedom_v2'}">
+            <xacro:FreedomHandV2 name="${side}_hand" direction="${1 if side == 'left' else -1}" fixed_joints="${eef_fixed_joints}"/>
+            <joint name="${side}_hand_base_joint" type="fixed">
+                <origin rpy="0 0 ${PI}"/>
+                <parent link="${side}_tcp"/>
+                <child link="${side}_hand_hand_base"/>
+            </joint>
+        </xacro:if>
+        <xacro:if value="${hand_type == 'inspire_e2'}">
+            <xacro:InspireHandRH56E2 name="${side}_hand" direction="${1 if side == 'left' else -1}" use_flange="true" fixed_joints="${eef_fixed_joints}"/>
+            <joint name="${side}_hand_base_joint" type="fixed">
+                <origin xyz="0 0 0.0045" rpy="0 0 ${PI if side == 'left' else -PI}"/>
+                <parent link="${side}_tcp"/>
+                <child link="${side}_hand_flange"/>
+            </joint>
+        </xacro:if>
+        <xacro:if value="${hand_type == 'inspire_f2'}">
+            <xacro:InspireHandRH56F2 name="${side}_hand" direction="${1 if side == 'left' else -1}" use_flange="true" fixed_joints="${eef_fixed_joints}"/>
+            <joint name="${side}_hand_base_joint" type="fixed">
+                <origin xyz="0 0 0.0045" rpy="0 0 ${PI if side == 'left' else -PI}"/>
+                <parent link="${side}_tcp"/>
+                <child link="${side}_hand_flange"/>
+            </joint>
+        </xacro:if>
+        <xacro:if value="${hand_type == 'xhand1'}">
+            <xacro:XHand1 name="${side}_hand" direction="${1 if side == 'left' else -1}" fixed_joints="${eef_fixed_joints}"/>
+            <joint name="${side}_hand_base_joint" type="fixed">
+                <origin rpy="0 0 ${PI}"/>
+                <parent link="${side}_tcp"/>
+                <child link="${side}_hand_hand_base"/>
+            </joint>
+        </xacro:if>
+        <xacro:if value="${hand_type == 'theohand_std16a'}">
+            <xacro:TheoHandStd16A name="${side}_hand" direction="${1 if side == 'left' else -1}" use_flange="true" fixed_joints="${eef_fixed_joints}"/>
+            <joint name="${side}_hand_base_joint" type="fixed">
+                <origin xyz="0 0 0.011043" rpy="0 0 ${PI/2 if side == 'left' else -PI/2}"/>
+                <parent link="${side}_tcp"/>
+                <child link="${side}_hand_flange"/>
+            </joint>
+        </xacro:if>
+        <xacro:if value="${hand_type in ('linkerhand_o6', 'linkerhand_l6', 'linkerhand_o7', 'freedom_v1', 'freedom_v2', 'inspire_e2', 'inspire_f2', 'xhand1', 'theohand_std16a')}">
             <link name="${side}_eef"/>
             <joint name="${side}_eef_joint" type="fixed">
@@ -67,8 +121,8 @@
     <xacro:macro name="SideEndEffector" params="side hand_type gripper_type gripper_pad eef_fixed_joints:=false">
         <xacro:if value="${eef_fixed_joints}">
-            <xacro:if value="${hand_type == 'linkerhand_o6' or hand_type == 'linkerhand_o7' or hand_type == 'linkerhand_l6'}">
+            <xacro:if value="${hand_type in ('linkerhand_o6', 'linkerhand_o7', 'linkerhand_l6', 'freedom_v1', 'freedom_v2', 'inspire_e2', 'inspire_f2', 'xhand1', 'theohand_std16a')}">
                 <xacro:SideEndEffectorLinkerHand side="${side}" hand_type="${hand_type}" eef_fixed_joints="true"/>
             </xacro:if>
-            <xacro:unless value="${hand_type == 'linkerhand_o6' or hand_type == 'linkerhand_o7' or hand_type == 'linkerhand_l6'}">
+            <xacro:unless value="${hand_type in ('linkerhand_o6', 'linkerhand_o7', 'linkerhand_l6', 'freedom_v1', 'freedom_v2', 'inspire_e2', 'inspire_f2', 'xhand1', 'theohand_std16a')}">
                 <xacro:if value="${gripper_type == 'ag2f90_c' or gripper_type == 'ag2f90_d'}">
                     <xacro:AG2F90-C name="${side}" use_flange="true" pad="${gripper_pad}" kinematic_only="true"/>
@@ -144,5 +198,5 @@
                 </joint>
             </xacro:if>
-            <xacro:if value="${hand_type == 'linkerhand_o6' or hand_type == 'linkerhand_o7' or hand_type == 'linkerhand_l6'}">
+            <xacro:if value="${hand_type in ('linkerhand_o6', 'linkerhand_o7', 'linkerhand_l6', 'freedom_v1', 'freedom_v2', 'inspire_e2', 'inspire_f2', 'xhand1', 'theohand_std16a')}">
                 <xacro:SideEndEffectorLinkerHand side="${side}" hand_type="${hand_type}" eef_fixed_joints="false"/>
             </xacro:if>

File: ar5_ccs_description/xacro/ros2_control/external_ee_systems.xacro (robot description, xacro)
@@ -2,7 +2,14 @@
 <robot xmlns:xacro="http://www.ros.org/wiki/xacro">
     <xacro:include filename="$(find ar5_ccs_description)/xacro/ros2_control/end_effector_interfaces.xacro"/>
-    <xacro:macro name="side_usb_hand_system" params="side hand_type serial_port">
+    <xacro:include filename="$(find jodell_description)/xacro/ros2_control/side_systems.xacro"/>
+    <xacro:include filename="$(find changingtek_description)/xacro/ros2_control/side_systems.xacro"/>
+    <xacro:include filename="$(find freedom_description)/xacro/ros2_control/side_systems.xacro"/>
+    <xacro:include filename="$(find inspire_description)/xacro/ros2_control/side_systems.xacro"/>
+    <xacro:include filename="$(find theohand_description)/xacro/ros2_control/side_systems.xacro"/>
+    <xacro:include filename="$(find xhand1_description)/xacro/ros2_control/side_systems.xacro"/>
+    <xacro:macro name="side_usb_hand_system" params="side hand_type serial_port rw_rate:=''">
         <xacro:property name="usb_hand_system_name" value="${str('linkerhand_7' if hand_type == 'linkerhand_o7' else 'linkerhand_6')}"/>
-        <ros2_control name="${usb_hand_system_name}_${side}_system" type="system">
+        <xacro:property name="usb_hand_rw_rate" value="${rw_rate if rw_rate != '' else 30}"/>
+        <ros2_control name="${usb_hand_system_name}_${side}_system" type="system" rw_rate="${usb_hand_rw_rate}">
             <hardware>
                 <plugin>modbus_ros2_control/DexterousHandHardware</plugin>
@@ -119,5 +126,8 @@
         right_ee_modbus_slave_id:=1
         left_read_tactile:=false
-        right_read_tactile:=false">
+        right_read_tactile:=false
+        left_ee_rw_rate:=''
+        right_ee_rw_rate:=''
+        usb_baudrate:=115200">
         <xacro:if value="${arm_driver == 'inex' and left_drive_type == 'inex_rs485' and left_gripper_type == 'ag2f90_d'}">
             <xacro:ag2f90d_inex_rs485_side_system side="left" rs485_channel="${left_ee_rs485_channel}" slave_id="${left_ee_modbus_slave_id}"/>
@@ -139,14 +149,62 @@
         </xacro:if>
         <xacro:if value="${left_drive_type == 'usb_can' and (left_hand_type == 'linkerhand_o6' or left_hand_type == 'linkerhand_l6' or left_hand_type == 'linkerhand_o7')}">
-            <xacro:linkerhand_usb_can_side_system side="left" hand_type="${left_hand_type}" can_interface="${left_ee_can_interface}" read_tactile="${left_read_tactile}"/>
+            <xacro:linkerhand_usb_can_side_system side="left" hand_type="${left_hand_type}" can_interface="${left_ee_can_interface}" read_tactile="${left_read_tactile}" rw_rate="${left_ee_rw_rate}"/>
         </xacro:if>
         <xacro:if value="${right_drive_type == 'usb_can' and (right_hand_type == 'linkerhand_o6' or right_hand_type == 'linkerhand_l6' or right_hand_type == 'linkerhand_o7')}">
-            <xacro:linkerhand_usb_can_side_system side="right" hand_type="${right_hand_type}" can_interface="${right_ee_can_interface}" read_tactile="${right_read_tactile}"/>
-        </xacro:if>
-        <xacro:if value="${left_drive_type == 'usb_rs485' and (left_hand_type == 'linkerhand_o6' or left_hand_type == 'linkerhand_l6' or left_hand_type == 'linkerhand_o7')}">
-            <xacro:side_usb_hand_system side="left" hand_type="${left_hand_type}" serial_port="${usb_left_port}"/>
-        </xacro:if>
-        <xacro:if value="${right_drive_type == 'usb_rs485' and (right_hand_type == 'linkerhand_o6' or right_hand_type == 'linkerhand_l6' or right_hand_type == 'linkerhand_o7')}">
-            <xacro:side_usb_hand_system side="right" hand_type="${right_hand_type}" serial_port="${usb_right_port}"/>
+            <xacro:linkerhand_usb_can_side_system side="right" hand_type="${right_hand_type}" can_interface="${right_ee_can_interface}" read_tactile="${right_read_tactile}" rw_rate="${right_ee_rw_rate}"/>
+        </xacro:if>
+        <xacro:if value="${left_drive_type in ('usb', 'usb_rs485') and (left_hand_type == 'linkerhand_o6' or left_hand_type == 'linkerhand_l6' or left_hand_type == 'linkerhand_o7')}">
+            <xacro:side_usb_hand_system side="left" hand_type="${left_hand_type}" serial_port="${usb_left_port}" rw_rate="${left_ee_rw_rate}"/>
+        </xacro:if>
+        <xacro:if value="${right_drive_type in ('usb', 'usb_rs485') and (right_hand_type == 'linkerhand_o6' or right_hand_type == 'linkerhand_l6' or right_hand_type == 'linkerhand_o7')}">
+            <xacro:side_usb_hand_system side="right" hand_type="${right_hand_type}" serial_port="${usb_right_port}" rw_rate="${right_ee_rw_rate}"/>
+        </xacro:if>
+        <xacro:if value="${left_drive_type in ('usb', 'usb_rs485') and left_hand_type == 'theohand_std16a'}">
+            <xacro:theohand_usb_side_system side="left" serial_port="${usb_left_port}" baudrate="${usb_baudrate}" rw_rate="${left_ee_rw_rate}"/>
+        </xacro:if>
+        <xacro:if value="${right_drive_type in ('usb', 'usb_rs485') and right_hand_type == 'theohand_std16a'}">
+            <xacro:theohand_usb_side_system side="right" serial_port="${usb_right_port}" baudrate="${usb_baudrate}" rw_rate="${right_ee_rw_rate}"/>
+        </xacro:if>
+        <xacro:if value="${left_drive_type in ('usb', 'usb_rs485') and left_hand_type in ('inspire_e2', 'inspire_f2')}">
+            <xacro:inspire_rs485_side_system side="left" serial_port="${usb_left_port}" hand_type="${left_hand_type}" rw_rate="${left_ee_rw_rate}"/>
+        </xacro:if>
+        <xacro:if value="${right_drive_type in ('usb', 'usb_rs485') and right_hand_type in ('inspire_e2', 'inspire_f2')}">
+            <xacro:inspire_rs485_side_system side="right" serial_port="${usb_right_port}" hand_type="${right_hand_type}" rw_rate="${right_ee_rw_rate}"/>
+        </xacro:if>
+        <xacro:if value="${left_drive_type in ('usb', 'usb_rs485') and left_hand_type in ('freedom_v1', 'freedom_v2')}">
+            <xacro:freedom_rs485_side_system side="left" serial_port="${usb_left_port}" type="${'freedomv2' if left_hand_type == 'freedom_v2' else 'freedomv1'}" rw_rate="${left_ee_rw_rate}"/>
+        </xacro:if>
+        <xacro:if value="${right_drive_type in ('usb', 'usb_rs485') and right_hand_type in ('freedom_v1', 'freedom_v2')}">
+            <xacro:freedom_rs485_side_system side="right" serial_port="${usb_right_port}" type="${'freedomv2' if right_hand_type == 'freedom_v2' else 'freedomv1'}" rw_rate="${right_ee_rw_rate}"/>
+        </xacro:if>
+        <xacro:if value="${left_drive_type in ('usb', 'usb_rs485') and left_hand_type == 'xhand1'}">
+            <xacro:xhand1_rs485_side_system side="left" serial_port="${usb_left_port}" rw_rate="${left_ee_rw_rate}"/>
+        </xacro:if>
+        <xacro:if value="${right_drive_type in ('usb', 'usb_rs485') and right_hand_type == 'xhand1'}">
+            <xacro:xhand1_rs485_side_system side="right" serial_port="${usb_right_port}" rw_rate="${right_ee_rw_rate}"/>
+        </xacro:if>
+        <xacro:if value="${left_drive_type == 'usb_can' and left_hand_type == 'freedom_v1'}">
+            <xacro:freedom_can_side_system side="left" can_interface="${left_ee_can_interface}" device_id="0" rw_rate="${left_ee_rw_rate}"/>
+        </xacro:if>
+        <xacro:if value="${right_drive_type == 'usb_can' and right_hand_type == 'freedom_v1'}">
+            <xacro:freedom_can_side_system side="right" can_interface="${right_ee_can_interface}" device_id="1" rw_rate="${right_ee_rw_rate}"/>
+        </xacro:if>
+        <xacro:if value="${left_drive_type == 'usb_can' and left_hand_type in ('inspire_e2', 'inspire_f2')}">
+            <xacro:inspire_canfd_side_system side="left" can_interface="${left_ee_can_interface}" hand_type="${left_hand_type}" rw_rate="${left_ee_rw_rate}"/>
+        </xacro:if>
+        <xacro:if value="${right_drive_type == 'usb_can' and right_hand_type in ('inspire_e2', 'inspire_f2')}">
+            <xacro:inspire_canfd_side_system side="right" can_interface="${right_ee_can_interface}" hand_type="${right_hand_type}" rw_rate="${right_ee_rw_rate}"/>
+        </xacro:if>
+        <xacro:if value="${left_drive_type in ('usb', 'usb_rs485') and left_gripper_type == 'ag2f90_d'}">
+            <xacro:changingtek_usb_side_system side="left" variant="90d" serial_port="${usb_left_port}" rw_rate="${left_ee_rw_rate}"/>
+        </xacro:if>
+        <xacro:if value="${right_drive_type in ('usb', 'usb_rs485') and right_gripper_type == 'ag2f90_d'}">
+            <xacro:changingtek_usb_side_system side="right" variant="90d" serial_port="${usb_right_port}" rw_rate="${right_ee_rw_rate}"/>
+        </xacro:if>
+        <xacro:if value="${left_drive_type in ('usb', 'usb_rs485') and left_gripper_type == 'rg75'}">
+            <xacro:jodell_usb_side_system side="left" serial_port="${usb_left_port}" rw_rate="${left_ee_rw_rate}"/>
+        </xacro:if>
+        <xacro:if value="${right_drive_type in ('usb', 'usb_rs485') and right_gripper_type == 'rg75'}">
+            <xacro:jodell_usb_side_system side="right" serial_port="${usb_right_port}" rw_rate="${right_ee_rw_rate}"/>
         </xacro:if>
     </xacro:macro>
