Commit message: add wujihand2 support

File: ar5_ccs_description/xacro/eef_type_resolver.xacro (robot description, xacro)
@@ -6,5 +6,5 @@
     grippers: rg75, rg75_heavy, leapmotor, erg32/ERG32, ag2f90/ag2f90_d, ag2f90_c/AG2F90-C, ag2f90_c_soft, ag2f120s, ag2f120s_d
     hands: linkerhand_o6, linkerhand_l6, linkerhand_o7, freedom_v1, freedom_v2,
-           inspire_e2, inspire_f2, xhand1, theohand_std16a
+           inspire_e2, inspire_f2, xhand1, theohand_std16a, wuji_hand2
 -->
     <!-- Map a type key (rg75, linkerhand_o7, ...) to per-side hand/gripper/pad properties. -->
@@ -52,5 +52,5 @@
             <xacro:property name="${side}_hand_type" value="linkerhand_o7" scope="parent"/>
         </xacro:if>
-        <xacro:if value="${type_key in ('freedom_v1', 'freedom_v2', 'inspire_e2', 'inspire_f2', 'xhand1', 'theohand_std16a')}">
+        <xacro:if value="${type_key in ('freedom_v1', 'freedom_v2', 'inspire_e2', 'inspire_f2', 'xhand1', 'theohand_std16a', 'wuji_hand2')}">
             <xacro:property name="${side}_hand_type" value="${type_key}" scope="parent"/>
         </xacro:if>

File: ar5_ccs_description/xacro/eefs.xacro (robot description, xacro)
@@ -13,4 +13,5 @@
     <xacro:include filename="$(find xhand1_description)/xacro/xhand1.xacro"/>
     <xacro:include filename="$(find theohand_description)/xacro/std16a.xacro"/>
+    <xacro:include filename="$(find wuji_description)/xacro/hand2.xacro"/>
     <xacro:macro name="Ocs2SideEefFrame" params="side parent_link">
         <link name="${side}_eef"/>
@@ -116,4 +117,14 @@
             </joint>
         </xacro:if>
+        <xacro:if value="${hand_type == 'wuji_hand2'}">
+            <xacro:WujiHand2 name="${side}_hand" direction="${1 if side == 'left' else -1}" use_mount="true" fixed_joints="${eef_fixed_joints}"/>
+            <!-- mount→hand_base has R_x(π); tcp→mount needs R_x(π) so hand_base +Z (fingers) = tcp +Z.
+                 L/R mesh mirror is via direction:=±1 — do not add opposite yaw (fights mirroring). -->
+            <joint name="${side}_hand_base_joint" type="fixed">
+                <origin xyz="0 0 0" rpy="${PI} 0 0"/>
+                <parent link="${side}_tcp"/>
+                <child link="${side}_hand_mount"/>
+            </joint>
+        </xacro:if>
         <xacro:if value="${hand_type == 'xhand1'}">
             <link name="${side}_eef"/>
@@ -123,5 +134,5 @@
             </joint>
         </xacro:if>
-        <xacro:if value="${hand_type in ('linkerhand_o6', 'linkerhand_l6', 'linkerhand_o7', 'freedom_v1', 'freedom_v2', 'inspire_e2', 'inspire_f2', 'theohand_std16a')}">
+        <xacro:if value="${hand_type in ('linkerhand_o6', 'linkerhand_l6', 'linkerhand_o7', 'freedom_v1', 'freedom_v2', 'inspire_e2', 'inspire_f2', 'theohand_std16a', 'wuji_hand2')}">
             <link name="${side}_eef"/>
             <joint name="${side}_eef_joint" type="fixed">
@@ -133,8 +144,8 @@
     <xacro:macro name="SideEndEffector" params="side hand_type gripper_type gripper_pad eef_fixed_joints:=false">
         <xacro:if value="${eef_fixed_joints}">
-            <xacro:if value="${hand_type in ('linkerhand_o6', 'linkerhand_o7', 'linkerhand_l6', 'freedom_v1', 'freedom_v2', 'inspire_e2', 'inspire_f2', 'xhand1', 'theohand_std16a')}">
+            <xacro:if value="${hand_type in ('linkerhand_o6', 'linkerhand_o7', 'linkerhand_l6', 'freedom_v1', 'freedom_v2', 'inspire_e2', 'inspire_f2', 'xhand1', 'theohand_std16a', 'wuji_hand2')}">
                 <xacro:SideEndEffectorLinkerHand side="${side}" hand_type="${hand_type}" eef_fixed_joints="true"/>
             </xacro:if>
-            <xacro:unless value="${hand_type in ('linkerhand_o6', 'linkerhand_o7', 'linkerhand_l6', 'freedom_v1', 'freedom_v2', 'inspire_e2', 'inspire_f2', 'xhand1', 'theohand_std16a')}">
+            <xacro:unless value="${hand_type in ('linkerhand_o6', 'linkerhand_o7', 'linkerhand_l6', 'freedom_v1', 'freedom_v2', 'inspire_e2', 'inspire_f2', 'xhand1', 'theohand_std16a', 'wuji_hand2')}">
                 <xacro:if value="${gripper_type == 'ag2f90_c' or gripper_type == 'ag2f90_d'}">
                     <xacro:AG2F90-C name="${side}" use_flange="true" pad="${gripper_pad}" kinematic_only="true"/>
@@ -210,5 +221,5 @@
                 </joint>
             </xacro:if>
-            <xacro:if value="${hand_type in ('linkerhand_o6', 'linkerhand_o7', 'linkerhand_l6', 'freedom_v1', 'freedom_v2', 'inspire_e2', 'inspire_f2', 'xhand1', 'theohand_std16a')}">
+            <xacro:if value="${hand_type in ('linkerhand_o6', 'linkerhand_o7', 'linkerhand_l6', 'freedom_v1', 'freedom_v2', 'inspire_e2', 'inspire_f2', 'xhand1', 'theohand_std16a', 'wuji_hand2')}">
                 <xacro:SideEndEffectorLinkerHand side="${side}" hand_type="${hand_type}" eef_fixed_joints="false"/>
             </xacro:if>

File: ar5_ccs_description/xacro/ros2_control/end_effector_interfaces.xacro (robot description, xacro)
@@ -9,4 +9,5 @@
     <xacro:include filename="$(find linkerhand_description)/xacro/ros2_control/o7.xacro"/>
     <xacro:include filename="$(find xhand1_description)/xacro/ros2_control/side_systems.xacro"/>
+    <xacro:include filename="$(find wuji_description)/xacro/ros2_control/hand2.xacro"/>
     <xacro:macro name="side_gripper_joint" params="side">
         <joint name="${side}_gripper_joint">
@@ -45,4 +46,7 @@
         <xacro:if value="${hand_type == 'xhand1'}">
             <xacro:xhand1_interfaces name="${side}_hand"/>
+        </xacro:if>
+        <xacro:if value="${hand_type == 'wuji_hand2'}">
+            <xacro:wuji_hand2_interfaces name="${side}_hand"/>
         </xacro:if>
     </xacro:macro>

File: ar5_ccs_description/xacro/ros2_control/external_ee_systems.xacro (robot description, xacro)
@@ -8,4 +8,5 @@
     <xacro:include filename="$(find theohand_description)/xacro/ros2_control/side_systems.xacro"/>
     <xacro:include filename="$(find xhand1_description)/xacro/ros2_control/side_systems.xacro"/>
+    <xacro:include filename="$(find wuji_description)/xacro/ros2_control/side_systems.xacro"/>
     <xacro:macro name="side_usb_hand_system" params="side hand_type serial_port rw_rate:=''">
         <xacro:property name="usb_hand_system_name" value="${str('linkerhand_7' if hand_type == 'linkerhand_o7' else 'linkerhand_6')}"/>
@@ -208,4 +209,10 @@
             <xacro:jodell_usb_side_system side="right" serial_port="${usb_right_port}" rw_rate="${right_ee_rw_rate}"/>
         </xacro:if>
+        <xacro:if value="${left_drive_type == 'ethernet' and left_hand_type == 'wuji_hand2'}">
+            <xacro:wuji_hand2_ethernet_side_system side="left" rw_rate="${left_ee_rw_rate}"/>
+        </xacro:if>
+        <xacro:if value="${right_drive_type == 'ethernet' and right_hand_type == 'wuji_hand2'}">
+            <xacro:wuji_hand2_ethernet_side_system side="right" rw_rate="${right_ee_rw_rate}"/>
+        </xacro:if>
     </xacro:macro>
 </robot>

File: ar5_ccs_description/xacro/ros2_control/robot.xacro (robot description, xacro)
@@ -37,6 +37,6 @@
 	<xacro:property name="validated_hardware_type" value="${1 if '$(arg ros2_control_hardware_type)' in ('mock_components', 'gz', 'isaac', 'real') else 0}"/>
 	<xacro:property name="validated_arm_driver" value="${1 if arm_driver in ('rokae', 'inex') else 0}"/>
-	<xacro:property name="validated_left_drive" value="${1 if arm_driver + ':' + left_drive_type in ('rokae:none', 'rokae:rokae_rs485', 'rokae:usb_rs485', 'rokae:usb_can', 'inex:none', 'inex:inex_rs485', 'inex:inex_can', 'inex:usb_rs485', 'inex:usb_can') else 0}"/>
-	<xacro:property name="validated_right_drive" value="${1 if arm_driver + ':' + right_drive_type in ('rokae:none', 'rokae:rokae_rs485', 'rokae:usb_rs485', 'rokae:usb_can', 'inex:none', 'inex:inex_rs485', 'inex:inex_can', 'inex:usb_rs485', 'inex:usb_can') else 0}"/>
+	<xacro:property name="validated_left_drive" value="${1 if arm_driver + ':' + left_drive_type in ('rokae:none', 'rokae:rokae_rs485', 'rokae:usb_rs485', 'rokae:usb_can', 'rokae:ethernet', 'inex:none', 'inex:inex_rs485', 'inex:inex_can', 'inex:usb_rs485', 'inex:usb_can', 'inex:ethernet') else 0}"/>
+	<xacro:property name="validated_right_drive" value="${1 if arm_driver + ':' + right_drive_type in ('rokae:none', 'rokae:rokae_rs485', 'rokae:usb_rs485', 'rokae:usb_can', 'rokae:ethernet', 'inex:none', 'inex:inex_rs485', 'inex:inex_can', 'inex:usb_rs485', 'inex:usb_can', 'inex:ethernet') else 0}"/>
 	<xacro:property name="rokae_ctrl_mode" value="${'JOINT_IMPEDANCE' if '$(arg arm_ctrl_mode)' == 'joint_impedance' else 'POSITION'}"/>
 	<!-- INEX needs the selected EEF type for payload lookup even when the EEF uses an external bus. -->
