Commit message: develop rokae

File: ar5_ccs_description/xacro/arm_ccs.xacro (robot description, xacro)
@@ -223,5 +223,5 @@
 			<parent link="${prefix}link5"/>
 			<child link="${prefix}link6"/>
-			<limit effort="19" lower="-1.0472" upper="1.0472" velocity="4.1887902047863905"/>
+			<limit effort="19" lower="-0.96" upper="0.96" velocity="4.1887902047863905"/>
 			<axis xyz="0 1 0"/>
 		</joint>
@@ -259,5 +259,5 @@
 			<parent link="${prefix}link6"/>
 			<child link="${prefix}link7"/>
-			<limit effort="19" lower="-1.0472" upper="1.0472" velocity="4.1887902047863905"/>
+			<limit effort="19" lower="-0.96" upper="0.96" velocity="4.1887902047863905"/>
 			<axis xyz="1 0 0"/>
 		</joint>

File: ar5_ccs_description/xacro/ros2_control/robot.xacro (robot description, xacro)
@@ -28,6 +28,6 @@
 	<xacro:property name="right_drive_type" value="${'$(arg right_ee_drive_type)' if '$(arg right_ee_drive_type)' != '' else ee_drive_type}"/>
 	<xacro:property name="rokae_ctrl_mode" value="${'JOINT_IMPEDANCE' if '$(arg arm_ctrl_mode)' == 'joint_impedance' else 'POSITION'}"/>
-	<xacro:property name="left_rokae_hand_type" value="${'' if ee_drive_type == 'usb' else left_hand_type}"/>
-	<xacro:property name="right_rokae_hand_type" value="${'' if ee_drive_type == 'usb' else right_hand_type}"/>
+	<xacro:property name="left_rokae_hand_type" value="${'' if left_drive_type == 'usb' else left_hand_type}"/>
+	<xacro:property name="right_rokae_hand_type" value="${'' if right_drive_type == 'usb' else right_hand_type}"/>
 	<link name="world"/>
 	<joint name="world_fixed" type="fixed">

Commit message: develop ccs_v2

File: ar5_ccs_description/xacro/arm_ccs.xacro (robot description, xacro)
@@ -12,11 +12,11 @@
 			<visual>
 				<geometry>
-					<mesh filename="file://$(find ar5_ccs_description)/meshes/base.glb"/>
-				</geometry>
-			</visual>
-			<xacro:if value="${collider == 'convex'}">
-				<collision>
-					<geometry>
-						<mesh filename="file://$(find ar5_ccs_description)/meshes/base.glb"/>
+					<mesh filename="file://$(find ar5_ccs_description)/meshes/ccs/base.glb"/>
+				</geometry>
+			</visual>
+			<xacro:if value="${collider == 'convex'}">
+				<collision>
+					<geometry>
+						<mesh filename="file://$(find ar5_ccs_description)/meshes/ccs/base.glb"/>
 					</geometry>
 				</collision>
@@ -48,11 +48,11 @@
 			<visual>
 				<geometry>
-					<mesh filename="file://$(find ar5_ccs_description)/meshes/link1.glb" scale="1 ${direction} 1"/>
-				</geometry>
-			</visual>
-			<xacro:if value="${collider == 'convex'}">
-				<collision>
-					<geometry>
-						<mesh filename="file://$(find ar5_ccs_description)/meshes/link1.glb" scale="1 ${direction} 1"/>
+					<mesh filename="file://$(find ar5_ccs_description)/meshes/ccs/link1.glb" scale="1 ${direction} 1"/>
+				</geometry>
+			</visual>
+			<xacro:if value="${collider == 'convex'}">
+				<collision>
+					<geometry>
+						<mesh filename="file://$(find ar5_ccs_description)/meshes/ccs/link1.glb" scale="1 ${direction} 1"/>
 					</geometry>
 				</collision>
@@ -77,11 +77,11 @@
 			<visual>
 				<geometry>
-					<mesh filename="file://$(find ar5_ccs_description)/meshes/link2.glb" scale="1 ${direction} 1"/>
-				</geometry>
-			</visual>
-			<xacro:if value="${collider == 'convex'}">
-				<collision>
-					<geometry>
-						<mesh filename="file://$(find ar5_ccs_description)/meshes/link2.glb" scale="1 ${direction} 1"/>
+					<mesh filename="file://$(find ar5_ccs_description)/meshes/ccs/link2.glb" scale="1 ${direction} 1"/>
+				</geometry>
+			</visual>
+			<xacro:if value="${collider == 'convex'}">
+				<collision>
+					<geometry>
+						<mesh filename="file://$(find ar5_ccs_description)/meshes/ccs/link2.glb" scale="1 ${direction} 1"/>
 					</geometry>
 				</collision>
@@ -120,11 +120,11 @@
 			<visual>
 				<geometry>
-					<mesh filename="file://$(find ar5_ccs_description)/meshes/link3.glb" scale="1 ${direction} 1"/>
-				</geometry>
-			</visual>
-			<xacro:if value="${collider == 'convex'}">
-				<collision>
-					<geometry>
-						<mesh filename="file://$(find ar5_ccs_description)/meshes/link3.glb" scale="1 ${direction} 1"/>
+					<mesh filename="file://$(find ar5_ccs_description)/meshes/ccs/link3.glb" scale="1 ${direction} 1"/>
+				</geometry>
+			</visual>
+			<xacro:if value="${collider == 'convex'}">
+				<collision>
+					<geometry>
+						<mesh filename="file://$(find ar5_ccs_description)/meshes/ccs/link3.glb" scale="1 ${direction} 1"/>
 					</geometry>
 				</collision>
@@ -163,11 +163,11 @@
 			<visual>
 				<geometry>
-					<mesh filename="file://$(find ar5_ccs_description)/meshes/link4.glb" scale="1 ${direction} 1"/>
-				</geometry>
-			</visual>
-			<xacro:if value="${collider == 'convex'}">
-				<collision>
-					<geometry>
-						<mesh filename="file://$(find ar5_ccs_description)/meshes/link4.glb" scale="1 ${direction} 1"/>
+					<mesh filename="file://$(find ar5_ccs_description)/meshes/ccs/link4.glb" scale="1 ${direction} 1"/>
+				</geometry>
+			</visual>
+			<xacro:if value="${collider == 'convex'}">
+				<collision>
+					<geometry>
+						<mesh filename="file://$(find ar5_ccs_description)/meshes/ccs/link4.glb" scale="1 ${direction} 1"/>
 					</geometry>
 				</collision>
@@ -200,11 +200,11 @@
 			<visual>
 				<geometry>
-					<mesh filename="file://$(find ar5_ccs_description)/meshes/link5.glb" scale="1 ${direction} 1"/>
-				</geometry>
-			</visual>
-			<xacro:if value="${collider == 'convex'}">
-				<collision>
-					<geometry>
-						<mesh filename="file://$(find ar5_ccs_description)/meshes/link5.glb" scale="1 ${direction} 1"/>
+					<mesh filename="file://$(find ar5_ccs_description)/meshes/ccs/link5.glb" scale="1 ${direction} 1"/>
+				</geometry>
+			</visual>
+			<xacro:if value="${collider == 'convex'}">
+				<collision>
+					<geometry>
+						<mesh filename="file://$(find ar5_ccs_description)/meshes/ccs/link5.glb" scale="1 ${direction} 1"/>
 					</geometry>
 				</collision>
@@ -236,11 +236,11 @@
 			<visual>
 				<geometry>
-					<mesh filename="file://$(find ar5_ccs_description)/meshes/link6.glb" scale="1 ${direction} 1"/>
-				</geometry>
-			</visual>
-			<xacro:if value="${collider == 'convex'}">
-				<collision>
-					<geometry>
-						<mesh filename="file://$(find ar5_ccs_description)/meshes/link6.glb" scale="1 ${direction} 1"/>
+					<mesh filename="file://$(find ar5_ccs_description)/meshes/ccs/link6.glb" scale="1 ${direction} 1"/>
+				</geometry>
+			</visual>
+			<xacro:if value="${collider == 'convex'}">
+				<collision>
+					<geometry>
+						<mesh filename="file://$(find ar5_ccs_description)/meshes/ccs/link6.glb" scale="1 ${direction} 1"/>
 					</geometry>
 				</collision>
@@ -272,11 +272,11 @@
 			<visual>
 				<geometry>
-					<mesh filename="file://$(find ar5_ccs_description)/meshes/link7.glb" scale="${direction} 1 1"/>
-				</geometry>
-			</visual>
-			<xacro:if value="${collider == 'convex'}">
-				<collision>
-					<geometry>
-						<mesh filename="file://$(find ar5_ccs_description)/meshes/link7.glb" scale=" ${direction} 1 1"/>
+					<mesh filename="file://$(find ar5_ccs_description)/meshes/ccs/link7.glb" scale="${direction} 1 1"/>
+				</geometry>
+			</visual>
+			<xacro:if value="${collider == 'convex'}">
+				<collision>
+					<geometry>
+						<mesh filename="file://$(find ar5_ccs_description)/meshes/ccs/link7.glb" scale=" ${direction} 1 1"/>
 					</geometry>
 				</collision>

File: ar5_ccs_description/xacro/robot.xacro (robot description, xacro)
@@ -2,4 +2,5 @@
 <robot name="AR5_CCS" xmlns:xacro="http://www.ros.org/wiki/xacro">
 	<xacro:arg name="collider" default="convex"/>
+	<xacro:arg name="arm" default="ar5_ccs"/>
 	<xacro:arg name="skin" default="default"/>
 	<xacro:arg name="variant" default=""/>
@@ -44,14 +45,28 @@
 		<xacro:property name="selected_gripper_pad" value="soft"/>
 	</xacro:if>
-	<!-- Include Component Macros -->
-	<xacro:include filename="$(find ar5_ccs_description)/xacro/arm_ccs.xacro"/>
+	<!-- Select the CCS generation while keeping one public description package. -->
+	<xacro:if value="${'$(arg arm)' == 'ar5_ccs'}">
+		<xacro:include filename="$(find ar5_ccs_description)/xacro/arm_ccs.xacro"/>
+	</xacro:if>
+	<xacro:if value="${'$(arg arm)' == 'ar5_ccs_v2'}">
+		<xacro:include filename="$(find ar5_ccs_description)/xacro/arm_ccs_v2.xacro"/>
+	</xacro:if>
+	<xacro:macro name="SelectedAR5CCS" params="name direction collider">
+		<xacro:if value="${'$(arg arm)' == 'ar5_ccs'}">
+			<xacro:AR5_CCS name="${name}" direction="${direction}" collider="${collider}"/>
+		</xacro:if>
+		<xacro:if value="${'$(arg arm)' == 'ar5_ccs_v2'}">
+			<xacro:AR5_CCS_V2 name="${name}" direction="${direction}" collider="${collider}"/>
+		</xacro:if>
+	</xacro:macro>
+	<!-- Include shared component macros. -->
 	<xacro:include filename="$(find ar5_ccs_description)/xacro/arm_mount.xacro"/>
 	<!-- <xacro:include filename="$(find ar5_ccs_description)/xacro/grippers.xacro"/> -->
 	<!-- 根据 arm_config 创建机械臂 -->
 	<xacro:if value="${selected_arm_config == 'left'}">
-		<xacro:AR5_CCS name="" collider="$(arg collider)" direction="1"/>
+		<xacro:SelectedAR5CCS name="" collider="$(arg collider)" direction="1"/>
 	</xacro:if>
 	<xacro:if value="${selected_arm_config == 'right'}">
-		<xacro:AR5_CCS name="" collider="$(arg collider)" direction="-1"/>
+		<xacro:SelectedAR5CCS name="" collider="$(arg collider)" direction="-1"/>
 	</xacro:if>
 	<xacro:if value="${selected_arm_config == 'dual'}">
@@ -70,6 +85,6 @@
 		</joint>
 		<xacro:DualArmMount parent="arm_base"/>
-		<xacro:AR5_CCS name="left" collider="$(arg collider)" direction="1"/>
-		<xacro:AR5_CCS name="right" collider="$(arg collider)" direction="-1"/>
+		<xacro:SelectedAR5CCS name="left" collider="$(arg collider)" direction="1"/>
+		<xacro:SelectedAR5CCS name="right" collider="$(arg collider)" direction="-1"/>
 		<xacro:include filename="$(find ar5_ccs_description)/xacro/eef_type_resolver.xacro"/>
 		<xacro:set_side_eef_types side="left" type_key="${effective_left_type}"/>

Commit message: feat: add joint limit adjustments for eef_fixed_joints in AR5-CCS and SRS configurations

File: ar5_ccs_description/xacro/arm_ccs.xacro (robot description, xacro)
@@ -1,6 +1,10 @@
 <?xml version="1.0" encoding="UTF-8"?>
 <robot xmlns:xacro="http://www.ros.org/wiki/xacro" name="ccs_arm">
+	<!-- Shared with parent robot.xacro; enabled by OCS2 planning URDF generation. -->
+	<xacro:arg name="eef_fixed_joints" default="false"/>
 	<xacro:macro name="AR5_CCS" params="name direction:=1 collider:=convex">
 		<xacro:property name="prefix" value="${name + '_' if name else ''}"/>
+		<!-- Planning keeps positive elbow flexion; visualization / ros2_control retain hardware limits. -->
+		<xacro:property name="joint4_lower" value="${0 if '$(arg eef_fixed_joints)' == 'true' else -1.0472}"/>
 		<!-- Base Link -->
 		<link name="${prefix}base_link">
@@ -149,5 +153,5 @@
 			<parent link="${prefix}link3"/>
 			<child link="${prefix}link4"/>
-			<limit effort="66" lower="-1.0472" upper="2.5307" velocity="5.235987755982989"/>
+			<limit effort="66" lower="${joint4_lower}" upper="2.5307" velocity="5.235987755982989"/>
 			<axis xyz="0 1 0"/>
 			<origin xyz="0.01 0.0 0.0"/>

File: ar5_ccs_description/xacro/arm_ccs_v2.xacro (robot description, xacro)
@@ -1,6 +1,10 @@
 <?xml version="1.0" encoding="UTF-8"?>
 <robot xmlns:xacro="http://www.ros.org/wiki/xacro" name="ccs_arm">
+	<!-- Shared with parent robot.xacro; enabled by OCS2 planning URDF generation. -->
+	<xacro:arg name="eef_fixed_joints" default="false"/>
 	<xacro:macro name="AR5_CCS_V2" params="name direction:=1 collider:=convex skin:='default'">
 		<xacro:property name="prefix" value="${name + '_' if name else ''}"/>
+		<!-- Planning keeps positive elbow flexion; visualization / ros2_control retain hardware limits. -->
+		<xacro:property name="joint4_lower" value="${0 if '$(arg eef_fixed_joints)' == 'true' else -1.0297}"/>
 		<!-- Visual skins live under ar5_ccs_description/meshes/ccs_v2/[fiveages]/ -->
 		<xacro:property name="visual_subdir" value="ccs_v2/"/>
@@ -149,5 +153,5 @@
 			<parent link="${prefix}link3"/>
 			<child link="${prefix}link4"/>
-			<limit effort="66" lower="-1.0297" upper="2.5132" velocity="5.235987755982989"/>
+			<limit effort="66" lower="${joint4_lower}" upper="2.5132" velocity="5.235987755982989"/>
 			<axis xyz="0 1 0"/>
 			<origin xyz="0.0105 0.0 0.0"/>

File: ar5_srs_description/xacro/arm_srs.xacro (robot description, xacro)
@@ -1,7 +1,11 @@
 <?xml version="1.0"?>
 <robot xmlns:xacro="http://www.ros.org/wiki/xacro">
+	<!-- Shared with parent robot.xacro; enabled by OCS2 planning URDF generation. -->
+	<xacro:arg name="eef_fixed_joints" default="false"/>
 	<xacro:property name="PI" value="3.1415926535897931"/>
 	<xacro:macro name="Arm" params="name direction:=1 collider:=convex">
 		<xacro:property name="prefix" value="${name + '_' if name else ''}"/>
+		<!-- Planning keeps positive elbow flexion; visualization / ros2_control retain hardware limits. -->
+		<xacro:property name="joint4_lower" value="${0 if '$(arg eef_fixed_joints)' == 'true' else -1.39}"/>
 		<!-- Arm Base Link -->
 		<link name="${prefix}base_link">
@@ -150,5 +154,5 @@
 			<parent link="${prefix}link3"/>
 			<child link="${prefix}link4"/>
-			<limit effort="66" lower="-1.39" upper="2.50" velocity="5.235987755982989"/>
+			<limit effort="66" lower="${joint4_lower}" upper="2.50" velocity="5.235987755982989"/>
 			<axis xyz="0 1 0"/>
 			<origin xyz="0.01 0.0 0.0"/>
