Commit message: 更新AR5-CCS和AR5-SRS描述，修正参数名称为variant，调整碰撞体位置和关节限制

File: ar5_ccs_description/xacro/arm_ccs_v2.xacro (robot description, xacro)
@@ -127,5 +127,5 @@
 			<xacro:if value="${collider == 'simple'}">
 				<collision>
-					<origin xyz="0 0 -0.0863"/>
+					<origin xyz="0 0 -0.0963"/>
 					<geometry>
 						<cylinder length="0.096" radius="0.053"/>
@@ -254,5 +254,5 @@
 			<parent link="${prefix}link6"/>
 			<child link="${prefix}link7"/>
-			<limit effort="19" lower="-0.96" upper="0.96" velocity="4.1887902047863905"/>
+			<limit effort="19" lower="-0.85" upper="0.85" velocity="4.1887902047863905"/>
 			<axis xyz="1 0 0"/>
 		</joint>
@@ -279,7 +279,7 @@
 			<xacro:if value="${collider == 'simple'}">
 				<collision>
-					<origin xyz="0 0 0.077681"/>
-					<geometry>
-						<cylinder length="0.038669" radius="0.03559"/>
+					<origin xyz="0 0 0.070681"/>
+					<geometry>
+						<cylinder length="0.040" radius="0.03559"/>
 					</geometry>
 				</collision>

File: ar5_ccs_description/xacro/robot.xacro (robot description, xacro)
@@ -2,7 +2,6 @@
 <robot name="AR5_CCS" xmlns:xacro="http://www.ros.org/wiki/xacro">
 	<xacro:arg name="collider" default="convex"/>
-	<xacro:arg name="arm" default="ar5_ccs"/>
 	<xacro:arg name="skin" default="default"/>
-	<xacro:arg name="variant" default=""/>
+	<xacro:arg name="variant" default="base_ar5_ccs"/>
 	<xacro:arg name="type" default="dual"/>
 	<xacro:arg name="left_type" default=""/>
@@ -46,15 +45,15 @@
 	</xacro:if>
 	<!-- Select the CCS generation while keeping one public description package. -->
-	<xacro:if value="${'$(arg arm)' == 'ar5_ccs'}">
+	<xacro:if value="${'$(arg variant)' != 'base_ar5_ccs_v2' and '$(arg variant)' != 'base_ar5_srs'}">
 		<xacro:include filename="$(find ar5_ccs_description)/xacro/arm_ccs.xacro"/>
 	</xacro:if>
-	<xacro:if value="${'$(arg arm)' == 'ar5_ccs_v2'}">
+	<xacro:if value="${'$(arg variant)' == 'base_ar5_ccs_v2'}">
 		<xacro:include filename="$(find ar5_ccs_description)/xacro/arm_ccs_v2.xacro"/>
 	</xacro:if>
 	<xacro:macro name="SelectedAR5CCS" params="name direction collider">
-		<xacro:if value="${'$(arg arm)' == 'ar5_ccs'}">
+		<xacro:if value="${'$(arg variant)' != 'base_ar5_ccs_v2' and '$(arg variant)' != 'base_ar5_srs'}">
 			<xacro:AR5_CCS name="${name}" direction="${direction}" collider="${collider}"/>
 		</xacro:if>
-		<xacro:if value="${'$(arg arm)' == 'ar5_ccs_v2'}">
+		<xacro:if value="${'$(arg variant)' == 'base_ar5_ccs_v2'}">
 			<xacro:AR5_CCS_V2 name="${name}" direction="${direction}" collider="${collider}"/>
 		</xacro:if>
@@ -74,5 +73,5 @@
 		<link name="arm_base">
 			<collision>
-				<origin xyz="0.0091 0 -0.096"/>
+				<origin xyz="0.0091 0 -0.2"/>
 				<geometry>
 					<box size="0.33 0.30 0.5029"/>

File: ar5_srs_description/xacro/robot.xacro (robot description, xacro)
@@ -53,5 +53,5 @@
 		<link name="arm_base">
 			<collision>
-				<origin xyz="0.0091 0 -0.086"/>
+				<origin xyz="0.0091 0 -0.2"/>
 				<geometry>
 					<box size="0.2509 0.35 0.5029"/>

Commit message: add fiveages color

File: ar5_ccs_description/xacro/arm_ccs_v2.xacro (robot description, xacro)
@@ -1,6 +1,11 @@
 <?xml version="1.0" encoding="UTF-8"?>
 <robot xmlns:xacro="http://www.ros.org/wiki/xacro" name="ccs_arm">
-	<xacro:macro name="AR5_CCS_V2" params="name direction:=1 collider:=convex">
+	<xacro:macro name="AR5_CCS_V2" params="name direction:=1 collider:=convex skin:='default'">
 		<xacro:property name="prefix" value="${name + '_' if name else ''}"/>
+		<!-- Visual skins live under ar5_ccs_description/meshes/ccs_v2/[fiveages]/ -->
+		<xacro:property name="visual_subdir" value="ccs_v2/"/>
+		<xacro:if value="${skin == 'fiveages'}">
+			<xacro:property name="visual_subdir" value="ccs_v2/fiveages/"/>
+		</xacro:if>
 		<!-- Base Link -->
 		<link name="${prefix}base_link">
@@ -43,5 +48,5 @@
 			<visual>
 				<geometry>
-					<mesh filename="file://$(find ar5_ccs_description)/meshes/ccs_v2/link1.glb" scale="1 ${direction} 1"/>
+					<mesh filename="file://$(find ar5_ccs_description)/meshes/${visual_subdir}link1.glb" scale="1 ${direction} 1"/>
 				</geometry>
 			</visual>
@@ -72,5 +77,5 @@
 			<visual>
 				<geometry>
-					<mesh filename="file://$(find ar5_ccs_description)/meshes/ccs_v2/link2.glb" scale="1 ${direction} 1"/>
+					<mesh filename="file://$(find ar5_ccs_description)/meshes/${visual_subdir}link2.glb" scale="1 ${direction} 1"/>
 				</geometry>
 			</visual>
@@ -115,5 +120,5 @@
 			<visual>
 				<geometry>
-					<mesh filename="file://$(find ar5_ccs_description)/meshes/ccs_v2/link3.glb" scale="1 ${direction} 1"/>
+					<mesh filename="file://$(find ar5_ccs_description)/meshes/${visual_subdir}link3.glb" scale="1 ${direction} 1"/>
 				</geometry>
 			</visual>
@@ -158,5 +163,5 @@
 			<visual>
 				<geometry>
-					<mesh filename="file://$(find ar5_ccs_description)/meshes/ccs_v2/link4.glb" scale="1 ${direction} 1"/>
+					<mesh filename="file://$(find ar5_ccs_description)/meshes/${visual_subdir}link4.glb" scale="1 ${direction} 1"/>
 				</geometry>
 			</visual>
@@ -195,5 +200,5 @@
 			<visual>
 				<geometry>
-					<mesh filename="file://$(find ar5_ccs_description)/meshes/ccs_v2/link5.glb" scale="1 ${direction} 1"/>
+					<mesh filename="file://$(find ar5_ccs_description)/meshes/${visual_subdir}link5.glb" scale="1 ${direction} 1"/>
 				</geometry>
 			</visual>
@@ -231,5 +236,5 @@
 			<visual>
 				<geometry>
-					<mesh filename="file://$(find ar5_ccs_description)/meshes/ccs_v2/link6.glb" scale="1 ${direction} 1"/>
+					<mesh filename="file://$(find ar5_ccs_description)/meshes/${visual_subdir}link6.glb" scale="1 ${direction} 1"/>
 				</geometry>
 			</visual>
@@ -267,5 +272,5 @@
 			<visual>
 				<geometry>
-					<mesh filename="file://$(find ar5_ccs_description)/meshes/ccs_v2/link7.glb" scale="1 ${direction} 1"/>
+					<mesh filename="file://$(find ar5_ccs_description)/meshes/${visual_subdir}link7.glb" scale="1 ${direction} 1"/>
 				</geometry>
 			</visual>

File: ar5_ccs_description/xacro/robot.xacro (robot description, xacro)
@@ -60,5 +60,5 @@
 		</xacro:if>
 		<xacro:if value="${'$(arg variant)' == 'ar5_ccs_v2'}">
-			<xacro:AR5_CCS_V2 name="${name}" direction="${direction}" collider="${collider}"/>
+			<xacro:AR5_CCS_V2 name="${name}" direction="${direction}" collider="${collider}" skin="$(arg skin)"/>
 		</xacro:if>
 	</xacro:macro>

Commit message: feat: update joint limits for improved arm motion control

File: ar5_ccs_description/xacro/arm_ccs_v2.xacro (robot description, xacro)
@@ -35,5 +35,5 @@
 			<parent link="${prefix}base_link"/>
 			<child link="${prefix}link1"/>
-			<limit effort="108" lower="-3.1067" upper="3.1067" velocity="3.0543261909900763"/>
+			<limit effort="108" lower="-3.0892" upper="3.0892" velocity="3.0543261909900763"/>
 			<axis xyz="0 0 1"/>
 		</joint>
@@ -63,5 +63,5 @@
 			<parent link="${prefix}link1"/>
 			<child link="${prefix}link2"/>
-			<limit effort="108" lower="-2.0944" upper="2.0944" velocity="3.0543261909900763"/>
+			<limit effort="108" lower="-2.0769" upper="2.0769" velocity="3.0543261909900763"/>
 			<axis xyz="0 1 0"/>
 			<origin xyz="0.0 0.0 0.1745"/>
@@ -106,5 +106,5 @@
 			<parent link="${prefix}link2"/>
 			<child link="${prefix}link3"/>
-			<limit effort="66" lower="-3.1067" upper="3.1067" velocity="4.71238898038469"/>
+			<limit effort="66" lower="-3.0892" upper="3.0892" velocity="4.71238898038469"/>
 			<axis xyz="0 0 1"/>
 			<origin xyz="0.0 0.0 0.332"/>
@@ -149,5 +149,5 @@
 			<parent link="${prefix}link3"/>
 			<child link="${prefix}link4"/>
-			<limit effort="66" lower="-1.0472" upper="2.5307" velocity="5.235987755982989"/>
+			<limit effort="66" lower="-1.0297" upper="2.5132" velocity="5.235987755982989"/>
 			<axis xyz="0 1 0"/>
 			<origin xyz="0.0105 0.0 0.0"/>
@@ -186,5 +186,5 @@
 			<parent link="${prefix}link4"/>
 			<child link="${prefix}link5"/>
-			<limit effort="19" lower="-3.1067" upper="3.1067" velocity="4.1887902047863905"/>
+			<limit effort="19" lower="-3.0892" upper="3.0892" velocity="4.1887902047863905"/>
 			<axis xyz="0 0 1"/>
 			<origin xyz="-0.0105 0.0 0.278"/>

Commit message: feat: update joint 6 limits for improved motion control

File: ar5_ccs_description/xacro/arm_ccs_v2.xacro (robot description, xacro)
@@ -223,5 +223,5 @@
 			<parent link="${prefix}link5"/>
 			<child link="${prefix}link6"/>
-			<limit effort="19" lower="-0.96" upper="0.96" velocity="4.1887902047863905"/>
+			<limit effort="19" lower="-0.85" upper="0.85" velocity="4.1887902047863905"/>
 			<axis xyz="0 1 0"/>
 		</joint>
