Commit message: 1

File: ar5_ccs_description/urdf/ar5_ccs_ag2f90_d.urdf (robot description, URDF)
Before this commit: robot AR5_CCS, 46 links, 45 joints
Links:
- link left_flange: geometry visual mesh filename=package://changingtek_description/meshes/AG2F90-C/visual/fl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
- link left_gripper_base: geometry visual mesh filename=package://changingtek_description/meshes/AG2F90-C/visual/gr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
- link left_left_1_link: geometry visual mesh filename=package://changingtek_description/meshes/AG2F90-C/visual/li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
- link left_left_2_link: geometry visual mesh filename=package://changingtek_description/meshes/AG2F90-C/visual/li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
- link left_left_in_link: geometry visual mesh filename=package://changingtek_description/meshes/AG2F90-C/visual/in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
- link left_left_up_link: geometry visual mesh filename=package://changingtek_description/meshes/AG2F90-C/visual/up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
- link left_right_1_link: geometry visual mesh filename=package://changingtek_description/meshes/AG2F90-C/visual/li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
- link left_right_2_link: geometry visual mesh filename=package://changingtek_description/meshes/AG2F90-C/visual/li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
- link left_right_in_link: geometry visual mesh filename=package://changingtek_description/meshes/AG2F90-C/visual/in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
- link left_right_up_link: geometry visual mesh filename=package://changingtek_description/meshes/AG2F90-C/visual/up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
- link right_flange: geometry visual mesh filename=package://changingtek_description/meshes/AG2F90-C/visual/fl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
- link right_gripper_base: geometry visual mesh filename=package://changingtek_description/meshes/AG2F90-C/visual/gr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
- link right_left_1_link: geometry visual mesh filename=package://changingtek_description/meshes/AG2F90-C/visual/li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
- link right_left_2_link: geometry visual mesh filename=package://changingtek_description/meshes/AG2F90-C/visual/li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
- link right_left_in_link: geometry visual mesh filename=package://changingtek_description/meshes/AG2F90-C/visual/in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
- link right_left_up_link: geometry visual mesh filename=package://changingtek_description/meshes/AG2F90-C/visual/up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
- link right_right_1_link: geometry visual mesh filename=package://changingtek_description/meshes/AG2F90-C/visual/li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
- link right_right_2_link: geometry visual mesh filename=package://changingtek_description/meshes/AG2F90-C/visual/li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
- link right_right_in_link: geometry visual mesh filename=package://changingtek_description/meshes/AG2F90-C/visual/in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
- link right_right_up_link: geometry visual mesh filename=package://changingtek_description/meshes/AG2F90-C/visual/up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

Commit message: fix urdf and xacro

File: ar5_ccs_description/urdf/ar5_ccs_ag2f90_d.urdf (robot description, URDF)
Before this commit: robot AR5_CCS, 46 links, 45 joints
Links:
- link left_left_Pad_link: mass None -> 0.0183171479595721; geometry visual mesh filename=package://changingtek_description/meshes/AG2F90-C/visual/pa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
- link left_right_Pad_link: mass None -> 0.0183171479595721; geometry visual mesh filename=package://changingtek_description/meshes/AG2F90-C/visual/pa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
- link right_left_Pad_link: mass None -> 0.0183171479595721; geometry visual mesh filename=package://changingtek_description/meshes/AG2F90-C/visual/pa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
- link right_right_Pad_link: mass None -> 0.0183171479595721; geometry visual mesh filename=package://changingtek_description/meshes/AG2F90-C/visual/pa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
Joints:
- joint left_eef_joint: origin (none) -> xyz=0 0 0.19
- joint left_gripper_base_joint: origin xyz=0 0 0 -> xyz=0 0 -0.0045
- joint right_eef_joint: origin (none) -> xyz=0 0 0.19
- joint right_gripper_base_joint: origin xyz=0 0 0 -> xyz=0 0 -0.0045

File: ar5_ccs_description/xacro/grippers.xacro (robot description, xacro)
@@ -48,5 +48,5 @@
             <xacro:include filename="$(find changingtek_description)/xacro/AG2F90-C.xacro"/>
             <xacro:if value="${arm_config == 'left'}">
-                <xacro:AG2F90-C name="" use_flange="true" pad="none"/>
+                <xacro:AG2F90-C name="" use_flange="true"/>
                 <joint name="gripper_base_joint" type="fixed">
                     <origin xyz="0 0 0" rpy="0 0 -1.5708"/>
@@ -56,5 +56,5 @@
             </xacro:if>
             <xacro:if value="${arm_config == 'right'}">
-                <xacro:AG2F90-C name="" use_flange="true" pad="none"/>
+                <xacro:AG2F90-C name="" use_flange="true"/>
                 <joint name="gripper_base_joint" type="fixed">
                     <origin xyz="0 0 0" rpy="0 0 1.5708"/>
@@ -64,6 +64,6 @@
             </xacro:if>
             <xacro:if value="${arm_config == 'dual'}">
-                <xacro:AG2F90-C name="left" use_flange="true" pad="none"/>
-                <xacro:AG2F90-C name="right" use_flange="true" pad="none"/>
+                <xacro:AG2F90-C name="left" use_flange="true"/>
+                <xacro:AG2F90-C name="right" use_flange="true"/>
                 <joint name="left_gripper_base_joint" type="fixed">
                     <origin xyz="0 0 0"/>

File: ar5_ccs_description/xacro/ros2_control/robot.xacro (robot description, xacro)
@@ -33,4 +33,7 @@
 						<param name="gripper_max_opening_distance">1.0</param>
 						<param name="gripper_configure_xpanel">false</param>
+						<param name="load_mass">0.0</param>
+					        <param name="load_cog">[0.0, 0.0, 0.0]</param>
+					        <param name="load_inertia">[0.0, 0.0, 0.0]</param>
 					</xacro:if>
 				</hardware>
@@ -63,4 +66,7 @@
 						<param name="gripper_max_opening_distance">1.0</param>
 						<param name="gripper_configure_xpanel">false</param>
+						<param name="load_mass">0.75</param>
+						<param name="load_cog">[-0.01, -0.03, 0.09]</param>
+						<param name="load_inertia">[0.0, 0.0, 0.0]</param>
 					</xacro:if>
 				</hardware>
