Commit message: Add tool load parameters for left and right arms in robot.xacro

File: ar5_ccs_description/xacro/ros2_control/robot.xacro (robot description, xacro)
@@ -8,13 +8,14 @@
 	<xacro:arg name="left_arm_cpu_affinity" default="2"/>
 	<xacro:arg name="right_arm_cpu_affinity" default="3"/>
+	<xacro:arg name="left_load_mass" default=""/>
+	<xacro:arg name="left_load_cog" default=""/>
+	<xacro:arg name="left_load_inertia" default=""/>
+	<xacro:arg name="right_load_mass" default=""/>
+	<xacro:arg name="right_load_cog" default=""/>
+	<xacro:arg name="right_load_inertia" default=""/>
 	<xacro:arg name="rokae_command_filter_mode" default="double_s"/>
 	<xacro:arg name="rokae_command_filter_max_velocity" default="6.0"/>
 	<xacro:arg name="rokae_command_filter_max_acceleration" default="30.0"/>
 	<xacro:arg name="rokae_command_filter_max_jerk" default="300.0"/>
-	<xacro:arg name="rokae_sdk_filter_limit_enable" default="true"/>
-	<xacro:arg name="rokae_sdk_filter_limit" default="10"/>
-	<xacro:arg name="rokae_sdk_filter_frequency_1" default="10"/>
-	<xacro:arg name="rokae_sdk_filter_frequency_2" default="10"/>
-	<xacro:arg name="rokae_sdk_filter_frequency_3" default="10"/>
 	<link name="world"/>
 	<joint name="world_fixed" type="fixed">
@@ -92,4 +93,15 @@
 		</xacro:if>
 	</xacro:macro>
+	<xacro:macro name="rokae_tool_load_params_with_override" params="side gripper_type gripper_pad load_mass load_cog load_inertia">
+		<xacro:property name="has_tool_load_override" value="${load_mass != '' and load_cog != '' and load_inertia != ''}"/>
+		<xacro:if value="${has_tool_load_override}">
+			<param name="load_mass">${load_mass}</param>
+			<param name="load_cog">${load_cog}</param>
+			<param name="load_inertia">${load_inertia}</param>
+		</xacro:if>
+		<xacro:unless value="${has_tool_load_override}">
+			<xacro:rokae_tool_load_params side="${side}" gripper_type="${gripper_type}" gripper_pad="${gripper_pad}"/>
+		</xacro:unless>
+	</xacro:macro>
 	<!-- 使用 robot.xacro 中已定义的 property 来判断 -->
 	<!-- selected_arm_config: left, right, dual -->
@@ -109,9 +121,4 @@
 					<param name="command_filter_max_acceleration">$(arg rokae_command_filter_max_acceleration)</param>
 					<param name="command_filter_max_jerk">$(arg rokae_command_filter_max_jerk)</param>
-					<param name="sdk_filter_limit_enable">$(arg rokae_sdk_filter_limit_enable)</param>
-					<param name="sdk_filter_limit">$(arg rokae_sdk_filter_limit)</param>
-					<param name="sdk_filter_frequency_1">$(arg rokae_sdk_filter_frequency_1)</param>
-					<param name="sdk_filter_frequency_2">$(arg rokae_sdk_filter_frequency_2)</param>
-					<param name="sdk_filter_frequency_3">$(arg rokae_sdk_filter_frequency_3)</param>
 					<xacro:if value="${left_gripper_type == 'rg75'}">
 						<param name="gripper_type">jodell</param>
@@ -129,5 +136,6 @@
 					</xacro:if>
 					<xacro:if value="${left_gripper_type != ''}">
-						<xacro:rokae_tool_load_params side="left" gripper_type="${left_gripper_type}" gripper_pad="${left_gripper_pad}"/>
+						<xacro:rokae_tool_load_params_with_override side="left" gripper_type="${left_gripper_type}" gripper_pad="${left_gripper_pad}"
+																   load_mass="$(arg left_load_mass)" load_cog="$(arg left_load_cog)" load_inertia="$(arg left_load_inertia)"/>
 					</xacro:if>
 				</hardware>
@@ -156,9 +164,4 @@
 					<param name="command_filter_max_acceleration">$(arg rokae_command_filter_max_acceleration)</param>
 					<param name="command_filter_max_jerk">$(arg rokae_command_filter_max_jerk)</param>
-					<param name="sdk_filter_limit_enable">$(arg rokae_sdk_filter_limit_enable)</param>
-					<param name="sdk_filter_limit">$(arg rokae_sdk_filter_limit)</param>
-					<param name="sdk_filter_frequency_1">$(arg rokae_sdk_filter_frequency_1)</param>
-					<param name="sdk_filter_frequency_2">$(arg rokae_sdk_filter_frequency_2)</param>
-					<param name="sdk_filter_frequency_3">$(arg rokae_sdk_filter_frequency_3)</param>
 					<xacro:if value="${right_gripper_type == 'rg75'}">
 						<param name="gripper_type">jodell</param>
@@ -176,5 +179,6 @@
 					</xacro:if>
 					<xacro:if value="${right_gripper_type != ''}">
-						<xacro:rokae_tool_load_params side="right" gripper_type="${right_gripper_type}" gripper_pad="${right_gripper_pad}"/>
+						<xacro:rokae_tool_load_params_with_override side="right" gripper_type="${right_gripper_type}" gripper_pad="${right_gripper_pad}"
+																   load_mass="$(arg right_load_mass)" load_cog="$(arg right_load_cog)" load_inertia="$(arg right_load_inertia)"/>
 					</xacro:if>
 				</hardware>
@@ -216,9 +220,4 @@
 					<param name="command_filter_max_acceleration">$(arg rokae_command_filter_max_acceleration)</param>
 					<param name="command_filter_max_jerk">$(arg rokae_command_filter_max_jerk)</param>
-					<param name="sdk_filter_limit_enable">$(arg rokae_sdk_filter_limit_enable)</param>
-					<param name="sdk_filter_limit">$(arg rokae_sdk_filter_limit)</param>
-					<param name="sdk_filter_frequency_1">$(arg rokae_sdk_filter_frequency_1)</param>
-					<param name="sdk_filter_frequency_2">$(arg rokae_sdk_filter_frequency_2)</param>
-					<param name="sdk_filter_frequency_3">$(arg rokae_sdk_filter_frequency_3)</param>
 					<xacro:if value="${selected_gripper_type == 'rg75'}">
 						<param name="gripper_type">jodell</param>
@@ -236,5 +235,8 @@
 					</xacro:if>
 					<xacro:if value="${selected_gripper_type != ''}">
-						<xacro:rokae_tool_load_params side="${'left' if selected_arm_config == 'left' else 'right'}" gripper_type="${selected_gripper_type}" gripper_pad="${selected_gripper_pad}"/>
+						<xacro:rokae_tool_load_params_with_override side="${'left' if selected_arm_config == 'left' else 'right'}" gripper_type="${selected_gripper_type}" gripper_pad="${selected_gripper_pad}"
+																   load_mass="${'$(arg left_load_mass)' if selected_arm_config == 'left' else '$(arg right_load_mass)'}"
+																   load_cog="${'$(arg left_load_cog)' if selected_arm_config == 'left' else '$(arg right_load_cog)'}"
+																   load_inertia="${'$(arg left_load_inertia)' if selected_arm_config == 'left' else '$(arg right_load_inertia)'}"/>
 					</xacro:if>
 				</hardware>

Commit message: Add dynamic control mode handling for robot arms in robot.xacro

File: ar5_ccs_description/xacro/ros2_control/robot.xacro (robot description, xacro)
@@ -2,4 +2,5 @@
 <robot xmlns:xacro="http://www.ros.org/wiki/xacro" name="AR5_CCS">
 	<xacro:arg name="ros2_control_hardware_type" default="mock_components"/>
+	<xacro:arg name="arm_ctrl_mode" default="position"/>
 	<xacro:arg name="left_arm_ip" default="192.168.1.160"/>
 	<xacro:arg name="left_local_ip" default="192.168.1.233"/>
@@ -18,4 +19,5 @@
 	<xacro:arg name="rokae_command_filter_max_acceleration" default="30.0"/>
 	<xacro:arg name="rokae_command_filter_max_jerk" default="300.0"/>
+	<xacro:property name="rokae_ctrl_mode" value="${'JOINT_IMPEDANCE' if '$(arg arm_ctrl_mode)' == 'joint_impedance' else 'POSITION'}"/>
 	<link name="world"/>
 	<joint name="world_fixed" type="fixed">
@@ -113,5 +115,5 @@
 					<plugin>rokae_ros2_control/RokaeHardware</plugin>
 					<param name="arm_ip">$(arg left_arm_ip)</param>
-					<param name="ctrl_mode">POSITION</param>
+					<param name="ctrl_mode">${rokae_ctrl_mode}</param>
 					<param name="joint_impedance">200,200,200,200,20,20,20</param>
 					<param name="local_ip">$(arg left_local_ip)</param>
@@ -156,5 +158,5 @@
 					<plugin>rokae_ros2_control/RokaeHardware</plugin>
 					<param name="arm_ip">$(arg right_arm_ip)</param>
-					<param name="ctrl_mode">POSITION</param>
+					<param name="ctrl_mode">${rokae_ctrl_mode}</param>
 					<param name="joint_impedance">200,200,200,200,20,20,20</param>
 					<param name="local_ip">$(arg right_local_ip)</param>
@@ -207,5 +209,5 @@
 						<param name="arm_ip">$(arg right_arm_ip)</param>
 					</xacro:if>
-					<param name="ctrl_mode">POSITION</param>
+					<param name="ctrl_mode">${rokae_ctrl_mode}</param>
 					<param name="joint_impedance">200,200,200,200,20,20,20</param>
 					<xacro:if value="${selected_arm_config == 'left'}">
