Commit message: feat: enhance INEX support by adding tool load parameters and updating hardware configurations

File: ar5_ccs_description/xacro/ros2_control/arm_hardware.xacro (robot description, xacro)
@@ -1,4 +1,5 @@
 <?xml version="1.0"?>
 <robot xmlns:xacro="http://www.ros.org/wiki/xacro">
+    <xacro:include filename="$(find ar5_ccs_description)/xacro/ros2_control/tool_load.xacro"/>
     <xacro:include filename="$(find ar5_ccs_description)/xacro/ros2_control/rokae_hardware.xacro"/>
     <xacro:include filename="$(find ar5_ccs_description)/xacro/ros2_control/inex_hardware.xacro"/>
@@ -15,5 +16,8 @@
                 state_timeout_ms="${state_timeout_ms}"
                 command_hold_timeout_ms="${command_hold_timeout_ms}"
-                command_fault_timeout_ms="${command_fault_timeout_ms}"/>
+                command_fault_timeout_ms="${command_fault_timeout_ms}"
+                gripper_type="${gripper_type}" gripper_pad="${gripper_pad}"
+                hand_type="${hand_type}" load_mass="${load_mass}"
+                load_cog="${load_cog}" load_inertia="${load_inertia}"/>
         </xacro:if>
         <xacro:if value="${driver == 'rokae'}">

File: ar5_ccs_description/xacro/ros2_control/inex_hardware.xacro (robot description, xacro)
@@ -8,5 +8,11 @@
         state_timeout_ms
         command_hold_timeout_ms
-        command_fault_timeout_ms">
+        command_fault_timeout_ms
+        gripper_type
+        gripper_pad
+        hand_type
+        load_mass
+        load_cog
+        load_inertia">
         <plugin>inex_ros2_control/InexSystemHardware</plugin>
         <param name="side">${side}</param>
@@ -22,4 +28,11 @@
         <param name="require_realtime">true</param>
         <param name="lock_memory">true</param>
+        <xacro:tool_load_params
+            side="${side}"
+            end_effector_type="${gripper_type if gripper_type != '' else hand_type}"
+            pad_type="${gripper_pad}"
+            mass="${load_mass}"
+            center_of_mass="${load_cog}"
+            diagonal_inertia="${load_inertia}"/>
     </xacro:macro>
 </robot>

File: ar5_ccs_description/xacro/ros2_control/robot.xacro (robot description, xacro)
@@ -40,8 +40,9 @@
 	<xacro:property name="validated_right_drive" value="${1 if arm_driver + ':' + right_drive_type in ('rokae:none', 'rokae:rokae_rs485', 'rokae:usb_rs485', 'rokae:usb_can', 'inex:none', 'inex:inex_rs485', 'inex:inex_can', 'inex:usb_rs485', 'inex:usb_can') else 0}"/>
 	<xacro:property name="rokae_ctrl_mode" value="${'JOINT_IMPEDANCE' if '$(arg arm_ctrl_mode)' == 'joint_impedance' else 'POSITION'}"/>
-	<xacro:property name="left_rokae_hand_type" value="${left_hand_type if arm_driver == 'rokae' and left_drive_type == 'rokae_rs485' else ''}"/>
-	<xacro:property name="right_rokae_hand_type" value="${right_hand_type if arm_driver == 'rokae' and right_drive_type == 'rokae_rs485' else ''}"/>
-	<xacro:property name="left_rokae_gripper_type" value="${left_gripper_type if arm_driver == 'rokae' and left_drive_type == 'rokae_rs485' else ''}"/>
-	<xacro:property name="right_rokae_gripper_type" value="${right_gripper_type if arm_driver == 'rokae' and right_drive_type == 'rokae_rs485' else ''}"/>
+	<!-- INEX needs the selected EEF type for payload lookup even when the EEF uses an external bus. -->
+	<xacro:property name="left_arm_hand_type" value="${left_hand_type if arm_driver == 'inex' or left_drive_type == 'rokae_rs485' else ''}"/>
+	<xacro:property name="right_arm_hand_type" value="${right_hand_type if arm_driver == 'inex' or right_drive_type == 'rokae_rs485' else ''}"/>
+	<xacro:property name="left_arm_gripper_type" value="${left_gripper_type if arm_driver == 'inex' or left_drive_type == 'rokae_rs485' else ''}"/>
+	<xacro:property name="right_arm_gripper_type" value="${right_gripper_type if arm_driver == 'inex' or right_drive_type == 'rokae_rs485' else ''}"/>
 	<link name="world"/>
 	<joint name="world_fixed" type="fixed">
@@ -66,8 +67,8 @@
 						command_filter_mode="$(arg rokae_command_filter_mode)" command_filter_max_velocity="$(arg rokae_command_filter_max_velocity)"
 						command_filter_max_acceleration="$(arg rokae_command_filter_max_acceleration)" command_filter_max_jerk="$(arg rokae_command_filter_max_jerk)"
-						gripper_type="${left_rokae_gripper_type}" gripper_pad="${left_gripper_pad}" hand_type="${left_rokae_hand_type}"
+						gripper_type="${left_arm_gripper_type}" gripper_pad="${left_gripper_pad}" hand_type="${left_arm_hand_type}"
 						load_mass="$(arg left_load_mass)" load_cog="$(arg left_load_cog)" load_inertia="$(arg left_load_inertia)"/>
 				</hardware>
-				<xacro:if value="${arm_driver == 'rokae' and left_drive_type == 'rokae_rs485'}"><xacro:side_arm_ee_block side="left" mode="real" hand_type="${left_rokae_hand_type}" gripper_type="${left_rokae_gripper_type}"/></xacro:if>
+				<xacro:if value="${arm_driver == 'rokae' and left_drive_type == 'rokae_rs485'}"><xacro:side_arm_ee_block side="left" mode="real" hand_type="${left_arm_hand_type}" gripper_type="${left_arm_gripper_type}"/></xacro:if>
 				<xacro:unless value="${arm_driver == 'rokae' and left_drive_type == 'rokae_rs485'}"><xacro:ar5_interfaces name="left"/></xacro:unless>
 			</ros2_control>
@@ -79,8 +80,8 @@
 						command_filter_mode="$(arg rokae_command_filter_mode)" command_filter_max_velocity="$(arg rokae_command_filter_max_velocity)"
 						command_filter_max_acceleration="$(arg rokae_command_filter_max_acceleration)" command_filter_max_jerk="$(arg rokae_command_filter_max_jerk)"
-						gripper_type="${right_rokae_gripper_type}" gripper_pad="${right_gripper_pad}" hand_type="${right_rokae_hand_type}"
+						gripper_type="${right_arm_gripper_type}" gripper_pad="${right_gripper_pad}" hand_type="${right_arm_hand_type}"
 						load_mass="$(arg right_load_mass)" load_cog="$(arg right_load_cog)" load_inertia="$(arg right_load_inertia)"/>
 				</hardware>
-				<xacro:if value="${arm_driver == 'rokae' and right_drive_type == 'rokae_rs485'}"><xacro:side_arm_ee_block side="right" mode="real" hand_type="${right_rokae_hand_type}" gripper_type="${right_rokae_gripper_type}"/></xacro:if>
+				<xacro:if value="${arm_driver == 'rokae' and right_drive_type == 'rokae_rs485'}"><xacro:side_arm_ee_block side="right" mode="real" hand_type="${right_arm_hand_type}" gripper_type="${right_arm_gripper_type}"/></xacro:if>
 				<xacro:unless value="${arm_driver == 'rokae' and right_drive_type == 'rokae_rs485'}"><xacro:ar5_interfaces name="right"/></xacro:unless>
 			</ros2_control>
@@ -96,7 +97,7 @@
 						command_filter_mode="$(arg rokae_command_filter_mode)" command_filter_max_velocity="$(arg rokae_command_filter_max_velocity)"
 						command_filter_max_acceleration="$(arg rokae_command_filter_max_acceleration)" command_filter_max_jerk="$(arg rokae_command_filter_max_jerk)"
-						gripper_type="${left_rokae_gripper_type if selected_arm_config == 'left' else right_rokae_gripper_type}"
+						gripper_type="${left_arm_gripper_type if selected_arm_config == 'left' else right_arm_gripper_type}"
 						gripper_pad="${left_gripper_pad if selected_arm_config == 'left' else right_gripper_pad}"
-						hand_type="${left_rokae_hand_type if selected_arm_config == 'left' else right_rokae_hand_type}"
+						hand_type="${left_arm_hand_type if selected_arm_config == 'left' else right_arm_hand_type}"
 						load_mass="${'$(arg left_load_mass)' if selected_arm_config == 'left' else '$(arg right_load_mass)'}"
 						load_cog="${'$(arg left_load_cog)' if selected_arm_config == 'left' else '$(arg right_load_cog)'}"

File: ar5_ccs_description/xacro/ros2_control/rokae_hardware.xacro (robot description, xacro)
@@ -1,82 +1,4 @@
 <?xml version="1.0"?>
 <robot xmlns:xacro="http://www.ros.org/wiki/xacro">
-    <!--
-        Default Rokae tool load table by gripper/pad.
-        All values are intentionally zero placeholders. Fill the real values here
-        when the measured mass/CoG/inertia for each end effector is available.
-    -->
-    <xacro:macro name="rokae_tool_load_params" params="side gripper_type gripper_pad">
-        <!-- Left RG75, default pad: TODO fill measured load. -->
-        <xacro:if value="${side == 'left' and gripper_type == 'rg75' and gripper_pad != 'heavy_carry'}">
-            <param name="load_mass">1.62</param>
-            <param name="load_cog">[-0.0014285, 0.000579, 0.10439]</param>
-            <param name="load_inertia">[0.04874, 0.001, 0.001936]</param>
-        </xacro:if>
-        <!-- Left RG75, heavy_carry pad: TODO fill measured load. -->
-        <xacro:if value="${side == 'left' and gripper_type == 'rg75' and gripper_pad == 'heavy_carry'}">
-            <param name="load_mass">0.0</param>
-            <param name="load_cog">[0.0, 0.0, 0.0]</param>
-            <param name="load_inertia">[0.0, 0.0, 0.0]</param>
-        </xacro:if>
-        <!-- Left AG2F90-C, default pad: TODO fill measured load. -->
-        <xacro:if value="${side == 'left' and gripper_type == 'ag2f90_c' and gripper_pad != 'soft'}">
-            <param name="load_mass">0.0</param>
-            <param name="load_cog">[0.0, 0.0, 0.0]</param>
-            <param name="load_inertia">[0.0, 0.0, 0.0]</param>
-        </xacro:if>
-        <!-- Left AG2F90-C, soft pad: TODO fill measured load. -->
-        <xacro:if value="${side == 'left' and gripper_type == 'ag2f90_c' and gripper_pad == 'soft'}">
-            <param name="load_mass">0.0</param>
-            <param name="load_cog">[0.0, 0.0, 0.0]</param>
-            <param name="load_inertia">[0.0, 0.0, 0.0]</param>
-        </xacro:if>
-        <!-- Left AG2F90-D, pad is ignored by the model: TODO fill measured load. -->
-        <xacro:if value="${side == 'left' and gripper_type == 'ag2f90_d'}">
-            <param name="load_mass">0.0</param>
-            <param name="load_cog">[0.0, 0.0, 0.0]</param>
-            <param name="load_inertia">[0.0, 0.0, 0.0]</param>
-        </xacro:if>
-        <!-- Right RG75, default pad. -->
-        <xacro:if value="${side == 'right' and gripper_type == 'rg75' and gripper_pad != 'heavy_carry'}">
-            <param name="load_mass">1.62</param>
-            <param name="load_cog">[-0.0014285, 0.000579, 0.10439]</param>
-            <param name="load_inertia">[0.04874, 0.001, 0.001936]</param>
-        </xacro:if>
-        <!-- Right RG75, heavy_carry pad: TODO fill measured load. -->
-        <xacro:if value="${side == 'right' and gripper_type == 'rg75' and gripper_pad == 'heavy_carry'}">
-            <param name="load_mass">0.0</param>
-            <param name="load_cog">[0.0, 0.0, 0.0]</param>
-            <param name="load_inertia">[0.0, 0.0, 0.0]</param>
-        </xacro:if>
-        <!-- Right AG2F90-C, default pad: TODO fill measured load. -->
-        <xacro:if value="${side == 'right' and gripper_type == 'ag2f90_c' and gripper_pad != 'soft'}">
-            <param name="load_mass">0.0</param>
-            <param name="load_cog">[0.0, 0.0, 0.0]</param>
-            <param name="load_inertia">[0.0, 0.0, 0.0]</param>
-        </xacro:if>
-        <!-- Right AG2F90-C, soft pad: TODO fill measured load. -->
-        <xacro:if value="${side == 'right' and gripper_type == 'ag2f90_c' and gripper_pad == 'soft'}">
-            <param name="load_mass">0.0</param>
-            <param name="load_cog">[0.0, 0.0, 0.0]</param>
-            <param name="load_inertia">[0.0, 0.0, 0.0]</param>
-        </xacro:if>
-        <!-- Right AG2F90-D, pad is ignored by the model. -->
-        <xacro:if value="${side == 'right' and gripper_type == 'ag2f90_d'}">
-            <param name="load_mass">0.859</param>
-            <param name="load_cog">[0.007246, 0.01, 0.081]</param>
-            <param name="load_inertia">[0.0242, 0.01596, 0.00745]</param>
-        </xacro:if>
-    </xacro:macro>
-    <xacro:macro name="rokae_tool_load_params_with_override" params="side gripper_type gripper_pad load_mass load_cog load_inertia">
-        <xacro:property name="has_tool_load_override" value="${load_mass != '' and load_cog != '' and load_inertia != ''}"/>
-        <xacro:if value="${has_tool_load_override}">
-            <param name="load_mass">${load_mass}</param>
-            <param name="load_cog">${load_cog}</param>
-            <param name="load_inertia">${load_inertia}</param>
-        </xacro:if>
-        <xacro:unless value="${has_tool_load_override}">
-            <xacro:rokae_tool_load_params side="${side}" gripper_type="${gripper_type}" gripper_pad="${gripper_pad}"/>
-        </xacro:unless>
-    </xacro:macro>
     <xacro:macro name="rokae_side_hardware_block" params="
         side
@@ -149,13 +71,11 @@
             <param name="${side}_tool_velocity">1.0</param>
         </xacro:if>
-        <xacro:if value="${gripper_type != '' or hand_type != ''}">
-            <xacro:rokae_tool_load_params_with_override
-                side="${side}"
-                gripper_type="${gripper_type if gripper_type != '' else hand_type}"
-                gripper_pad="${gripper_pad}"
-                load_mass="${load_mass}"
-                load_cog="${load_cog}"
-                load_inertia="${load_inertia}"/>
-        </xacro:if>
+        <xacro:tool_load_params
+            side="${side}"
+            end_effector_type="${gripper_type if gripper_type != '' else hand_type}"
+            pad_type="${gripper_pad}"
+            mass="${load_mass}"
+            center_of_mass="${load_cog}"
+            diagonal_inertia="${load_inertia}"/>
     </xacro:macro>
 </robot>
