Commit message: Add external CAN support for LinkerHand

File: ar5_ccs_description/xacro/ros2_control/external_ee_systems.xacro (robot description, xacro)
@@ -15,7 +15,39 @@
         </ros2_control>
     </xacro:macro>
+    <xacro:macro name="linkerhand_usb_can_side_system" params="side hand_type can_interface read_tactile:=false">
+        <ros2_control name="${hand_type}_${side}_can_system" type="system" rw_rate="50">
+            <hardware>
+                <xacro:if value="${hand_type == 'linkerhand_o6'}">
+                    <plugin>can_ros2_control/O6CanHardware</plugin>
+                </xacro:if>
+                <xacro:if value="${hand_type == 'linkerhand_l6'}">
+                    <plugin>can_ros2_control/L6CanHardware</plugin>
+                </xacro:if>
+                <xacro:if value="${hand_type == 'linkerhand_o7'}">
+                    <plugin>can_ros2_control/O7CanHardware</plugin>
+                </xacro:if>
+                <param name="can_interface">${can_interface}</param>
+                <param name="hand_side">${side}</param>
+                <param name="read_feedback">true</param>
+                <param name="read_tactile">${read_tactile}</param>
+                <param name="${side}_tool_torque">1.0</param>
+                <param name="${side}_tool_velocity">1.0</param>
+            </hardware>
+            <xacro:side_hand_interfaces side="${side}" hand_type="${hand_type}"/>
+        </ros2_control>
+    </xacro:macro>
     <xacro:macro name="external_ee_systems" params="
         usb_left_port:=/dev/ttyUSB0
-        usb_right_port:=/dev/ttyUSB2">
+        usb_right_port:=/dev/ttyUSB2
+        left_ee_can_interface:=can0
+        right_ee_can_interface:=can1
+        left_read_tactile:=false
+        right_read_tactile:=false">
+        <xacro:if value="${left_drive_type == 'usb_can' and (left_hand_type == 'linkerhand_o6' or left_hand_type == 'linkerhand_l6' or left_hand_type == 'linkerhand_o7')}">
+            <xacro:linkerhand_usb_can_side_system side="left" hand_type="${left_hand_type}" can_interface="${left_ee_can_interface}" read_tactile="${left_read_tactile}"/>
+        </xacro:if>
+        <xacro:if value="${right_drive_type == 'usb_can' and (right_hand_type == 'linkerhand_o6' or right_hand_type == 'linkerhand_l6' or right_hand_type == 'linkerhand_o7')}">
+            <xacro:linkerhand_usb_can_side_system side="right" hand_type="${right_hand_type}" can_interface="${right_ee_can_interface}" read_tactile="${right_read_tactile}"/>
+        </xacro:if>
         <xacro:if value="${left_drive_type == 'usb' and (left_hand_type == 'linkerhand_o6' or left_hand_type == 'linkerhand_l6' or left_hand_type == 'linkerhand_o7')}">
             <xacro:side_usb_hand_system side="left" hand_type="${left_hand_type}" serial_port="${usb_left_port}"/>

File: ar5_ccs_description/xacro/ros2_control/robot.xacro (robot description, xacro)
@@ -21,4 +21,8 @@
 	<xacro:arg name="usb_left_port" default="/dev/ttyUSB0"/>
 	<xacro:arg name="usb_right_port" default="/dev/ttyUSB2"/>
+	<xacro:arg name="left_ee_can_interface" default="can0"/>
+	<xacro:arg name="right_ee_can_interface" default="can1"/>
+	<xacro:arg name="left_read_tactile" default="false"/>
+	<xacro:arg name="right_read_tactile" default="false"/>
 	<xacro:arg name="left_ee_drive_type" default=""/>
 	<xacro:arg name="right_ee_drive_type" default=""/>
@@ -28,6 +32,6 @@
 	<xacro:property name="right_drive_type" value="${'$(arg right_ee_drive_type)' if '$(arg right_ee_drive_type)' != '' else ee_drive_type}"/>
 	<xacro:property name="rokae_ctrl_mode" value="${'JOINT_IMPEDANCE' if '$(arg arm_ctrl_mode)' == 'joint_impedance' else 'POSITION'}"/>
-	<xacro:property name="left_rokae_hand_type" value="${'' if left_drive_type == 'usb' else left_hand_type}"/>
-	<xacro:property name="right_rokae_hand_type" value="${'' if right_drive_type == 'usb' else right_hand_type}"/>
+	<xacro:property name="left_rokae_hand_type" value="${'' if left_drive_type == 'usb' or left_drive_type == 'usb_can' else left_hand_type}"/>
+	<xacro:property name="right_rokae_hand_type" value="${'' if right_drive_type == 'usb' or right_drive_type == 'usb_can' else right_hand_type}"/>
 	<link name="world"/>
 	<joint name="world_fixed" type="fixed">
@@ -111,5 +115,9 @@
 		<xacro:external_ee_systems
 			usb_left_port="$(arg usb_left_port)"
-			usb_right_port="$(arg usb_right_port)"/>
+			usb_right_port="$(arg usb_right_port)"
+			left_ee_can_interface="$(arg left_ee_can_interface)"
+			right_ee_can_interface="$(arg right_ee_can_interface)"
+			left_read_tactile="$(arg left_read_tactile)"
+			right_read_tactile="$(arg right_read_tactile)"/>
 	</xacro:if>
 	<xacro:unless value="${is_real_hardware}">

Commit message: feat: add iNexus CAN end-effector mode

File: ar5_ccs_description/xacro/ros2_control/external_ee_systems.xacro (robot description, xacro)
@@ -11,4 +11,29 @@
                 <param name="hand_side">${side}</param>
                 <param name="max_speed_ratio">1.0</param>
+            </hardware>
+            <xacro:side_hand_interfaces side="${side}" hand_type="${hand_type}"/>
+        </ros2_control>
+    </xacro:macro>
+    <xacro:macro name="linkerhand_inex_can_side_system" params="side hand_type">
+        <!-- rw_rate controls how often ros2_control offers a new position target.
+             The plugin independently enforces the iNexus CAN TX frame interval. -->
+        <ros2_control name="${hand_type}_${side}_inex_can_system" type="system" rw_rate="50">
+            <hardware>
+                <xacro:if value="${hand_type == 'linkerhand_o6'}">
+                    <plugin>inex_ros2_control/O6Hardware</plugin>
+                </xacro:if>
+                <xacro:if value="${hand_type == 'linkerhand_l6'}">
+                    <plugin>inex_ros2_control/L6Hardware</plugin>
+                </xacro:if>
+                <xacro:if value="${hand_type == 'linkerhand_o7'}">
+                    <plugin>inex_ros2_control/O7Hardware</plugin>
+                </xacro:if>
+                <param name="hand_side">${side}</param>
+                <param name="read_feedback">true</param>
+                <param name="tx_interval_ms">5</param>
+                <param name="position_feedback_period_ms">20</param>
+                <param name="position_feedback_timeout_ms">40</param>
+                <param name="${side}_tool_torque">1.0</param>
+                <param name="${side}_tool_velocity">1.0</param>
             </hardware>
             <xacro:side_hand_interfaces side="${side}" hand_type="${hand_type}"/>
@@ -44,4 +69,10 @@
         left_read_tactile:=false
         right_read_tactile:=false">
+        <xacro:if value="${left_drive_type == 'inex_can' and (left_hand_type == 'linkerhand_o6' or left_hand_type == 'linkerhand_l6' or left_hand_type == 'linkerhand_o7')}">
+            <xacro:linkerhand_inex_can_side_system side="left" hand_type="${left_hand_type}"/>
+        </xacro:if>
+        <xacro:if value="${right_drive_type == 'inex_can' and (right_hand_type == 'linkerhand_o6' or right_hand_type == 'linkerhand_l6' or right_hand_type == 'linkerhand_o7')}">
+            <xacro:linkerhand_inex_can_side_system side="right" hand_type="${right_hand_type}"/>
+        </xacro:if>
         <xacro:if value="${left_drive_type == 'usb_can' and (left_hand_type == 'linkerhand_o6' or left_hand_type == 'linkerhand_l6' or left_hand_type == 'linkerhand_o7')}">
             <xacro:linkerhand_usb_can_side_system side="left" hand_type="${left_hand_type}" can_interface="${left_ee_can_interface}" read_tactile="${left_read_tactile}"/>

File: ar5_ccs_description/xacro/ros2_control/robot.xacro (robot description, xacro)
@@ -37,6 +37,6 @@
 	<xacro:property name="right_drive_type" value="${'$(arg right_ee_drive_type)' if '$(arg right_ee_drive_type)' != '' else ee_drive_type}"/>
 	<xacro:property name="rokae_ctrl_mode" value="${'JOINT_IMPEDANCE' if '$(arg arm_ctrl_mode)' == 'joint_impedance' else 'POSITION'}"/>
-	<xacro:property name="left_rokae_hand_type" value="${'' if left_drive_type == 'usb' or left_drive_type == 'usb_can' else left_hand_type}"/>
-	<xacro:property name="right_rokae_hand_type" value="${'' if right_drive_type == 'usb' or right_drive_type == 'usb_can' else right_hand_type}"/>
+	<xacro:property name="left_rokae_hand_type" value="${'' if left_drive_type == 'usb' or left_drive_type == 'usb_can' or left_drive_type == 'inex_can' else left_hand_type}"/>
+	<xacro:property name="right_rokae_hand_type" value="${'' if right_drive_type == 'usb' or right_drive_type == 'usb_can' or right_drive_type == 'inex_can' else right_hand_type}"/>
 	<link name="world"/>
 	<joint name="world_fixed" type="fixed">
