Commit message: feat: add linkerhand INEX RS-485 side system support in external EE systems

File: ar5_ccs_description/xacro/ros2_control/external_ee_systems.xacro (robot description, xacro)
@@ -59,4 +59,32 @@
         </ros2_control>
     </xacro:macro>
+    <xacro:macro name="linkerhand_inex_rs485_side_system" params="side hand_type rs485_channel">
+        <ros2_control name="${hand_type}_${side}_inex_rs485_system" type="system" rw_rate="30">
+            <hardware>
+                <xacro:if value="${hand_type == 'linkerhand_o6'}">
+                    <plugin>inex_ros2_control/O6LinkerHandRs485Hardware</plugin>
+                </xacro:if>
+                <xacro:if value="${hand_type == 'linkerhand_l6'}">
+                    <plugin>inex_ros2_control/L6LinkerHandRs485Hardware</plugin>
+                </xacro:if>
+                <xacro:if value="${hand_type == 'linkerhand_o7'}">
+                    <plugin>inex_ros2_control/O7LinkerHandRs485Hardware</plugin>
+                </xacro:if>
+                <param name="hand_side">${side}</param>
+                <param name="rs485_channel">${rs485_channel}</param>
+                <!-- slave_id intentionally omitted: right=0x27, left=0x28. -->
+                <param name="transaction_interval_ms">10</param>
+                <param name="position_period_ms">33</param>
+                <param name="position_feedback_period_ms">33</param>
+                <param name="position_feedback_timeout_ms">40</param>
+                <param name="command_deadband_raw">0</param>
+                <param name="max_consecutive_failures">5</param>
+                <param name="read_feedback">true</param>
+                <param name="${side}_tool_torque">1.0</param>
+                <param name="${side}_tool_velocity">1.0</param>
+            </hardware>
+            <xacro:side_hand_interfaces side="${side}" hand_type="${hand_type}"/>
+        </ros2_control>
+    </xacro:macro>
     <xacro:macro name="linkerhand_usb_can_side_system" params="side hand_type can_interface read_tactile:=false">
         <ros2_control name="${hand_type}_${side}_can_system" type="system" rw_rate="50">
@@ -98,4 +126,10 @@
             <xacro:ag2f90d_inex_rs485_side_system side="right" rs485_channel="${right_ee_rs485_channel}" slave_id="${right_ee_modbus_slave_id}"/>
         </xacro:if>
+        <xacro:if value="${arm_driver == 'inex' and left_drive_type == 'inex_rs485' and (left_hand_type == 'linkerhand_o6' or left_hand_type == 'linkerhand_l6' or left_hand_type == 'linkerhand_o7')}">
+            <xacro:linkerhand_inex_rs485_side_system side="left" hand_type="${left_hand_type}" rs485_channel="${left_ee_rs485_channel}"/>
+        </xacro:if>
+        <xacro:if value="${arm_driver == 'inex' and right_drive_type == 'inex_rs485' and (right_hand_type == 'linkerhand_o6' or right_hand_type == 'linkerhand_l6' or right_hand_type == 'linkerhand_o7')}">
+            <xacro:linkerhand_inex_rs485_side_system side="right" hand_type="${right_hand_type}" rs485_channel="${right_ee_rs485_channel}"/>
+        </xacro:if>
         <xacro:if value="${arm_driver == 'inex' and left_drive_type == 'inex_can' and (left_hand_type == 'linkerhand_o6' or left_hand_type == 'linkerhand_l6' or left_hand_type == 'linkerhand_o7')}">
             <xacro:linkerhand_inex_can_side_system side="left" hand_type="${left_hand_type}"/>

File: ar5_ccs_description/xacro/ros2_control/robot.xacro (robot description, xacro)
@@ -37,6 +37,6 @@
 	<xacro:property name="validated_hardware_type" value="${1 if '$(arg ros2_control_hardware_type)' in ('mock_components', 'gz', 'isaac', 'real') else 0}"/>
 	<xacro:property name="validated_arm_driver" value="${1 if arm_driver in ('rokae', 'inex') else 0}"/>
-	<xacro:property name="validated_left_drive" value="${1 if arm_driver + ':' + left_drive_type in ('rokae:none', 'rokae:rokae_rs485', 'rokae:usb_rs485', 'rokae:usb_can', 'inex:none', 'inex:inex_can', 'inex:usb_rs485', 'inex:usb_can') else 0}"/>
-	<xacro:property name="validated_right_drive" value="${1 if arm_driver + ':' + right_drive_type in ('rokae:none', 'rokae:rokae_rs485', 'rokae:usb_rs485', 'rokae:usb_can', 'inex:none', 'inex:inex_can', 'inex:usb_rs485', 'inex:usb_can') else 0}"/>
+	<xacro:property name="validated_left_drive" value="${1 if arm_driver + ':' + left_drive_type in ('rokae:none', 'rokae:rokae_rs485', 'rokae:usb_rs485', 'rokae:usb_can', 'inex:none', 'inex:inex_rs485', 'inex:inex_can', 'inex:usb_rs485', 'inex:usb_can') else 0}"/>
+	<xacro:property name="validated_right_drive" value="${1 if arm_driver + ':' + right_drive_type in ('rokae:none', 'rokae:rokae_rs485', 'rokae:usb_rs485', 'rokae:usb_can', 'inex:none', 'inex:inex_rs485', 'inex:inex_can', 'inex:usb_rs485', 'inex:usb_can') else 0}"/>
 	<xacro:property name="rokae_ctrl_mode" value="${'JOINT_IMPEDANCE' if '$(arg arm_ctrl_mode)' == 'joint_impedance' else 'POSITION'}"/>
 	<xacro:property name="left_rokae_hand_type" value="${left_hand_type if arm_driver == 'rokae' and left_drive_type == 'rokae_rs485' else ''}"/>

Commit message: fix: update validated drive properties for left and right arms in robot.xacro

File: ar5_ccs_description/xacro/ros2_control/external_ee_systems.xacro (robot description, xacro)
@@ -94,6 +94,6 @@
         </ros2_control>
     </xacro:macro>
-    <xacro:macro name="linkerhand_usb_can_side_system" params="side hand_type can_interface read_tactile:=false">
-        <ros2_control name="${hand_type}_${side}_can_system" type="system" rw_rate="50">
+    <xacro:macro name="linkerhand_usb_can_side_system" params="side hand_type can_interface read_tactile:=false rw_rate:=''">
+        <ros2_control name="${hand_type}_${side}_can_system" type="system" rw_rate="${rw_rate if rw_rate != '' else 50}">
             <hardware>
                 <xacro:if value="${hand_type == 'linkerhand_o6'}">

File: ar5_ccs_description/xacro/ros2_control/robot.xacro (robot description, xacro)
@@ -37,6 +37,6 @@
 	<xacro:property name="validated_hardware_type" value="${1 if '$(arg ros2_control_hardware_type)' in ('mock_components', 'gz', 'isaac', 'real') else 0}"/>
 	<xacro:property name="validated_arm_driver" value="${1 if arm_driver in ('rokae', 'inex') else 0}"/>
-	<xacro:property name="validated_left_drive" value="${1 if arm_driver + ':' + left_drive_type in ('rokae:none', 'rokae:rokae_rs485', 'rokae:usb_rs485', 'rokae:usb_can', 'inex:none', 'inex:inex_rs485', 'inex:inex_can', 'inex:usb_rs485', 'inex:usb_can') else 0}"/>
-	<xacro:property name="validated_right_drive" value="${1 if arm_driver + ':' + right_drive_type in ('rokae:none', 'rokae:rokae_rs485', 'rokae:usb_rs485', 'rokae:usb_can', 'inex:none', 'inex:inex_rs485', 'inex:inex_can', 'inex:usb_rs485', 'inex:usb_can') else 0}"/>
+	<xacro:property name="validated_left_drive" value="${1 if (arm_driver + ':' + left_drive_type in ('rokae:none', 'rokae:rokae_rs485', 'inex:none', 'inex:inex_rs485', 'inex:inex_can') and (left_drive_type != 'inex_rs485' or left_gripper_type == 'ag2f90_d' or left_hand_type in ('linkerhand_o6', 'linkerhand_l6', 'linkerhand_o7'))) or (left_drive_type in ('usb', 'usb_rs485') and (left_hand_type in ('linkerhand_o6', 'linkerhand_l6', 'linkerhand_o7', 'freedom_v1', 'freedom_v2', 'inspire_e2', 'inspire_f2', 'xhand1', 'theohand_std16a') or left_gripper_type in ('rg75', 'ag2f90_d'))) or (left_drive_type == 'usb_can' and left_hand_type in ('linkerhand_o6', 'linkerhand_l6', 'linkerhand_o7', 'freedom_v1', 'inspire_e2', 'inspire_f2')) else 0}"/>
+	<xacro:property name="validated_right_drive" value="${1 if (arm_driver + ':' + right_drive_type in ('rokae:none', 'rokae:rokae_rs485', 'inex:none', 'inex:inex_rs485', 'inex:inex_can') and (right_drive_type != 'inex_rs485' or right_gripper_type == 'ag2f90_d' or right_hand_type in ('linkerhand_o6', 'linkerhand_l6', 'linkerhand_o7'))) or (right_drive_type in ('usb', 'usb_rs485') and (right_hand_type in ('linkerhand_o6', 'linkerhand_l6', 'linkerhand_o7', 'freedom_v1', 'freedom_v2', 'inspire_e2', 'inspire_f2', 'xhand1', 'theohand_std16a') or right_gripper_type in ('rg75', 'ag2f90_d'))) or (right_drive_type == 'usb_can' and right_hand_type in ('linkerhand_o6', 'linkerhand_l6', 'linkerhand_o7', 'freedom_v1', 'inspire_e2', 'inspire_f2')) else 0}"/>
 	<xacro:property name="rokae_ctrl_mode" value="${'JOINT_IMPEDANCE' if '$(arg arm_ctrl_mode)' == 'joint_impedance' else 'POSITION'}"/>
 	<!-- INEX needs the selected EEF type for payload lookup even when the EEF uses an external bus. -->

Commit message: feat: enhance left and right drive validation for gripper types in robot.xacro

File: ar5_ccs_description/xacro/ros2_control/external_ee_systems.xacro (robot description, xacro)
@@ -196,9 +196,9 @@
             <xacro:inspire_canfd_side_system side="right" can_interface="${right_ee_can_interface}" hand_type="${right_hand_type}" rw_rate="${right_ee_rw_rate}"/>
         </xacro:if>
-        <xacro:if value="${left_drive_type in ('usb', 'usb_rs485') and left_gripper_type == 'ag2f90_d'}">
-            <xacro:changingtek_usb_side_system side="left" variant="90d" serial_port="${usb_left_port}" rw_rate="${left_ee_rw_rate}"/>
-        </xacro:if>
-        <xacro:if value="${right_drive_type in ('usb', 'usb_rs485') and right_gripper_type == 'ag2f90_d'}">
-            <xacro:changingtek_usb_side_system side="right" variant="90d" serial_port="${usb_right_port}" rw_rate="${right_ee_rw_rate}"/>
+        <xacro:if value="${left_drive_type in ('usb', 'usb_rs485') and left_gripper_type in ('ag2f90_c', 'ag2f90_d')}">
+            <xacro:changingtek_usb_side_system side="left" variant="${'90c' if left_gripper_type == 'ag2f90_c' else '90d'}" serial_port="${usb_left_port}" rw_rate="${left_ee_rw_rate}"/>
+        </xacro:if>
+        <xacro:if value="${right_drive_type in ('usb', 'usb_rs485') and right_gripper_type in ('ag2f90_c', 'ag2f90_d')}">
+            <xacro:changingtek_usb_side_system side="right" variant="${'90c' if right_gripper_type == 'ag2f90_c' else '90d'}" serial_port="${usb_right_port}" rw_rate="${right_ee_rw_rate}"/>
         </xacro:if>
         <xacro:if value="${left_drive_type in ('usb', 'usb_rs485') and left_gripper_type == 'rg75'}">

File: ar5_ccs_description/xacro/ros2_control/robot.xacro (robot description, xacro)
@@ -37,6 +37,6 @@
 	<xacro:property name="validated_hardware_type" value="${1 if '$(arg ros2_control_hardware_type)' in ('mock_components', 'gz', 'isaac', 'real') else 0}"/>
 	<xacro:property name="validated_arm_driver" value="${1 if arm_driver in ('rokae', 'inex') else 0}"/>
-	<xacro:property name="validated_left_drive" value="${1 if (arm_driver + ':' + left_drive_type in ('rokae:none', 'rokae:rokae_rs485', 'inex:none', 'inex:inex_rs485', 'inex:inex_can') and (left_drive_type != 'inex_rs485' or left_gripper_type == 'ag2f90_d' or left_hand_type in ('linkerhand_o6', 'linkerhand_l6', 'linkerhand_o7'))) or (left_drive_type in ('usb', 'usb_rs485') and (left_hand_type in ('linkerhand_o6', 'linkerhand_l6', 'linkerhand_o7', 'freedom_v1', 'freedom_v2', 'inspire_e2', 'inspire_f2', 'xhand1', 'theohand_std16a') or left_gripper_type in ('rg75', 'ag2f90_d'))) or (left_drive_type == 'usb_can' and left_hand_type in ('linkerhand_o6', 'linkerhand_l6', 'linkerhand_o7', 'freedom_v1', 'inspire_e2', 'inspire_f2')) else 0}"/>
-	<xacro:property name="validated_right_drive" value="${1 if (arm_driver + ':' + right_drive_type in ('rokae:none', 'rokae:rokae_rs485', 'inex:none', 'inex:inex_rs485', 'inex:inex_can') and (right_drive_type != 'inex_rs485' or right_gripper_type == 'ag2f90_d' or right_hand_type in ('linkerhand_o6', 'linkerhand_l6', 'linkerhand_o7'))) or (right_drive_type in ('usb', 'usb_rs485') and (right_hand_type in ('linkerhand_o6', 'linkerhand_l6', 'linkerhand_o7', 'freedom_v1', 'freedom_v2', 'inspire_e2', 'inspire_f2', 'xhand1', 'theohand_std16a') or right_gripper_type in ('rg75', 'ag2f90_d'))) or (right_drive_type == 'usb_can' and right_hand_type in ('linkerhand_o6', 'linkerhand_l6', 'linkerhand_o7', 'freedom_v1', 'inspire_e2', 'inspire_f2')) else 0}"/>
+	<xacro:property name="validated_left_drive" value="${1 if (arm_driver + ':' + left_drive_type in ('rokae:none', 'rokae:rokae_rs485', 'inex:none', 'inex:inex_rs485', 'inex:inex_can') and (left_drive_type != 'inex_rs485' or left_gripper_type == 'ag2f90_d' or left_hand_type in ('linkerhand_o6', 'linkerhand_l6', 'linkerhand_o7'))) or (left_drive_type in ('usb', 'usb_rs485') and (left_hand_type in ('linkerhand_o6', 'linkerhand_l6', 'linkerhand_o7', 'freedom_v1', 'freedom_v2', 'inspire_e2', 'inspire_f2', 'xhand1', 'theohand_std16a') or left_gripper_type in ('rg75', 'ag2f90_c', 'ag2f90_d'))) or (left_drive_type == 'usb_can' and left_hand_type in ('linkerhand_o6', 'linkerhand_l6', 'linkerhand_o7', 'freedom_v1', 'inspire_e2', 'inspire_f2')) else 0}"/>
+	<xacro:property name="validated_right_drive" value="${1 if (arm_driver + ':' + right_drive_type in ('rokae:none', 'rokae:rokae_rs485', 'inex:none', 'inex:inex_rs485', 'inex:inex_can') and (right_drive_type != 'inex_rs485' or right_gripper_type == 'ag2f90_d' or right_hand_type in ('linkerhand_o6', 'linkerhand_l6', 'linkerhand_o7'))) or (right_drive_type in ('usb', 'usb_rs485') and (right_hand_type in ('linkerhand_o6', 'linkerhand_l6', 'linkerhand_o7', 'freedom_v1', 'freedom_v2', 'inspire_e2', 'inspire_f2', 'xhand1', 'theohand_std16a') or right_gripper_type in ('rg75', 'ag2f90_c', 'ag2f90_d'))) or (right_drive_type == 'usb_can' and right_hand_type in ('linkerhand_o6', 'linkerhand_l6', 'linkerhand_o7', 'freedom_v1', 'inspire_e2', 'inspire_f2')) else 0}"/>
 	<xacro:property name="rokae_ctrl_mode" value="${'JOINT_IMPEDANCE' if '$(arg arm_ctrl_mode)' == 'joint_impedance' else 'POSITION'}"/>
 	<!-- INEX needs the selected EEF type for payload lookup even when the EEF uses an external bus. -->
